File: fm-rpt-control-roger-beep.kicad_sch (KiCad schematic)
At the start: 21 parts, among them Q1 BC858, Q2 BC858, Q3 BC848, U10 HEF4093B

Commit message: daily
Parts:
- renumbered C7 to C10, C8 to C11, C9 to C12, C5 to C8, C6 to C9, D2 to D8, Q1 to Q2, Q2 to Q3, Q3 to Q4, R9 to R32, R10 to R33, R11 to R34, R12 to R35, R13 to R36, R14 to R37, R15 to R38, R16 to R39, U10 to U27

Commit message: second daily
Parts:
- renumbered Q2 to Q3, Q3 to Q4, Q4 to Q5, U27 to U37
Changed lines of the file:
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@@
   (symbol (lib_id "Transistor_BJT:BC858") (at 110.49 66.04 0) (mirror x) (unit 1)
     (in_bom yes) (on_board yes) (fields_autoplaced)
-    (property "Reference" "Q2" (id 0) (at 115.3414 65.2053 0)
+    (property "Reference" "Q3" (id 0) (at 115.3414 65.2053 0)
       (effects (font (size 1.27 1.27)) (justify left))
     )
@@
   (symbol (lib_id "4xxx:HEF4093B") (at 162.56 119.38 0) (unit 4)
     (in_bom yes) (on_board yes) (fields_autoplaced)
-    (property "Reference" "U27" (id 0) (at 162.56 111.8702 0))
+    (property "Reference" "U37" (id 0) (at 162.56 111.8702 0))
     (property "Value" "HEF4093B" (id 1) (at 162.56 114.4071 0))
     (property "Footprint" "" (id 2) (at 162.56 119.38 0)
@@
   (symbol (lib_id "4xxx:HEF4093B") (at 167.64 86.36 0) (unit 1)
     (in_bom yes) (on_board yes) (fields_autoplaced)
-    (property "Reference" "U27" (id 0) (at 167.64 78.8502 0))
+    (property "Reference" "U37" (id 0) (at 167.64 78.8502 0))
     (property "Value" "HEF4093B" (id 1) (at 167.64 81.3871 0))
     (property "Footprint" "Package_SO:SO-14_3.9x8.65mm_P1.27mm" (id 2) (at 167.64 86.36 0)
@@
   (symbol (lib_id "4xxx:HEF4093B") (at 127 95.25 0) (mirror y) (unit 3)
     (in_bom yes) (on_board yes) (fields_autoplaced)
-    (property "Reference" "U27" (id 0) (at 127 87.7402 0))
+    (property "Reference" "U37" (id 0) (at 127 87.7402 0))
     (property "Value" "HEF4093B" (id 1) (at 127 90.2771 0))
     (property "Footprint" "" (id 2) (at 127 95.25 0)
@@
   (symbol (lib_id "paratnc_cp_import:GND") (at 214.63 104.14 0) (unit 1)
     (in_bom yes) (on_board yes) (fields_autoplaced)
-    (property "Reference" "#GND043" (id 0) (at 214.63 104.14 0)
+    (property "Reference" "#GND045" (id 0) (at 214.63 104.14 0)
       (effects (font (size 1.27 1.27)) hide)
     )
@@
   (symbol (lib_id "4xxx:HEF4093B") (at 214.63 87.63 0) (unit 5)
     (in_bom yes) (on_board yes) (fields_autoplaced)
-    (property "Reference" "U27" (id 0) (at 220.472 86.7953 0)
+    (property "Reference" "U37" (id 0) (at 220.472 86.7953 0)
       (effects (font (size 1.27 1.27)) (justify left))
     )
@@
   (symbol (lib_id "paratnc_cp_import:GND") (at 140.97 138.43 0) (unit 1)
     (in_bom yes) (on_board yes) (fields_autoplaced)
-    (property "Reference" "#GND038" (id 0) (at 140.97 138.43 0)
+    (property "Reference" "#GND040" (id 0) (at 140.97 138.43 0)
       (effects (font (size 1.27 1.27)) hide)
     )
@@
   (symbol (lib_id "paratnc_cp_import:GND") (at 196.85 138.43 0) (unit 1)
     (in_bom yes) (on_board yes) (fields_autoplaced)
-    (property "Reference" "#GND042" (id 0) (at 196.85 138.43 0)
+    (property "Reference" "#GND044" (id 0) (at 196.85 138.43 0)
       (effects (font (size 1.27 1.27)) hide)
     )
@@
   (symbol (lib_id "paratnc_cp_import:GND") (at 113.03 90.17 0) (unit 1)
     (in_bom yes) (on_board yes) (fields_autoplaced)
-    (property "Reference" "#GND037" (id 0) (at 113.03 90.17 0)
+    (property "Reference" "#GND039" (id 0) (at 113.03 90.17 0)
       (effects (font (size 1.27 1.27)) hide)
     )
@@
   (symbol (lib_id "paratnc_cp_import:GND") (at 182.88 138.43 0) (unit 1)
     (in_bom yes) (on_board yes) (fields_autoplaced)
-    (property "Reference" "#GND041" (id 0) (at 182.88 138.43 0)
+    (property "Reference" "#GND043" (id 0) (at 182.88 138.43 0)
       (effects (font (size 1.27 1.27)) hide)
     )
@@
   (symbol (lib_id "paratnc_cp_import:GND") (at 149.86 138.43 0) (unit 1)
     (in_bom yes) (on_board yes) (fields_autoplaced)
-    (property "Reference" "#GND039" (id 0) (at 149.86 138.43 0)
+    (property "Reference" "#GND041" (id 0) (at 149.86 138.43 0)
       (effects (font (size 1.27 1.27)) hide)
     )
@@
   (symbol (lib_id "Transistor_BJT:BC858") (at 110.49 118.11 180) (unit 1)
     (in_bom yes) (on_board yes) (fields_autoplaced)
-    (property "Reference" "Q3" (id 0) (at 105.6386 117.2753 0)
+    (property "Reference" "Q4" (id 0) (at 105.6386 117.2753 0)
       (effects (font (size 1.27 1.27)) (justify left))
     )
@@
   (symbol (lib_id "Transistor_BJT:BC848") (at 138.43 127 0) (unit 1)
     (in_bom yes) (on_board yes) (fields_autoplaced)
-    (property "Reference" "Q4" (id 0) (at 143.2814 126.1653 0)
+    (property "Reference" "Q5" (id 0) (at 143.2814 126.1653 0)
       (effects (font (size 1.27 1.27)) (justify left))
     )
@@
   (symbol (lib_id "paratnc_cp_import:GND") (at 168.91 95.25 90) (unit 1)
     (in_bom yes) (on_board yes) (fields_autoplaced)
-    (property "Reference" "#GND040" (id 0) (at 168.91 95.25 0)
+    (property "Reference" "#GND042" (id 0) (at 168.91 95.25 0)
       (effects (font (size 1.27 1.27)) hide)
     )
@@
   (symbol (lib_id "4xxx:HEF4093B") (at 128.27 77.47 0) (unit 2)
     (in_bom yes) (on_board yes) (fields_autoplaced)
-    (property "Reference" "U27" (id 0) (at 128.27 69.9602 0))
+    (property "Reference" "U37" (id 0) (at 128.27 69.9602 0))
     (property "Value" "HEF4093B" (id 1) (at 128.27 72.4971 0))
     (property "Footprint" "" (id 2) (at 128.27 77.47 0)
@@
   (symbol (lib_id "paratnc_cp_import:GND") (at 107.95 138.43 0) (unit 1)
     (in_bom yes) (on_board yes) (fields_autoplaced)
-    (property "Reference" "#GND036" (id 0) (at 107.95 138.43 0)
-      (effects (font (size 1.27 1.27)) hide)
-    )
+    (property "Reference" "#GND038" (id 0) (at 107.95 138.43 0)
+      (effects (font (size 1.27 1.27)) hide)
+    )

Commit message: daily
Parts:
- C16: renamed from C8; footprint (none) -> Capacitor_SMD:C_0805_2012Metric_Pad1.18x1.45mm_HandSolder
- C18: renamed from C10; footprint (none) -> Capacitor_SMD:C_0805_2012Metric_Pad1.18x1.45mm_HandSolder
- C19: renamed from C11; footprint (none) -> Capacitor_Tantalum_SMD:CP_EIA-3528-21_Kemet-B_Pad1.50x2.35mm_HandSolder
- C20: renamed from C12; footprint (none) -> Capacitor_SMD:C_0805_2012Metric_Pad1.18x1.45mm_HandSolder
- R52: renamed from R32; footprint (none) -> Resistor_SMD:R_0805_2012Metric_Pad1.20x1.40mm_HandSolder
- R53: renamed from R33; footprint (none) -> Resistor_SMD:R_0805_2012Metric_Pad1.20x1.40mm_HandSolder
- R54: renamed from R34; footprint (none) -> Resistor_SMD:R_0805_2012Metric_Pad1.20x1.40mm_HandSolder
- R55: renamed from R35; footprint (none) -> Resistor_SMD:R_0805_2012Metric_Pad1.20x1.40mm_HandSolder
- R56: renamed from R36; footprint (none) -> Resistor_SMD:R_0805_2012Metric_Pad1.20x1.40mm_HandSolder
- R57: renamed from R37; footprint (none) -> Resistor_SMD:R_0805_2012Metric_Pad1.20x1.40mm_HandSolder
- R58: renamed from R38; footprint (none) -> Resistor_SMD:R_0805_2012Metric_Pad1.20x1.40mm_HandSolder
- R59: renamed from R39; footprint (none) -> Resistor_SMD:R_0805_2012Metric_Pad1.20x1.40mm_HandSolder
- renumbered C9 to C17, D8 to D11, Q3 to Q5, Q4 to Q6, Q5 to Q7, U37 to U30

Commit message: schematic design ready
Parts:
- RV1, RV2, RV3: footprint (none) -> Potentiometer_SMD:Potentiometer_Bourns_3314J_Vertical
- U30: footprint (none) -> Package_SO:SO-8_3.9x4.9mm_P1.27mm
- U30: footprint Package_SO:SO-14_3.9x8.65mm_P1.27mm -> Package_SO:SO-8_3.9x4.9mm_P1.27mm
Changed lines of the file:
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@@
     (property "Reference" "RV1" (id 0) (at 143.51 84.1842 90))
     (property "Value" "100k" (id 1) (at 143.51 86.7211 90))
-    (property "Footprint" "" (id 2) (at 143.51 88.9 0)
+    (property "Footprint" "Potentiometer_SMD:Potentiometer_Bourns_3314J_Vertical" (id 2) (at 143.51 88.9 0)
       (effects (font (size 1.27 1.27)) hide)
     )
@@
     (property "Reference" "U30" (id 0) (at 162.56 111.8702 0))
     (property "Value" "HEF4093B" (id 1) (at 162.56 114.4071 0))
-    (property "Footprint" "" (id 2) (at 162.56 119.38 0)
+    (property "Footprint" "Package_SO:SO-8_3.9x4.9mm_P1.27mm" (id 2) (at 162.56 119.38 0)
       (effects (font (size 1.27 1.27)) hide)
     )
@@
     (property "Reference" "U30" (id 0) (at 167.64 78.8502 0))
     (property "Value" "HEF4093B" (id 1) (at 167.64 81.3871 0))
-    (property "Footprint" "Package_SO:SO-14_3.9x8.65mm_P1.27mm" (id 2) (at 167.64 86.36 0)
+    (property "Footprint" "Package_SO:SO-8_3.9x4.9mm_P1.27mm" (id 2) (at 167.64 86.36 0)
       (effects (font (size 1.27 1.27)) hide)
     )
@@
     (property "Reference" "U30" (id 0) (at 127 87.7402 0))
     (property "Value" "HEF4093B" (id 1) (at 127 90.2771 0))
-    (property "Footprint" "" (id 2) (at 127 95.25 0)
+    (property "Footprint" "Package_SO:SO-8_3.9x4.9mm_P1.27mm" (id 2) (at 127 95.25 0)
       (effects (font (size 1.27 1.27)) hide)
     )
@@
     (property "Reference" "RV2" (id 0) (at 162.56 99.4242 90))
     (property "Value" "10k" (id 1) (at 162.56 101.9611 90))
-    (property "Footprint" "" (id 2) (at 162.56 104.14 0)
+    (property "Footprint" "Potentiometer_SMD:Potentiometer_Bourns_3314J_Vertical" (id 2) (at 162.56 104.14 0)
       (effects (font (size 1.27 1.27)) hide)
     )
@@
       (effects (font (size 1.27 1.27)) (justify left))
     )
-    (property "Footprint" "" (id 2) (at 214.63 87.63 0)
+    (property "Footprint" "Package_SO:SO-8_3.9x4.9mm_P1.27mm" (id 2) (at 214.63 87.63 0)
       (effects (font (size 1.27 1.27)) hide)
     )
@@
     (property "Reference" "U30" (id 0) (at 128.27 69.9602 0))
     (property "Value" "HEF4093B" (id 1) (at 128.27 72.4971 0))
-    (property "Footprint" "" (id 2) (at 128.27 77.47 0)
+    (property "Footprint" "Package_SO:SO-8_3.9x4.9mm_P1.27mm" (id 2) (at 128.27 77.47 0)
       (effects (font (size 1.27 1.27)) hide)
     )
@@
       (effects (font (size 1.27 1.27)) (justify right))
     )
-    (property "Footprint" "" (id 2) (at 196.85 129.54 0)
-      (effects (font (size 1.27 1.27)) hide)
-    )
+    (property "Footprint" "Potentiometer_SMD:Potentiometer_Bourns_3314J_Vertical" (id 2) (at 196.85 129.54 0)
+      (effects (font (size 1.27 1.27)) hide)
+    )
