File: fm-rpt-control-roger-beep.kicad_sch (KiCad schematic)
At the start: 26 parts, among them Q5 BC858, Q6 BC858, Q7 BC848, U31 HEF4093B, U32 74AHC1G32GW

Commit message: before replacing some pinheaders with switches
Connections:
- net VDDA is gone; now on net VCC: C19.1, C20.1, Q5.2 (E), Q6.2 (E), R64.1, U31.14 (VCC)
Changed lines of the file:
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@@
     (effects (font (size 1.27 1.27)) (justify left bottom))
-  )
-  (global_label "VDDA" (shape input) (at 113.03 58.42 90) (fields_autoplaced)
-    (effects (font (size 1.27 1.27)) (justify left))
-    (property "Intersheet References" "${INTERSHEET_REFS}" (id 0) (at 112.9506 51.2898 90)
-      (effects (font (size 1.27 1.27)) (justify left) hide)
-    )
   )
   (global_label "+5V" (shape input) (at 159.385 33.02 90) (fields_autoplaced)
@@
     )
   )
+  (global_label "+5V" (shape input) (at 140.97 106.68 90) (fields_autoplaced)
+    (effects (font (size 1.27 1.27)) (justify left))
+    (property "Intersheet References" "${INTERSHEET_REFS}" (id 0) (at 140.8906 100.3964 90)
+      (effects (font (size 1.27 1.27)) (justify left) hide)
+    )
+  )
   (global_label "ROGER_PTT_INPUT" (shape input) (at 95.25 66.04 180) (fields_autoplaced)
     (effects (font (size 1.27 1.27)) (justify right))
     (property "Intersheet References" "${INTERSHEET_REFS}" (id 0) (at 75.9036 65.9606 0)
       (effects (font (size 1.27 1.27)) (justify right) hide)
-    )
-  )
-  (global_label "VDDA" (shape input) (at 214.63 72.39 90) (fields_autoplaced)
-    (effects (font (size 1.27 1.27)) (justify left))
-    (property "Intersheet References" "${INTERSHEET_REFS}" (id 0) (at 214.5506 65.2598 90)
-      (effects (font (size 1.27 1.27)) (justify left) hide)
     )
   )
@@
     )
   )
-  (global_label "VDDA" (shape input) (at 140.97 106.68 90) (fields_autoplaced)
-    (effects (font (size 1.27 1.27)) (justify left))
-    (property "Intersheet References" "${INTERSHEET_REFS}" (id 0) (at 140.8906 99.5498 90)
-      (effects (font (size 1.27 1.27)) (justify left) hide)
-    )
-  )
   (global_label "RETRANSMIT_DBCED" (shape input) (at 125.095 42.545 180) (fields_autoplaced)
     (effects (font (size 1.27 1.27)) (justify right))
@@
     )
   )
-  (global_label "VDDA" (shape input) (at 107.95 110.49 90) (fields_autoplaced)
+  (global_label "+5V" (shape input) (at 107.95 110.49 90) (fields_autoplaced)
     (effects (font (size 1.27 1.27)) (justify left))
-    (property "Intersheet References" "${INTERSHEET_REFS}" (id 0) (at 107.8706 103.3598 90)
+    (property "Intersheet References" "${INTERSHEET_REFS}" (id 0) (at 107.8706 104.2064 90)
       (effects (font (size 1.27 1.27)) (justify left) hide)
     )
+  )
+  (global_label "+5V" (shape input) (at 214.63 72.39 90) (fields_autoplaced)
+    (effects (font (size 1.27 1.27)) (justify left))
+    (property "Intersheet References" "${INTERSHEET_REFS}" (id 0) (at 214.5506 66.1064 90)
+      (effects (font (size 1.27 1.27)) (justify left) hide)
+    )
+  )
+  (global_label "+5V" (shape input) (at 113.03 58.42 90) (fields_autoplaced)
+    (effects (font (size 1.27 1.27)) (justify left))
+    (property "Intersheet References" "${INTERSHEET_REFS}" (id 0) (at 112.9506 52.1364 90)
+      (effects (font (size 1.27 1.27)) (justify left) hide)
+    )

Commit message: +5v bus removed completely
Connections:
- net VCC: no longer C19.1, C20.1, Q5.2 (E), Q6.2 (E), R64.1, U31.14 (VCC)
- new net: C19.1, C20.1, U31.14 (VCC)
Changed lines of the file:
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@@
     (effects (font (size 1.27 1.27)) (justify left bottom))
-  )
-  (global_label "+5V" (shape input) (at 159.385 33.02 90) (fields_autoplaced)
-    (effects (font (size 1.27 1.27)) (justify left))
-    (property "Intersheet References" "${INTERSHEET_REFS}" (id 0) (at 159.3056 26.7364 90)
-      (effects (font (size 1.27 1.27)) (justify left) hide)
-    )
-  )
-  (global_label "+5V" (shape input) (at 140.97 106.68 90) (fields_autoplaced)
-    (effects (font (size 1.27 1.27)) (justify left))
-    (property "Intersheet References" "${INTERSHEET_REFS}" (id 0) (at 140.8906 100.3964 90)
-      (effects (font (size 1.27 1.27)) (justify left) hide)
-    )
   )
   (global_label "ROGER_PTT_INPUT" (shape input) (at 95.25 66.04 180) (fields_autoplaced)
@@
       (effects (font (size 1.27 1.27)) (justify left) hide)
     )
-  )
-  (global_label "+5V" (shape input) (at 107.95 110.49 90) (fields_autoplaced)
-    (effects (font (size 1.27 1.27)) (justify left))
-    (property "Intersheet References" "${INTERSHEET_REFS}" (id 0) (at 107.8706 104.2064 90)
-      (effects (font (size 1.27 1.27)) (justify left) hide)
-    )
-  )
-  (global_label "+5V" (shape input) (at 214.63 72.39 90) (fields_autoplaced)
-    (effects (font (size 1.27 1.27)) (justify left))
-    (property "Intersheet References" "${INTERSHEET_REFS}" (id 0) (at 214.5506 66.1064 90)
-      (effects (font (size 1.27 1.27)) (justify left) hide)
-    )
-  )
-  (global_label "+5V" (shape input) (at 113.03 58.42 90) (fields_autoplaced)
-    (effects (font (size 1.27 1.27)) (justify left))
-    (property "Intersheet References" "${INTERSHEET_REFS}" (id 0) (at 112.9506 52.1364 90)
-      (effects (font (size 1.27 1.27)) (justify left) hide)
-    )

Commit message: short fixed
Connections:
- net +5V: now reaches Q5.2 (E)
- net +5V: now also C19.1, C20.1, Q6.2 (E), R64.1, U31.14 (VCC)
Changed lines of the file:
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@@
     (effects (font (size 1.27 1.27)) (justify left bottom))
+  )
+  (global_label "+5V" (shape input) (at 214.63 72.39 90) (fields_autoplaced)
+    (effects (font (size 1.27 1.27)) (justify left))
+    (property "Intersheet References" "${INTERSHEET_REFS}" (id 0) (at 214.5506 66.1064 90)
+      (effects (font (size 1.27 1.27)) (justify left) hide)
+    )
+  )
+  (global_label "+5V" (shape input) (at 113.03 58.42 90) (fields_autoplaced)
+    (effects (font (size 1.27 1.27)) (justify left))
+    (property "Intersheet References" "${INTERSHEET_REFS}" (id 0) (at 112.9506 52.1364 90)
+      (effects (font (size 1.27 1.27)) (justify left) hide)
+    )
   )
   (global_label "ROGER_PTT_INPUT" (shape input) (at 95.25 66.04 180) (fields_autoplaced)
@@
       (effects (font (size 1.27 1.27)) (justify left) hide)
     )
+  )
+  (global_label "+5V" (shape input) (at 140.97 106.68 90) (fields_autoplaced)
+    (effects (font (size 1.27 1.27)) (justify left))
+    (property "Intersheet References" "${INTERSHEET_REFS}" (id 0) (at 140.8906 100.3964 90)
+      (effects (font (size 1.27 1.27)) (justify left) hide)
+    )
+  )
+  (global_label "+5V" (shape input) (at 107.95 110.49 90) (fields_autoplaced)
+    (effects (font (size 1.27 1.27)) (justify left))
+    (property "Intersheet References" "${INTERSHEET_REFS}" (id 0) (at 107.8706 104.2064 90)
+      (effects (font (size 1.27 1.27)) (justify left) hide)
+    )

Commit message: connector annotated
pcb updated after manually annotating back connector sheet

all scheets reanotated in new way

all scheets reanotated in new way ...
Parts:
- renumbered C16 to C201, C17 to C202, C18 to C203, C19 to C204, C20 to C205, D19 to D201, Q5 to Q201, Q6 to Q202, Q7 to Q203, R57 to R201, R58 to R202, R59 to R203, R60 to R204, R61 to R205, R62 to R206, R63 to R207, R64 to R208, R65 to R209, R66 to R210, R67 to R211, R68 to R212, RV1 to RV201, RV2 to RV202, RV3 to RV203, U31 to U201, U32 to U202

Commit message: roger beep sligtly redesigned during assembly and debugging, bom with prices
Parts:
- removed Q201, Q202: BC858, Package_TO_SOT_SMD:SOT-23, symbol Transistor_BJT:BC858
- removed R201, R204: 5k1, Resistor_SMD:R_0805_2012Metric_Pad1.20x1.40mm_HandSolder, symbol Device:R
- removed R202, R203: R, Resistor_SMD:R_0805_2012Metric_Pad1.20x1.40mm_HandSolder, symbol Device:R
- added R?: 2k7, Resistor_SMD:R_0805_2012Metric_Pad1.20x1.40mm_HandSolder, symbol Device:R
- added R?: 6k2, Resistor_SMD:R_0805_2012Metric_Pad1.20x1.40mm_HandSolder, symbol Device:R
- C202: value 220u -> 22u; footprint Capacitor_Tantalum_SMD:CP_EIA-7343-31_Kemet-D_Pad2.25x2.55mm_HandSolder -> Capacitor_SMD:C_1206_3216Metric_Pad1.33x1.80mm_HandSolder
- R209, R210: value 10k -> 510k
- RV201: value 100k -> 20k
Connections:
- net ROGER_PTT_CNTRL_OUT: now also Q203.3 (C), R208.2, U201.13
- net ROGER_PTT_INPUT: now also U201.5
- net at C202.1, D201.2 (A), U201.1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: now also R?.1; no longer RV201.1
- net at C201.1, U201.12: now also R?.2; no longer RV202.3
- new net: R?.2, RV201.1
- new net: R?.1, RV202.3
Other:
- moved on the sheet: RV201, RV202

Commit message: changes in pcb design rerouted except chanes around roger beep genrator. new hw rev
Parts:
- gave numbers to parts that had none: 2
Changed lines of the file:
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@@
     (title "ParaCNTRL - FM repeater controller made of 74xx and analog")
     (date "2023-02-23")
-    (rev "A")
+    (rev "B")
     (company "ML Elektronika Mateusz Lubecki")
     (comment 1 "Roger Beep generator")
@@
   (symbol (lib_id "Device:R") (at 155.956 104.14 270) (unit 1)
     (in_bom yes) (on_board yes) (fields_autoplaced)
-    (property "Reference" "R?" (id 0) (at 155.956 99.4242 90))
+    (property "Reference" "R202" (id 0) (at 155.956 99.4242 90))
     (property "Value" "2k7" (id 1) (at 155.956 101.9611 90))
     (property "Footprint" "Resistor_SMD:R_0805_2012Metric_Pad1.20x1.40mm_HandSolder" (id 2) (at 155.956 102.362 90)
@@
   (symbol (lib_id "Device:R") (at 148.844 88.9 270) (unit 1)
     (in_bom yes) (on_board yes)
-    (property "Reference" "R?" (id 0) (at 148.844 86.868 90))
+    (property "Reference" "R201" (id 0) (at 148.844 86.868 90))
     (property "Value" "6k2" (id 1) (at 148.844 91.186 90))
     (property "Footprint" "Resistor_SMD:R_0805_2012Metric_Pad1.20x1.40mm_HandSolder" (id 2) (at 148.844 87.122 90)

Commit message: roger beep generator pcb design reworked
Parts:
- RV201, RV202: footprint Potentiometer_SMD:Potentiometer_Bourns_3314J_Vertical -> potentiometers:Potentiometer_SRpassives_1028F
Changed lines of the file:
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@@
     (property "Reference" "RV201" (id 0) (at 140.716 84.1842 90))
     (property "Value" "20k" (id 1) (at 140.716 86.7211 90))
-    (property "Footprint" "Potentiometer_SMD:Potentiometer_Bourns_3314J_Vertical" (id 2) (at 140.716 88.9 0)
+    (property "Footprint" "potentiometers:Potentiometer_SRpassives_1028F" (id 2) (at 140.716 88.9 0)
       (effects (font (size 1.27 1.27)) hide)
     )
@@
     (property "Reference" "RV202" (id 0) (at 165.608 99.4242 90))
     (property "Value" "10k" (id 1) (at 165.608 101.9611 90))
-    (property "Footprint" "Potentiometer_SMD:Potentiometer_Bourns_3314J_Vertical" (id 2) (at 165.608 104.14 0)
+    (property "Footprint" "potentiometers:Potentiometer_SRpassives_1028F" (id 2) (at 165.608 104.14 0)
       (effects (font (size 1.27 1.27)) hide)
     )
