File: fm-rpt-control-roger-beep.kicad_sch (KiCad schematic)
At the start: 22 parts, among them Q203 BC848, U201 HEF4093B, U202 74AHC1G32GW

Commit message: simplex remote control tone detector redesigned, gerber files for hw-rev b
Parts:
- removed C204: 10u, Capacitor_Tantalum_SMD:CP_EIA-3528-21_Kemet-B_Pad1.50x2.35mm_HandSolder, symbol Device:C_Polarized
Changed lines of the file:
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@@
   (title_block
     (title "ParaCNTRL - FM repeater controller made of 74xx and analog")
-    (date "2023-02-23")
+    (date "2023-05-07")
     (rev "B")
     (company "ML Elektronika Mateusz Lubecki")
@@
   (junction (at 149.225 42.545) (diameter 0) (color 0 0 0 0)
   )
-  (junction (at 200.66 100.33) (diameter 0) (color 0 0 0 0)
-  )
   (junction (at 135.89 83.82) (diameter 0) (color 0 0 0 0)
   )
@@
   )
   (junction (at 214.63 100.33) (diameter 0) (color 0 0 0 0)
-  )
-  (junction (at 200.66 73.66) (diameter 0) (color 0 0 0 0)
   )
   (no_connect (at 142.24 42.545))
@@
     (stroke (width 0) (type default) (color 0 0 0 0))
   )
-  (wire (pts (xy 191.77 83.82) (xy 191.77 73.66))
-    (stroke (width 0) (type default) (color 0 0 0 0))
-  )
   (wire (pts (xy 135.89 92.71) (xy 140.716 92.71))
     (stroke (width 0) (type default) (color 0 0 0 0))
@@
     (stroke (width 0) (type default) (color 0 0 0 0))
   )
-  (wire (pts (xy 191.77 100.33) (xy 200.66 100.33))
-    (stroke (width 0) (type default) (color 0 0 0 0))
-  )
   (wire (pts (xy 172.72 104.14) (xy 172.72 109.22))
-    (stroke (width 0) (type default) (color 0 0 0 0))
-  )
-  (wire (pts (xy 191.77 91.44) (xy 191.77 100.33))
-    (stroke (width 0) (type default) (color 0 0 0 0))
-  )
-  (wire (pts (xy 191.77 73.66) (xy 200.66 73.66))
     (stroke (width 0) (type default) (color 0 0 0 0))
   )
@@
       (effects (font (size 1.27 1.27)) hide)
     )
-    (pin "1")
-    (pin "2")
-  )
-  (symbol (lib_id "Device:C_Polarized") (at 191.77 87.63 0) (unit 1)
-    (in_bom yes) (on_board yes) (fields_autoplaced)
-    (property "Reference" "C204" (id 0) (at 194.691 85.9063 0)
-      (effects (font (size 1.27 1.27)) (justify left))
-    )
-    (property "Value" "10u" (id 1) (at 194.691 88.4432 0)
-      (effects (font (size 1.27 1.27)) (justify left))
-    )
-    (property "Footprint" "Capacitor_Tantalum_SMD:CP_EIA-3528-21_Kemet-B_Pad1.50x2.35mm_HandSolder" (id 2) (at 192.7352 91.44 0)
-      (effects (font (size 1.27 1.27)) hide)
-    )
-    (property "Datasheet" "~" (id 3) (at 191.77 87.63 0)
-      (effects (font (size 1.27 1.27)) hide)
-    )

Commit message: changing rogereep duration depends on simplex enable or not
Parts:
- added Q201: BC858, Package_TO_SOT_SMD:SOT-23, symbol Transistor_BJT:BC858
- added R203: 6k2, Resistor_SMD:R_0805_2012Metric_Pad1.20x1.40mm_HandSolder, symbol Device:R
Connections:
- net at R201.2, RV201.1: now also Q201.3 (C)
- net at D201.1 (K), RV201.2, RV201.3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: now also Q201.2 (E)
- new net: Q201.1 (B), R203.1
- new net ~{SPX_ENABLE_CNTRL}: R203.2
Other:
- moved on the sheet: C202, D201, R201, R208, RV201, U201A

Commit message: values of few resistors changed according to testing first unit of hw rev b
Parts:
- R201: value 6k2 -> 2k2
- R202: value 2k7 -> 4k7
- R208: value 4k7 -> 2k2
- RV201: value 20k -> 10k
Changed lines of the file:
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@@
     (in_bom yes) (on_board yes) (fields_autoplaced)
     (property "Reference" "RV201" (id 0) (at 140.716 77.8342 90))
-    (property "Value" "20k" (id 1) (at 140.716 80.3711 90))
+    (property "Value" "10k" (id 1) (at 140.716 80.3711 90))
     (property "Footprint" "potentiometers:Potentiometer_SRpassives_1028F" (id 2) (at 140.716 82.55 0)
       (effects (font (size 1.27 1.27)) hide)
@@
     (in_bom yes) (on_board yes) (fields_autoplaced)
     (property "Reference" "R202" (id 0) (at 155.956 99.4242 90))
-    (property "Value" "2k7" (id 1) (at 155.956 101.9611 90))
+    (property "Value" "4k7" (id 1) (at 155.956 101.9611 90))
     (property "Footprint" "Resistor_SMD:R_0805_2012Metric_Pad1.20x1.40mm_HandSolder" (id 2) (at 155.956 102.362 90)
       (effects (font (size 1.27 1.27)) hide)
@@
       (effects (font (size 1.27 1.27)) (justify left))
     )
-    (property "Value" "4k7" (id 1) (at 142.748 115.4942 0)
+    (property "Value" "2k2" (id 1) (at 142.748 115.4942 0)
       (effects (font (size 1.27 1.27)) (justify left))
     )
@@
     (in_bom yes) (on_board yes)
     (property "Reference" "R201" (id 0) (at 150.876 80.518 90))
-    (property "Value" "6k2" (id 1) (at 150.876 84.836 90))
+    (property "Value" "2k2" (id 1) (at 150.876 84.836 90))
     (property "Footprint" "Resistor_SMD:R_0805_2012Metric_Pad1.20x1.40mm_HandSolder" (id 2) (at 150.876 80.772 90)
       (effects (font (size 1.27 1.27)) hide)
