File: fm-rpt-control-audio-filters.kicad_sch (KiCad schematic)
At the start: 0 parts

Commit message: second daily
Parts:
- added C13, C29, C30, C31, C32: 22u, symbol Device:C
- added C14, C15, C18, C19, C20, C21, C22, C23, C28, C37: 10n, symbol Device:C
- added C16, C17, C24, C25, C26, C27, C35, C36: 100u, symbol Device:C_Polarized
- added C33: 2u2, symbol Device:C
- added C34: 10u, symbol Device:C_Polarized
- added IC8: LM567CH, sterownik:H08C, symbol sterownik_eagle_import:LM567CH
- added IC9: 74HC107D, Package_SO:SO-14_3.9x8.65mm_P1.27mm, symbol jk_flipflop:74HC107D
- added R40, R41, R42, R43, R44, R45, R46, R47: R, symbol Device:R
- added R48, R49, R50, R51, R52, R53, R58, R59: 51k, symbol Device:R
- added R54, R55, R56, R57, R60, R61, R62, R63, R64, R65, R66, R67, R68, R69, R70, R71, R74, R?: 20k, symbol Device:R
- added R72, R73: 33k, symbol Device:R
- added RV10, RV11, RV4, RV5, RV6, RV7, RV8, RV9: 10k, symbol Device:R_Potentiometer
- added U38, U39, U40: LMV358, symbol Amplifier_Operational:LMV358
- added U? (x7): 74HC04, symbol 74xx:74HC04
Connections:
- new net: IC8.8 (OUTPUT), R?.1, U?.1
- new net: IC9.9 (~{CLK}), U?.2
- new net: C14.2, R40.2, R41.1
- new net: R53.1, R57.1, R59.2
- new net: C18.1, R55.2, U38.5 (+)
- new net: C24.1, R60.2, U38.6 (-), U38.7
- new net: C29.2, R64.1
- new net: R64.2, R65.2, R72.1, U40.2 (-)
- new net: C36.1, R73.2, U40.7
- new net: R74.1, RV11.2, RV11.3
- new net: C37.1, IC8.6 (TIMCAP), R74.2
- new net: C21.2, R63.2, U39.3 (+)
- new net: C34.1, IC8.1 (OUTFILTER)
- new net: C24.2, RV8.3
- new net: C20.2, R62.2, U38.3 (+)
- new net: C23.1, R56.2, R63.1
- new net: C23.2, C27.1, U39.1, U39.2 (-)
- new net: C35.1, R72.2, U40.1
- new net: C33.2, IC8.2 (LOOPFIL)
- new net: C28.2, IC8.3 (INPUT)
- new net: IC8.5 (TIMRES), RV11.1
- new net: R68.2, R70.1, U40.3 (+)
- new net: C16.1, R48.2, R49.1, R54.1
- new net: C22.1, R54.2, R62.1
- new net: C29.1, RV7.2
- new net: C19.1, R57.2, U39.5 (+)
- new net: C15.1, C19.2, R61.1
- new net: C30.1, RV8.2
- new net: R69.2, R71.1, U40.5 (+)
- new net: R66.2, R67.2, R73.1, U40.6 (-)
- new net: C25.1, R61.2, U39.6 (-), U39.7
- new net: C25.2, RV10.3
- new net: C15.2, R42.2, R43.1
- new net: C26.2, RV7.1
- new net: C30.2, R65.1
- new net: R42.1, R46.1, RV6.2
- new net: C32.1, RV10.2
- new net: C14.1, C18.2, R60.1
- new net: C22.2, C26.1, U38.1, U38.2 (-)
- new net: R52.1, R55.1, R58.2
- new net: C27.2, RV9.1
- new net: C13.1, RV4.2
- new net: C17.1, R50.2, R51.1, R56.1
- new net: C17.2, R46.2, R47.1
- new net: C31.2, R66.1
- new net: C16.2, R44.2, R45.1
- new net: C32.2, R67.1
- new net: C31.1, RV9.2
- new net +5V: IC9.10 (~{RST}), IC9.11 (K), IC9.8 (J)
- new net +5VA: IC8.4 (V+), R?.2
- new net DPX_RX_ISOL_SW: RV5.1
- new net DPX_RX_ISOL_SW_VOL: C28.1, R40.1, R44.1, RV5.2
- new net DUPLEX_MIX: C35.2
- new net GND: C20.1, C21.1, C33.1, C34.2, C37.2, IC8.7 (GND), R41.2, R43.2, R45.2, R47.2, R49.2, R51.2, R58.1, R59.1, R68.1, R69.1, RV10.1, RV4.3, RV5.3, RV6.3, RV7.3, RV8.1, RV9.3
- new net PC_MIX: C13.2
- new net PC_RX_ISOL: RV4.1
- new net SIMPLEX_MIX: C36.2
- new net SPX_ENABLE: IC9.5 (Q)
- new net SPX_RX_ISOL_SW: RV6.1
- new net VDDA: R48.1, R50.1, R52.2, R53.2, R70.2, R71.2

Commit message: daily
Parts:
- removed C35, C36: 100u, symbol Device:C_Polarized
- added C22, C42, C48: 220u, Capacitor_Tantalum_SMD:CP_EIA-3528-21_Kemet-B_Pad1.50x2.35mm_HandSolder, symbol Device:C_Polarized
- added C45, C46: 22u, Capacitor_SMD:C_1206_3216Metric_Pad1.33x1.80mm_HandSolder, symbol Device:C
- added R107, R112, R60, R65, R90, R94: 51k, Resistor_SMD:R_0805_2012Metric_Pad1.20x1.40mm_HandSolder, symbol Device:R
- added R108, R109, R61, R62, R63, R64, R91, R92, R93: 10k, Resistor_SMD:R_0805_2012Metric_Pad1.20x1.40mm_HandSolder, symbol Device:R
- added RV14, RV7, RV8: 10k, symbol Device:R_Potentiometer
- added unit 3 of U31
- added unit 1 of U31
- added U34, U36: LMV358, symbol Amplifier_Operational:LMV358
- C21: renamed from C13; footprint (none) -> Capacitor_SMD:C_1206_3216Metric_Pad1.33x1.80mm_HandSolder
- C23: renamed from C14; footprint (none) -> Capacitor_SMD:C_0805_2012Metric_Pad1.18x1.45mm_HandSolder
- C24: renamed from C15; footprint (none) -> Capacitor_SMD:C_0805_2012Metric_Pad1.18x1.45mm_HandSolder
- C25: renamed from C16; value 100u -> 22u; footprint (none) -> Capacitor_Tantalum_SMD:CP_EIA-3528-21_Kemet-B_Pad1.50x2.35mm_HandSolder
- C26: renamed from C17; value 100u -> 22u; footprint (none) -> Capacitor_Tantalum_SMD:CP_EIA-3528-21_Kemet-B_Pad1.50x2.35mm_HandSolder
- C27: renamed from C18; footprint (none) -> Capacitor_SMD:C_0805_2012Metric_Pad1.18x1.45mm_HandSolder
- C28: renamed from C19; footprint (none) -> Capacitor_SMD:C_0805_2012Metric_Pad1.18x1.45mm_HandSolder
- C29: renamed from C20; footprint (none) -> Capacitor_SMD:C_0805_2012Metric_Pad1.18x1.45mm_HandSolder
- C30: renamed from C21; footprint (none) -> Capacitor_SMD:C_0805_2012Metric_Pad1.18x1.45mm_HandSolder
- C31: renamed from C22; footprint (none) -> Capacitor_SMD:C_0805_2012Metric_Pad1.18x1.45mm_HandSolder
- C32: renamed from C23; footprint (none) -> Capacitor_SMD:C_0805_2012Metric_Pad1.18x1.45mm_HandSolder
- C33: renamed from C24; value 100u -> 22u; footprint (none) -> Capacitor_Tantalum_SMD:CP_EIA-3528-21_Kemet-B_Pad1.50x2.35mm_HandSolder
- C34: renamed from C25; value 100u -> 22u; footprint (none) -> Capacitor_Tantalum_SMD:CP_EIA-3528-21_Kemet-B_Pad1.50x2.35mm_HandSolder
- C35: renamed from C26; value 100u -> 22u; footprint (none) -> Capacitor_Tantalum_SMD:CP_EIA-3528-21_Kemet-B_Pad1.50x2.35mm_HandSolder
- C36: renamed from C27; value 100u -> 22u; footprint (none) -> Capacitor_Tantalum_SMD:CP_EIA-3528-21_Kemet-B_Pad1.50x2.35mm_HandSolder
- C37: renamed from C28; footprint (none) -> Capacitor_SMD:C_0805_2012Metric_Pad1.18x1.45mm_HandSolder
- C38: renamed from C29; footprint (none) -> Capacitor_SMD:C_1206_3216Metric_Pad1.33x1.80mm_HandSolder
- C39: renamed from C30; footprint (none) -> Capacitor_SMD:C_1206_3216Metric_Pad1.33x1.80mm_HandSolder
- C40: renamed from C31; footprint (none) -> Capacitor_SMD:C_1206_3216Metric_Pad1.33x1.80mm_HandSolder
- C41: renamed from C32; footprint (none) -> Capacitor_SMD:C_1206_3216Metric_Pad1.33x1.80mm_HandSolder
- C43: renamed from C33; footprint (none) -> Capacitor_SMD:C_0805_2012Metric_Pad1.18x1.45mm_HandSolder
- C44: renamed from C34; footprint (none) -> Capacitor_Tantalum_SMD:CP_EIA-3528-21_Kemet-B_Pad1.50x2.35mm_HandSolder
- C47: renamed from C37; footprint (none) -> Capacitor_SMD:C_0805_2012Metric_Pad1.18x1.45mm_HandSolder
- R100: renamed from R69; footprint (none) -> Resistor_SMD:R_0805_2012Metric_Pad1.20x1.40mm_HandSolder
- R101: renamed from R70; footprint (none) -> Resistor_SMD:R_0805_2012Metric_Pad1.20x1.40mm_HandSolder
- R102: renamed from R71; footprint (none) -> Resistor_SMD:R_0805_2012Metric_Pad1.20x1.40mm_HandSolder
- R103: renamed from R72; footprint (none) -> Resistor_SMD:R_0805_2012Metric_Pad1.20x1.40mm_HandSolder
- R104: renamed from R73; footprint (none) -> Resistor_SMD:R_0805_2012Metric_Pad1.20x1.40mm_HandSolder
- R105: renamed from R?; footprint (none) -> Resistor_SMD:R_0805_2012Metric_Pad1.20x1.40mm_HandSolder
- R106: renamed from R74; footprint (none) -> Resistor_SMD:R_0805_2012Metric_Pad1.20x1.40mm_HandSolder
- R66: renamed from R40; footprint (none) -> Resistor_SMD:R_0805_2012Metric_Pad1.20x1.40mm_HandSolder
- R67: renamed from R41; footprint (none) -> Resistor_SMD:R_0805_2012Metric_Pad1.20x1.40mm_HandSolder
- R68: renamed from R42; footprint (none) -> Resistor_SMD:R_0805_2012Metric_Pad1.20x1.40mm_HandSolder
- R69: renamed from R43; footprint (none) -> Resistor_SMD:R_0805_2012Metric_Pad1.20x1.40mm_HandSolder
- R70: renamed from R44; footprint (none) -> Resistor_SMD:R_0805_2012Metric_Pad1.20x1.40mm_HandSolder
- R71: renamed from R45; footprint (none) -> Resistor_SMD:R_0805_2012Metric_Pad1.20x1.40mm_HandSolder
- R72: renamed from R46; footprint (none) -> Resistor_SMD:R_0805_2012Metric_Pad1.20x1.40mm_HandSolder
- R73: renamed from R47; footprint (none) -> Resistor_SMD:R_0805_2012Metric_Pad1.20x1.40mm_HandSolder
- R74: renamed from R48; footprint (none) -> Resistor_SMD:R_0805_2012Metric_Pad1.20x1.40mm_HandSolder
- R75: renamed from R49; footprint (none) -> Resistor_SMD:R_0805_2012Metric_Pad1.20x1.40mm_HandSolder
- R76: renamed from R50; footprint (none) -> Resistor_SMD:R_0805_2012Metric_Pad1.20x1.40mm_HandSolder
- R77: renamed from R51; footprint (none) -> Resistor_SMD:R_0805_2012Metric_Pad1.20x1.40mm_HandSolder
- R78: renamed from R52; footprint (none) -> Resistor_SMD:R_0805_2012Metric_Pad1.20x1.40mm_HandSolder
- R79: renamed from R53; footprint (none) -> Resistor_SMD:R_0805_2012Metric_Pad1.20x1.40mm_HandSolder
- R80: renamed from R54; footprint (none) -> Resistor_SMD:R_0805_2012Metric_Pad1.20x1.40mm_HandSolder
- R81: renamed from R55; footprint (none) -> Resistor_SMD:R_0805_2012Metric_Pad1.20x1.40mm_HandSolder
- R82: renamed from R56; footprint (none) -> Resistor_SMD:R_0805_2012Metric_Pad1.20x1.40mm_HandSolder
- R83: renamed from R57; footprint (none) -> Resistor_SMD:R_0805_2012Metric_Pad1.20x1.40mm_HandSolder
- R84: renamed from R58; footprint (none) -> Resistor_SMD:R_0805_2012Metric_Pad1.20x1.40mm_HandSolder
- R85: renamed from R59; footprint (none) -> Resistor_SMD:R_0805_2012Metric_Pad1.20x1.40mm_HandSolder
- R86: renamed from R60; footprint (none) -> Resistor_SMD:R_0805_2012Metric_Pad1.20x1.40mm_HandSolder
- R87: renamed from R61; footprint (none) -> Resistor_SMD:R_0805_2012Metric_Pad1.20x1.40mm_HandSolder
- R88: renamed from R62; footprint (none) -> Resistor_SMD:R_0805_2012Metric_Pad1.20x1.40mm_HandSolder
- R89: renamed from R63; footprint (none) -> Resistor_SMD:R_0805_2012Metric_Pad1.20x1.40mm_HandSolder
- R95: renamed from R64; footprint (none) -> Resistor_SMD:R_0805_2012Metric_Pad1.20x1.40mm_HandSolder
- R96: renamed from R65; footprint (none) -> Resistor_SMD:R_0805_2012Metric_Pad1.20x1.40mm_HandSolder
- R97: renamed from R66; footprint (none) -> Resistor_SMD:R_0805_2012Metric_Pad1.20x1.40mm_HandSolder
- R98: renamed from R67; footprint (none) -> Resistor_SMD:R_0805_2012Metric_Pad1.20x1.40mm_HandSolder
- R99: renamed from R68; footprint (none) -> Resistor_SMD:R_0805_2012Metric_Pad1.20x1.40mm_HandSolder
- U37: renamed from U?; footprint (none) -> Package_SO:SOIC-14_3.9x8.7mm_P1.27mm
- renumbered IC8 to IC6, IC9 to IC7, RV8 to RV10, RV9 to RV11, RV10 to RV12, RV11 to RV13, RV7 to RV9, U38 to U31, U39 to U32, U38 to U33, U40 to U35
Connections:
- net +5V: now also IC7.14 (VCC)
- net DPX_TX_ISOL: now also C22.2
- net DUPLEX_MIX: now also C45.2, R109.1, R62.1, R91.1
- net GND: now also IC7.7 (GND), U32.4 (V-), U33.4 (V-), U35.4 (V-), R112.2, R65.2, R94.2
- net PC_MIX: now also R63.1, R92.1
- net PC_TX_ISOL: now also C48.2
- net SIMPLEX_MIX: now also C46.2, R108.1, R61.1
- net SPX_TX_ISOL: now also C42.2
- net VDDA: now also U32.8 (V+), U33.8 (V+), U35.8 (V+), R107.1, R60.1, R90.1, U31.8 (V+)
- net at R104.2, U35.7: now also C46.1
- net at R103.2, U35.1: now also C45.1
- new net: C22.1, RV7.2, RV7.3, U31.1
- new net: R61.2, R62.2, R63.2, R64.2, RV7.1, U31.2 (-)
- new net: C48.1, RV14.2, RV14.3, U36.1
- new net: R60.2, R65.1, U31.3 (+)
- new net: R91.2, R92.2, R93.2, RV8.1, U34.2 (-)
- new net: C42.1, RV8.2, RV8.3, U34.1
- new net: R108.2, R109.2, RV14.1, U36.2 (-)
- new net: R107.2, R112.1, U36.3 (+)
- new net: R90.2, R94.1, U34.3 (+)
- new net ROGER_AUDIO: R64.1, R93.1
Other:
- moved on the sheet: U37B, U37C, U37D, U37E, U37F, U37G

Commit message: schematic design ready
Parts:
- removed unit 6 of U37
- removed unit 3 of U37
- removed unit 4 of U37
- removed unit 2 of U37
- removed unit 5 of U37
- added R? (x3): 10k, Resistor_SMD:R_0805_2012Metric_Pad1.20x1.40mm_HandSolder, symbol Device:R
- RV10, RV11, RV12, RV13, RV4, RV5, RV6, RV9: footprint (none) -> Potentiometer_SMD:Potentiometer_Bourns_3314J_Vertical
- RV14, RV7, RV8: footprint (none) -> Potentiometer_THT:Potentiometer_Alps_RK163_Single_Horizontal
- U31, U32, U33, U34, U35, U36: footprint (none) -> Package_SO:SOIC-8_3.9x4.9mm_P1.27mm
Connections:
- net +5V: now also U37.14 (VCC)
- net DPX_TX_ISOL: now also RV7.2; no longer C22.2
- net GND: now also RV14.3, RV7.3, RV8.3, U37.7 (GND)
- net PC_TX_ISOL: now also RV14.2; no longer C48.2
- net SPX_TX_ISOL: now also RV8.2; no longer C42.2
- net at C22.1, U31.1: now also R?.2; no longer RV7.2, RV7.3
- net at R61.2, R62.2, R63.2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: now also R?.1; no longer RV7.1
- net at C48.1, U36.1: now also R?.2; no longer RV14.2, RV14.3
- net at R91.2, R92.2, R93.2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: now also R?.1; no longer RV8.1
- net at C42.1, U34.1: now also R?.2; no longer RV8.2, RV8.3
- net at R108.2, R109.2, U36.2 (-): now also R?.1; no longer RV14.1
- new net: C22.2, RV7.1
- new net: C48.2, RV14.1
- new net: C42.2, RV8.1
Other:
- moved on the sheet: RV14, RV7, RV8, U37G

Commit message: PCB dimenstions set and db/din sockets, pots, switches and leds placed
Parts:
- IC5: renamed from IC6; footprint sterownik:H08C -> Package_SO:SOIC-8_3.9x4.9mm_P1.27mm
- gave numbers to parts that had none: 3
- renumbered RV10 to DPX_HI1, RV9 to DPX_LO1, RV5 to DPX_VOL_1, IC7 to IC6, RV7 to MASTER_AUD_DPX_1, RV14 to MASTER_AUD_PC_1, RV8 to MASTER_AUD_SPX_1, RV4 to PC_VOL_1, R94 to R100, R95 to R102, R96 to R103, R97 to R104, R98 to R105, R99 to R106, R100 to R107, R101 to R108, R102 to R109, R103 to R110, R104 to R111, R105 to R112, R106 to R113, R107 to R114, R108 to R115, R109 to R116, R112 to R117, R60 to R65, R61 to R66, R62 to R67, R63 to R68, R64 to R69, R65 to R70, R66 to R72, R67 to R73, R68 to R74, R69 to R75, R70 to R76, R71 to R77, R72 to R78, R73 to R79, R74 to R80, R75 to R81, R76 to R82, R77 to R83, R78 to R84, R79 to R85, R80 to R86, R81 to R87, R82 to R88, R83 to R89, R84 to R90, R85 to R91, R86 to R92, R87 to R93, R88 to R94, R89 to R95, R90 to R96, R91 to R97, R92 to R98, R93 to R99, RV13 to RV4, RV12 to SPX_HI1, RV11 to SPX_LO1, RV6 to SPX_VOL_1, U31 to U32, U32 to U33, U33 to U34, U34 to U35, U35 to U36, U36 to U37, U37 to U38
Other:
- title: (none) -> ParaCNTRL - FM repeater controller made of 74xx and analog
- moved on the sheet: MASTER_AUD_DPX_1, MASTER_AUD_SPX_1

Commit message: controlling to_pc_retransmission line
Parts:
- renumbered IC5 to IC4, IC6 to IC5, MASTER_AUD_DPX_1 to MAIN_OUT_VOL_DPX_1, MASTER_AUD_PC_1 to MAIN_OUT_VOL_PC_1, MASTER_AUD_SPX_1 to MAIN_OUT_VOL_SPX_1, U32 to U33, U33 to U34, U34 to U35, U35 to U36, U36 to U37, U37 to U38, U38 to U39

Commit message: logic ics, relays and relay driving electronics, voltage regulators placed
Parts:
- DPX_HI1, DPX_LO1, DPX_VOL_1, PC_VOL_1, SPX_HI1, SPX_LO1, SPX_VOL_1: footprint Potentiometer_SMD:Potentiometer_Bourns_3314J_Vertical -> potentiometers:Potentiometer_SRpassives_1028F
- renumbered R96 to R100, R97 to R101, R98 to R102, R99 to R103, R100 to R104, R101 to R105, R102 to R106, R103 to R107, R104 to R108, R105 to R109, R106 to R110, R107 to R111, R108 to R112, R109 to R113, R110 to R114, R111 to R115, R112 to R116, R113 to R117, R114 to R118, R115 to R119, R116 to R120, R117 to R121, R118 to R122, R65 to R69, R66 to R70, R67 to R71, R68 to R72, R69 to R73, R70 to R74, R71 to R75, R72 to R76, R73 to R77, R74 to R78, R75 to R79, R76 to R80, R77 to R81, R78 to R82, R79 to R83, R80 to R84, R81 to R85, R82 to R86, R83 to R87, R84 to R88, R85 to R89, R86 to R90, R87 to R91, R88 to R92, R89 to R93, R90 to R94, R91 to R95, R92 to R96, R93 to R97, R94 to R98, R95 to R99
Connections:
- net TONE_DET: now reaches IC4.8 (OUTPUT), R116.1, U39.1
- net ROGER_AUDIO renamed ROGER_AUDIO_SW

Commit message: before replacing some pinheaders with switches
Parts:
- removed U35: LMV358, Package_SO:SOIC-8_3.9x4.9mm_P1.27mm, symbol Amplifier_Operational:LMV358
- added unit 1 of U33
- added unit 3 of U36
- renumbered U33 to U36
Connections:
- net GND: now also U33.4 (V-), U38.4 (V-), U36.4 (V-)
- net VDDA: now also U38.8 (V+), U36.8 (V+)
- net at C29.2, R98.2: now also U33.3 (+)
- net at R101.2, R102.2, R103.2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: now also U36.6 (-); no longer U36.2 (-)
- net at R100.2, R104.1: now also U36.5 (+); no longer U36.3 (+)
- net at C31.2, C35.1: now also U33.1, U33.2 (-)
- net at C42.1, R105.2: now also U36.7; no longer U36.1
