File: fm-rpt-control-audio-filters.kicad_sch (KiCad schematic)
At the start: 101 parts, among them IC4 LM567CH, IC5 74HC107D, U33 LMV358, U34 LMV358, U36 LMV358, U37 LMV358, U38 LMV358, U39 74HC04

Commit message: short
Connections:
- net +5V: now also IC4.4 (V+)
- net +5VA: no longer IC4.4 (V+)
Changed lines of the file:
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@@
+    (stroke (width 0) (type default) (color 0 0 0 0))
+  )
+  (wire (pts (xy 176.53 94.615) (xy 179.705 94.615))
+    (stroke (width 0) (type default) (color 0 0 0 0))
+  )
+  (wire (pts (xy 176.53 92.71) (xy 176.53 94.615))
     (stroke (width 0) (type default) (color 0 0 0 0))
   )
@@
     (pin "2")
   )
-  (symbol (lib_id "power:+5VA") (at 176.53 92.71 180) (unit 1)
-    (in_bom yes) (on_board yes)
-    (property "Reference" "#PWR064" (id 0) (at 176.53 88.9 0)
-      (effects (font (size 1.27 1.27)) hide)
-    )
-    (property "Value" "+5VA" (id 1) (at 176.53 96.52 0))
-    (property "Footprint" "" (id 2) (at 176.53 92.71 0)
-      (effects (font (size 1.27 1.27)) hide)
-    )
-    (property "Datasheet" "" (id 3) (at 176.53 92.71 0)
-      (effects (font (size 1.27 1.27)) hide)
-    )
-    (pin "1")
-  )
   (symbol (lib_id "paratnc_cp_import:GND") (at 62.23 118.11 0) (unit 1)
     (in_bom yes) (on_board yes) (fields_autoplaced)
@@
     (pin "7")
   )
+  (symbol (lib_id "power:+5V") (at 179.705 94.615 270) (mirror x) (unit 1)
+    (in_bom yes) (on_board yes)
+    (property "Reference" "#PWR?" (id 0) (at 175.895 94.615 0)
+      (effects (font (size 1.27 1.27)) hide)
+    )
+    (property "Value" "+5V" (id 1) (at 186.055 94.615 90)
+      (effects (font (size 1.27 1.27)) (justify right))
+    )
+    (property "Footprint" "" (id 2) (at 179.705 94.615 0)
+      (effects (font (size 1.27 1.27)) hide)
+    )
+    (property "Datasheet" "" (id 3) (at 179.705 94.615 0)
+      (effects (font (size 1.27 1.27)) hide)
+    )
+    (pin "1")
+  )
   (symbol (lib_id "power:+5V") (at 224.79 73.66 90) (mirror x) (unit 1)

Commit message: +5v bus removed completely
Connections:
- removed net +5V: IC4.4 (V+), IC5.10 (~{RST}), IC5.11 (K), IC5.14 (VCC), IC5.8 (J), U39.14 (VCC)
Changed lines of the file:
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@@
-    (pin "1")
-  )
-  (symbol (lib_id "power:+5V") (at 260.35 76.2 0) (mirror y) (unit 1)
-    (in_bom yes) (on_board yes)
-    (property "Reference" "#PWR075" (id 0) (at 260.35 80.01 0)
-      (effects (font (size 1.27 1.27)) hide)
-    )
-    (property "Value" "+5V" (id 1) (at 260.35 69.85 90)
-      (effects (font (size 1.27 1.27)) (justify right))
-    )
-    (property "Footprint" "" (id 2) (at 260.35 76.2 0)
-      (effects (font (size 1.27 1.27)) hide)
-    )
-    (property "Datasheet" "" (id 3) (at 260.35 76.2 0)
-      (effects (font (size 1.27 1.27)) hide)
-    )
     (pin "1")
   )
@@
     (pin "2")
   )
-  (symbol (lib_id "power:+5V") (at 232.41 25.4 0) (mirror y) (unit 1)
-    (in_bom yes) (on_board yes)
-    (property "Reference" "#PWR072" (id 0) (at 232.41 29.21 0)
-      (effects (font (size 1.27 1.27)) hide)
-    )
-    (property "Value" "+5V" (id 1) (at 232.41 19.05 90)
-      (effects (font (size 1.27 1.27)) (justify right))
-    )
-    (property "Footprint" "" (id 2) (at 232.41 25.4 0)
-      (effects (font (size 1.27 1.27)) hide)
-    )
-    (property "Datasheet" "" (id 3) (at 232.41 25.4 0)
-      (effects (font (size 1.27 1.27)) hide)
-    )
-    (pin "1")
-  )
   (symbol (lib_id "Device:C_Polarized") (at 129.54 107.95 90) (unit 1)
     (in_bom yes) (on_board yes) (fields_autoplaced)
@@
     (pin "1")
   )
-  (symbol (lib_id "power:+5V") (at 224.79 60.96 90) (mirror x) (unit 1)
-    (in_bom yes) (on_board yes)
-    (property "Reference" "#PWR069" (id 0) (at 228.6 60.96 0)
-      (effects (font (size 1.27 1.27)) hide)
-    )
-    (property "Value" "+5V" (id 1) (at 218.44 60.96 90)
-      (effects (font (size 1.27 1.27)) (justify right))
-    )
-    (property "Footprint" "" (id 2) (at 224.79 60.96 0)
-      (effects (font (size 1.27 1.27)) hide)
-    )
-    (property "Datasheet" "" (id 3) (at 224.79 60.96 0)
-      (effects (font (size 1.27 1.27)) hide)
-    )
-    (pin "1")
-  )
   (symbol (lib_id "Device:C") (at 201.93 74.93 90) (unit 1)
     (in_bom yes) (on_board yes) (fields_autoplaced)
@@
     (pin "7")
   )
-  (symbol (lib_id "power:+5V") (at 179.705 94.615 270) (mirror x) (unit 1)
-    (in_bom yes) (on_board yes)
-    (property "Reference" "#PWR?" (id 0) (at 175.895 94.615 0)
-      (effects (font (size 1.27 1.27)) hide)
-    )
-    (property "Value" "+5V" (id 1) (at 186.055 94.615 90)
-      (effects (font (size 1.27 1.27)) (justify right))
-    )
-    (property "Footprint" "" (id 2) (at 179.705 94.615 0)
-      (effects (font (size 1.27 1.27)) hide)
-    )
-    (property "Datasheet" "" (id 3) (at 179.705 94.615 0)
-      (effects (font (size 1.27 1.27)) hide)
-    )
-    (pin "1")
-  )
-  (symbol (lib_id "power:+5V") (at 224.79 73.66 90) (mirror x) (unit 1)
-    (in_bom yes) (on_board yes)
-    (property "Reference" "#PWR071" (id 0) (at 228.6 73.66 0)
-      (effects (font (size 1.27 1.27)) hide)
-    )
-    (property "Value" "+5V" (id 1) (at 218.44 73.66 90)
-      (effects (font (size 1.27 1.27)) (justify right))
-    )
-    (property "Footprint" "" (id 2) (at 224.79 73.66 0)
-      (effects (font (size 1.27 1.27)) hide)
-    )
-    (property "Datasheet" "" (id 3) (at 224.79 73.66 0)
-      (effects (font (size 1.27 1.27)) hide)
-    )
-    (pin "1")
-  )
   (symbol (lib_id "paratnc_cp_import:GND") (at 130.81 54.61 270) (unit 1)
     (in_bom yes) (on_board yes) (fields_autoplaced)
@@
       (effects (font (size 1.27 1.27)) hide)
     )
-    (pin "1")
-  )
-  (symbol (lib_id "power:+5V") (at 224.79 71.12 90) (mirror x) (unit 1)
-    (in_bom yes) (on_board yes)
-    (property "Reference" "#PWR070" (id 0) (at 228.6 71.12 0)
-      (effects (font (size 1.27 1.27)) hide)
-    )
-    (property "Value" "+5V" (id 1) (at 218.44 71.12 90)
-      (effects (font (size 1.27 1.27)) (justify right))
-    )
-    (property "Footprint" "" (id 2) (at 224.79 71.12 0)
-      (effects (font (size 1.27 1.27)) hide)
-    )
-    (property "Datasheet" "" (id 3) (at 224.79 71.12 0)
-      (effects (font (size 1.27 1.27)) hide)
-    )

Commit message: short fixed
Connections:
- net +5VA is gone; now on net +5V: R116.2
- net DUPLEX_MIX: no longer R71.1
- net +5V: now reaches IC4.4 (V+)
- net +5V: now also IC5.10 (~{RST}), IC5.11 (K), IC5.14 (VCC), IC5.8 (J), U39.14 (VCC)
- new net DUPLEX_MIX_SW: R71.1
Changed lines of the file:
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@@
     (stroke (width 0) (type default) (color 0 0 0 0))
   )
-  (wire (pts (xy 232.41 25.4) (xy 232.41 26.67))
+  (wire (pts (xy 232.41 24.13) (xy 232.41 26.67))
     (stroke (width 0) (type default) (color 0 0 0 0))
   )
@@
   (label "TONE_DET" (at 195.58 67.31 0)
     (effects (font (size 1.27 1.27)) (justify left bottom))
+  )
+  (global_label "+5V" (shape input) (at 224.79 71.12 180) (fields_autoplaced)
+    (effects (font (size 1.27 1.27)) (justify right))
+    (property "Intersheet References" "${INTERSHEET_REFS}" (id 0) (at 218.5064 71.1994 0)
+      (effects (font (size 1.27 1.27)) (justify right) hide)
+    )
+  )
+  (global_label "+5V" (shape input) (at 224.79 73.66 180) (fields_autoplaced)
+    (effects (font (size 1.27 1.27)) (justify right))
+    (property "Intersheet References" "${INTERSHEET_REFS}" (id 0) (at 218.5064 73.7394 0)
+      (effects (font (size 1.27 1.27)) (justify right) hide)
+    )
   )
   (global_label "SPX_RX_ISOL_SW" (shape input) (at 33.02 86.36 180) (fields_autoplaced)
@@
     )
   )
+  (global_label "+5V" (shape input) (at 232.41 24.13 90) (fields_autoplaced)
+    (effects (font (size 1.27 1.27)) (justify left))
+    (property "Intersheet References" "${INTERSHEET_REFS}" (id 0) (at 232.3306 17.8464 90)
+      (effects (font (size 1.27 1.27)) (justify left) hide)
+    )
+  )
   (global_label "SPX_TX_ISOL" (shape input) (at 160.02 172.72 0) (fields_autoplaced)
     (effects (font (size 1.27 1.27)) (justify left))
@@
     )
   )
-  (global_label "DUPLEX_MIX" (shape input) (at 31.75 171.45 180) (fields_autoplaced)
+  (global_label "DUPLEX_MIX_SW" (shape input) (at 31.75 171.45 180) (fields_autoplaced)
     (effects (font (size 1.27 1.27)) (justify right))
-    (property "Intersheet References" "${INTERSHEET_REFS}" (id 0) (at 17.8464 171.5294 0)
+    (property "Intersheet References" "${INTERSHEET_REFS}" (id 0) (at 14.2179 171.3706 0)
       (effects (font (size 1.27 1.27)) (justify right) hide)
     )
@@
     )
   )
+  (global_label "+5V" (shape input) (at 260.35 76.2 90) (fields_autoplaced)
+    (effects (font (size 1.27 1.27)) (justify left))
+    (property "Intersheet References" "${INTERSHEET_REFS}" (id 0) (at 260.2706 69.9164 90)
+      (effects (font (size 1.27 1.27)) (justify left) hide)
+    )
+  )
   (global_label "PC_RX_ISOL" (shape input) (at 27.94 59.69 180) (fields_autoplaced)
     (effects (font (size 1.27 1.27)) (justify right))
@@
     )
   )
+  (global_label "+5V" (shape input) (at 179.705 94.615 0) (fields_autoplaced)
+    (effects (font (size 1.27 1.27)) (justify left))
+    (property "Intersheet References" "${INTERSHEET_REFS}" (id 0) (at 185.9886 94.5356 0)
+      (effects (font (size 1.27 1.27)) (justify left) hide)
+    )
+  )
   (global_label "ROGER_AUDIO_SW" (shape input) (at 31.75 186.69 180) (fields_autoplaced)
     (effects (font (size 1.27 1.27)) (justify right))
@@
     )
   )
+  (global_label "+5V" (shape input) (at 224.79 60.96 180) (fields_autoplaced)
+    (effects (font (size 1.27 1.27)) (justify right))
+    (property "Intersheet References" "${INTERSHEET_REFS}" (id 0) (at 218.5064 61.0394 0)
+      (effects (font (size 1.27 1.27)) (justify right) hide)
+    )
+  )
   (global_label "DPX_RX_ISOL_SW_VOL" (shape input) (at 134.62 82.55 180) (fields_autoplaced)
     (effects (font (size 1.27 1.27)) (justify right))
     (property "Intersheet References" "${INTERSHEET_REFS}" (id 0) (at 111.8264 82.6294 0)
       (effects (font (size 1.27 1.27)) (justify right) hide)
+    )
+  )
+  (global_label "+5V" (shape input) (at 194.31 57.15 90) (fields_autoplaced)
+    (effects (font (size 1.27 1.27)) (justify left))
+    (property "Intersheet References" "${INTERSHEET_REFS}" (id 0) (at 194.2306 50.8664 90)
+      (effects (font (size 1.27 1.27)) (justify left) hide)
     )
   )
@@
     (pin "7")
   )
-  (symbol (lib_id "power:+5VA") (at 194.31 57.15 0) (unit 1)
-    (in_bom yes) (on_board yes)
-    (property "Reference" "#PWR066" (id 0) (at 194.31 60.96 0)
-      (effects (font (size 1.27 1.27)) hide)
-    )
-    (property "Value" "+5VA" (id 1) (at 194.31 53.34 0))
-    (property "Footprint" "" (id 2) (at 194.31 57.15 0)
-      (effects (font (size 1.27 1.27)) hide)
-    )
-    (property "Datasheet" "" (id 3) (at 194.31 57.15 0)
-      (effects (font (size 1.27 1.27)) hide)
-    )
-    (pin "1")
-  )
   (symbol (lib_id "Device:R_Potentiometer") (at 34.29 64.77 0) (unit 1)

Commit message: all components placed on pcb
Parts:
- added J3: AudioJack3, Connector_Audio:Jack_3.5mm_Lumberg_1503_07_Horizontal, symbol Connector:AudioJack3
Connections:
- net TONE_DET: now also U39.5; no longer U39.1
- net at IC5.9 (~{CLK}): now also U39.6; no longer U39.2
Changed lines of the file:
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@@
     )
   )
-  (symbol (lib_id "74xx:74HC04") (at 213.36 67.31 0) (unit 1)
+  (symbol (lib_id "74xx:74HC04") (at 213.36 67.31 0) (unit 3)
     (in_bom yes) (on_board yes) (fields_autoplaced)
     (property "Reference" "U39" (id 0) (at 213.36 59.8002 0))
@@
       (effects (font (size 1.27 1.27)) hide)
     )
-    (pin "1")
-    (pin "2")
+    (pin "5")
+    (pin "6")
   )
   (symbol (lib_id "paratnc_cp_import:GND") (at 99.06 49.53 0) (unit 1)
@@
     (pin "1")
   )
+  (symbol (lib_id "Connector:AudioJack3") (at 179.07 147.32 0) (unit 1)
+    (in_bom yes) (on_board yes) (fields_autoplaced)
+    (property "Reference" "J3" (id 0) (at 177.165 139.8102 0))
+    (property "Value" "AudioJack3" (id 1) (at 177.165 142.3471 0))
+    (property "Footprint" "Connector_Audio:Jack_3.5mm_Lumberg_1503_07_Horizontal" (id 2) (at 179.07 147.32 0)
+      (effects (font (size 1.27 1.27)) hide)
+    )
+    (property "Datasheet" "~" (id 3) (at 179.07 147.32 0)
+      (effects (font (size 1.27 1.27)) hide)
+    )
+    (pin "R")
+    (pin "S")
+    (pin "T")
+  )
   (symbol (lib_id "Device:C_Polarized") (at 62.23 161.29 90) (unit 1)

Commit message: daily
Connections:
- net DPX_TX_ISOL renamed DUPLEX_MASTER_AUD
- net PC_TX_ISOL renamed PC_MASTER_AUD
- net SPX_TX_ISOL renamed SIMPLEX_MASTER_AUD
Changed lines of the file:
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@@
     )
   )
-  (global_label "SPX_TX_ISOL" (shape input) (at 160.02 172.72 0) (fields_autoplaced)
+  (global_label "SIMPLEX_MASTER_AUD" (shape input) (at 160.02 172.72 0) (fields_autoplaced)
     (effects (font (size 1.27 1.27)) (justify left))
-    (property "Intersheet References" "${INTERSHEET_REFS}" (id 0) (at 174.4074 172.6406 0)
+    (property "Intersheet References" "${INTERSHEET_REFS}" (id 0) (at 183.116 172.6406 0)
       (effects (font (size 1.27 1.27)) (justify left) hide)
     )
@@
     )
   )
-  (global_label "DPX_TX_ISOL" (shape input) (at 74.93 166.37 0) (fields_autoplaced)
+  (global_label "DUPLEX_MASTER_AUD" (shape input) (at 74.93 166.37 0) (fields_autoplaced)
     (effects (font (size 1.27 1.27)) (justify left))
-    (property "Intersheet References" "${INTERSHEET_REFS}" (id 0) (at 89.3779 166.4494 0)
+    (property "Intersheet References" "${INTERSHEET_REFS}" (id 0) (at 97.3607 166.2906 0)
       (effects (font (size 1.27 1.27)) (justify left) hide)
     )
@@
     )
   )
-  (global_label "PC_TX_ISOL" (shape input) (at 261.62 137.16 0) (fields_autoplaced)
+  (global_label "PC_MASTER_AUD" (shape input) (at 261.62 137.16 0) (fields_autoplaced)
     (effects (font (size 1.27 1.27)) (justify left))
-    (property "Intersheet References" "${INTERSHEET_REFS}" (id 0) (at 274.8583 137.0806 0)
+    (property "Intersheet References" "${INTERSHEET_REFS}" (id 0) (at 279.3336 137.0806 0)
       (effects (font (size 1.27 1.27)) (justify left) hide)
     )

Commit message: connector annotated
pcb updated after manually annotating back connector sheet

all scheets reanotated in new way

all scheets reanotated in new way ...
Parts:
- renumbered C21 to C301, C22 to C302, C23 to C303, C24 to C304, C25 to C305, C26 to C306, C27 to C307, C28 to C308, C29 to C309, C30 to C310, C31 to C311, C32 to C312, C33 to C313, C34 to C314, C35 to C315, C36 to C316, C37 to C317, C38 to C318, C39 to C319, C40 to C320, C41 to C321, C42 to C322, C43 to C323, C44 to C324, C45 to C325, C46 to C326, C47 to C327, C48 to C328, DPX_HI1 to DPX_HI3, DPX_LO1 to DPX_LO3, DPX_VOL_1 to DPX_VOL_3, IC4 to IC301, IC5 to IC302, J3 to J301, MAIN_OUT_VOL_DPX_1 to MAIN_OUT_VOL_DPX_3, MAIN_OUT_VOL_PC_1 to MAIN_OUT_VOL_PC_3, MAIN_OUT_VOL_SPX_1 to MAIN_OUT_VOL_SPX_3, PC_VOL_1 to PC_VOL_3, R69 to R301, R70 to R302, R71 to R303, R72 to R304, R73 to R305, R74 to R306, R75 to R307, R76 to R308, R77 to R309, R78 to R310, R79 to R311, R80 to R312, R81 to R313, R82 to R314, R83 to R315, R84 to R316, R85 to R317, R86 to R318, R87 to R319, R88 to R320, R89 to R321, R90 to R322, R91 to R323, R92 to R324, R93 to R325, R94 to R326, R95 to R327, R96 to R328, R97 to R329, R98 to R330, R99 to R331, R100 to R332, R101 to R333, R102 to R334, R103 to R335, R104 to R336, R105 to R337, R106 to R338, R107 to R339, R108 to R340, R109 to R341, R110 to R342, R111 to R343, R112 to R344, R113 to R345, R114 to R346, R115 to R347, R116 to R348, R117 to R349, R118 to R350, R119 to R351, R120 to R352, R121 to R353, R122 to R354, RV4 to RV301, SPX_HI1 to SPX_HI3, SPX_LO1 to SPX_LO3, SPX_VOL_1 to SPX_VOL_3, U36 to U301, U33 to U302, U34 to U303, U37 to U304, U38 to U305, U39 to U306
