File: fm-rpt-control-audio-filters.kicad_sch (KiCad schematic)
At the start: 102 parts, among them IC301 LM567CH, IC302 74HC107D, J301 AudioJack3, U301 LMV358, U302 LMV358, U303 LMV358, U304 LMV358, U305 LMV358, U306 74HC04

Commit message: simplex remote control tone detector redesigned, gerber files for hw-rev b
Parts:
- removed C317, C327: 10n, Capacitor_SMD:C_0805_2012Metric_Pad1.18x1.45mm_HandSolder, symbol Device:C
- removed C323: 2u2, Capacitor_SMD:C_0805_2012Metric_Pad1.18x1.45mm_HandSolder, symbol Device:C
- removed C324: 10u, Capacitor_Tantalum_SMD:CP_EIA-3528-21_Kemet-B_Pad1.50x2.35mm_HandSolder, symbol Device:C_Polarized
- removed IC301: LM567CH, Package_SO:SOIC-8_3.9x4.9mm_P1.27mm, symbol sterownik_eagle_import:LM567CH
- removed IC302: 74HC107D, Package_SO:SO-14_3.9x8.65mm_P1.27mm, symbol jk_flipflop:74HC107D
- removed R348, R349: 20k, Resistor_SMD:R_0805_2012Metric_Pad1.20x1.40mm_HandSolder, symbol Device:R
- removed RV301: 10k, Potentiometer_SMD:Potentiometer_Bourns_3314J_Vertical, symbol Device:R_Potentiometer
- removed U306: 74HC04, Package_SO:SOIC-14_3.9x8.7mm_P1.27mm, symbol 74xx:74HC04
Other:
- moved on the sheet: R345

Commit message: values of few resistors changed according to testing first unit of hw rev b
Parts:
- R307, R337, R354: value 10k -> 51k
- R308, R310, R312, R314: value R -> 2k2
- R309, R311, R313, R315: value R -> 20k
- R346, R347: value 33k -> 51k
Changed lines of the file:
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@@
       (effects (font (size 1.27 1.27)) (justify left))
     )
-    (property "Value" "R" (id 1) (at 52.578 32.1822 0)
+    (property "Value" "2k2" (id 1) (at 52.578 32.1822 0)
       (effects (font (size 1.27 1.27)) (justify left))
     )
@@
       (effects (font (size 1.27 1.27)) (justify left))
     )
-    (property "Value" "R" (id 1) (at 52.578 42.3422 0)
+    (property "Value" "20k" (id 1) (at 52.578 42.3422 0)
       (effects (font (size 1.27 1.27)) (justify left))
     )
@@
     (in_bom yes) (on_board yes) (fields_autoplaced)
     (property "Reference" "R354" (id 0) (at 233.68 137.5242 90))
-    (property "Value" "10k" (id 1) (at 233.68 140.0611 90))
+    (property "Value" "51k" (id 1) (at 233.68 140.0611 90))
     (property "Footprint" "Resistor_SMD:R_0805_2012Metric_Pad1.20x1.40mm_HandSolder" (id 2) (at 233.68 144.018 90)
       (effects (font (size 1.27 1.27)) hide)
@@
     (in_bom yes) (on_board yes) (fields_autoplaced)
     (property "Reference" "R307" (id 0) (at 49.53 166.7342 90))
-    (property "Value" "10k" (id 1) (at 49.53 169.2711 90))
+    (property "Value" "51k" (id 1) (at 49.53 169.2711 90))
     (property "Footprint" "Resistor_SMD:R_0805_2012Metric_Pad1.20x1.40mm_HandSolder" (id 2) (at 49.53 173.228 90)
       (effects (font (size 1.27 1.27)) hide)
@@
     (in_bom yes) (on_board yes) (fields_autoplaced)
     (property "Reference" "R347" (id 0) (at 172.72 118.4742 90))
-    (property "Value" "33k" (id 1) (at 172.72 121.0111 90))
+    (property "Value" "51k" (id 1) (at 172.72 121.0111 90))
     (property "Footprint" "Resistor_SMD:R_0805_2012Metric_Pad1.20x1.40mm_HandSolder" (id 2) (at 172.72 124.968 90)
       (effects (font (size 1.27 1.27)) hide)
@@
     (in_bom yes) (on_board yes) (fields_autoplaced)
     (property "Reference" "R346" (id 0) (at 172.72 48.6242 90))
-    (property "Value" "33k" (id 1) (at 172.72 51.1611 90))
+    (property "Value" "51k" (id 1) (at 172.72 51.1611 90))
     (property "Footprint" "Resistor_SMD:R_0805_2012Metric_Pad1.20x1.40mm_HandSolder" (id 2) (at 172.72 55.118 90)
       (effects (font (size 1.27 1.27)) hide)
@@
       (effects (font (size 1.27 1.27)) (justify left))
     )
-    (property "Value" "R" (id 1) (at 64.008 112.1922 0)
+    (property "Value" "20k" (id 1) (at 64.008 112.1922 0)
       (effects (font (size 1.27 1.27)) (justify left))
     )
@@
       (effects (font (size 1.27 1.27)) (justify left))
     )
-    (property "Value" "R" (id 1) (at 64.008 102.0322 0)
+    (property "Value" "2k2" (id 1) (at 64.008 102.0322 0)
       (effects (font (size 1.27 1.27)) (justify left))
     )
@@
       (effects (font (size 1.27 1.27)) (justify left))
     )
-    (property "Value" "R" (id 1) (at 52.578 102.0322 0)
+    (property "Value" "2k2" (id 1) (at 52.578 102.0322 0)
       (effects (font (size 1.27 1.27)) (justify left))
     )
@@
       (effects (font (size 1.27 1.27)) (justify left))
     )
-    (property "Value" "R" (id 1) (at 52.578 112.1922 0)
+    (property "Value" "20k" (id 1) (at 52.578 112.1922 0)
       (effects (font (size 1.27 1.27)) (justify left))
     )
@@
     (in_bom yes) (on_board yes) (fields_autoplaced)
     (property "Reference" "R337" (id 0) (at 133.35 173.0842 90))
-    (property "Value" "10k" (id 1) (at 133.35 175.6211 90))
+    (property "Value" "51k" (id 1) (at 133.35 175.6211 90))
     (property "Footprint" "Resistor_SMD:R_0805_2012Metric_Pad1.20x1.40mm_HandSolder" (id 2) (at 133.35 179.578 90)
       (effects (font (size 1.27 1.27)) hide)
@@
       (effects (font (size 1.27 1.27)) (justify left))
     )
-    (property "Value" "R" (id 1) (at 64.008 42.3422 0)
+    (property "Value" "20k" (id 1) (at 64.008 42.3422 0)
       (effects (font (size 1.27 1.27)) (justify left))
     )
@@
       (effects (font (size 1.27 1.27)) (justify left))
     )
-    (property "Value" "R" (id 1) (at 64.008 32.1822 0)
-      (effects (font (size 1.27 1.27)) (justify left))
-    )
+    (property "Value" "2k2" (id 1) (at 64.008 32.1822 0)
+      (effects (font (size 1.27 1.27)) (justify left))
+    )

Commit message: daily???
Connections:
- net DPX_RX_ISOL_SW renamed DPX_RX_ISOL_SW_LOOP
- net DPX_RX_ISOL_SW_VOL renamed DPX_RX_ISOL_SW_LOOP_VOL
Changed lines of the file:
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@@
     (stroke (width 0) (type default) (color 0 0 0 0))
   )
-  (wire (pts (xy 33.02 16.51) (xy 40.64 16.51))
+  (wire (pts (xy 37.084 16.51) (xy 40.64 16.51))
     (stroke (width 0) (type default) (color 0 0 0 0))
   )
@@
     )
   )
-  (global_label "DPX_RX_ISOL_SW_VOL" (shape input) (at 52.07 16.51 0) (fields_autoplaced)
+  (global_label "DPX_RX_ISOL_SW_LOOP_VOL" (shape input) (at 52.07 16.51 0) (fields_autoplaced)
     (effects (font (size 1.27 1.27)) (justify left))
-    (property "Intersheet References" "${INTERSHEET_REFS}" (id 0) (at 74.8636 16.4306 0)
+    (property "Intersheet References" "${INTERSHEET_REFS}" (id 0) (at 80.7902 16.4306 0)
       (effects (font (size 1.27 1.27)) (justify left) hide)
     )
@@
     )
   )
-  (global_label "DPX_RX_ISOL_SW" (shape input) (at 33.02 16.51 180) (fields_autoplaced)
-    (effects (font (size 1.27 1.27)) (justify right))
-    (property "Intersheet References" "${INTERSHEET_REFS}" (id 0) (at 14.6412 16.5894 0)
-      (effects (font (size 1.27 1.27)) (justify right) hide)
-    )
+  (global_label "DPX_RX_ISOL_SW_LOOP" (shape input) (at 37.084 16.51 180) (fields_autoplaced)
+    (effects (font (size 1.27 1.27)) (justify right))
+    (property "Intersheet References" "${INTERSHEET_REFS}" (id 0) (at 12.7785 16.4306 0)
+      (effects (font (size 1.27 1.27)) (justify right) hide)
+    )
