File: fm-rpt-control-power.kicad_sch (KiCad schematic)
At the start: 0 parts

Commit message: schematic design ready
Parts:
- added C? (x6): 100n, Capacitor_SMD:C_0805_2012Metric_Pad1.18x1.45mm_HandSolder, symbol Device:C
- added C?: 67u, Capacitor_THT:CP_Radial_D8.0mm_P3.50mm, symbol Device:C_Polarized
- added C? (x2): 10u, Capacitor_Tantalum_SMD:CP_EIA-3528-21_Kemet-B_Pad1.50x2.35mm_HandSolder, symbol Device:C_Polarized
- added C?: 1u, Capacitor_SMD:C_0805_2012Metric_Pad1.18x1.45mm_HandSolder, symbol Device:C
- added D?: 1N4148W, Diode_SMD:D_SOD-123, symbol Diode:1N4148W
- added F? (x3): Polyfuse, Fuse:Fuse_2010_5025Metric_Pad1.52x2.65mm_HandSolder, symbol Device:Polyfuse
- added FL?: NFE31PT222Z1E9L, FIL_NFE31PT222Z1E9L, symbol murata_NFE31PT:NFE31PT222Z1E9L
- added J?: Jack-DC, Connector_BarrelJack:BarrelJack_GCT_DCJ200-10-A_Horizontal, symbol Connector:Jack-DC
- added L?: 100n, Inductor_SMD:L_0805_2012Metric_Pad1.15x1.40mm_HandSolder, symbol Device:L
- added U? (x2): L7805, Package_TO_SOT_THT:TO-220-2_Horizontal_TabDown, symbol Regulator_Linear:L7805
Connections:
- new net: C?.1, C?.1, C?.1, F?.1, U?.3 (OUT)
- new net: C?.1, C?.1, C?.1, L?.1, U?.3 (OUT)
- new net: C?.1, F?.1, L?.2
- new net: F?.2, FL?.1
- new net: D?.2 (A), J?.1
- new net: D?.1 (K), F?.1
- new net +5V: F?.2
- new net +VDC: C?.1, C?.1, C?.1, FL?.3, U?.1 (IN), U?.1 (IN)
- new net GND: C?.2, C?.2, C?.2, C?.2, C?.2, C?.2, C?.2, C?.2, C?.2, C?.2, FL?.2, FL?.2_1, FL?.2_2, J?.2, U?.2 (GND), U?.2 (GND)
- new net VDDA: F?.2

Commit message: PCB dimenstions set and db/din sockets, pots, switches and leds placed
Parts:
- U39, U40: renamed from U?; footprint Package_TO_SOT_THT:TO-220-2_Horizontal_TabDown -> Package_TO_SOT_THT:TO-220-3_Horizontal_TabDown
- gave numbers to parts that had none: 17
Other:
- company: (none) -> ML Elektronika Mateusz Lubecki
- title: (none) -> ParaCNTRL - FM repeater controller made of 74xx and analog

Commit message: controlling to_pc_retransmission line
Parts:
- renumbered D19 to D20, U39 to U40, U40 to U41
Connections:
- net +BATT: now reaches D20.2 (A), J9.1
Changed lines of the file:
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@@
   (junction (at 193.04 80.01) (diameter 0) (color 0 0 0 0)
   )
+  (junction (at 83.185 55.88) (diameter 0) (color 0 0 0 0)
+  )
   (junction (at 193.04 55.88) (diameter 0) (color 0 0 0 0)
   )
@@
     (stroke (width 0) (type default) (color 0 0 0 0))
   )
-  (wire (pts (xy 81.28 55.88) (xy 86.36 55.88))
+  (wire (pts (xy 81.28 55.88) (xy 83.185 55.88))
     (stroke (width 0) (type default) (color 0 0 0 0))
   )
@@
     (stroke (width 0) (type default) (color 0 0 0 0))
   )
+  (wire (pts (xy 83.185 55.88) (xy 86.36 55.88))
+    (stroke (width 0) (type default) (color 0 0 0 0))
+  )
   (wire (pts (xy 208.28 55.88) (xy 213.36 55.88))
     (stroke (width 0) (type default) (color 0 0 0 0))
@@
   )
   (wire (pts (xy 93.98 55.88) (xy 95.25 55.88))
+    (stroke (width 0) (type default) (color 0 0 0 0))
+  )
+  (wire (pts (xy 83.185 53.975) (xy 83.185 55.88))
     (stroke (width 0) (type default) (color 0 0 0 0))
   )
@@
   (symbol (lib_id "Regulator_Linear:L7805") (at 162.56 55.88 0) (unit 1)
     (in_bom yes) (on_board yes) (fields_autoplaced)
-    (property "Reference" "U39" (id 0) (at 162.56 50.2752 0))
+    (property "Reference" "U40" (id 0) (at 162.56 50.2752 0))
     (property "Value" "L7805" (id 1) (at 162.56 52.8121 0))
     (property "Footprint" "Package_TO_SOT_THT:TO-220-3_Horizontal_TabDown" (id 2) (at 163.195 59.69 0)
@@
   (symbol (lib_id "Regulator_Linear:L7805") (at 162.56 80.01 0) (unit 1)
     (in_bom yes) (on_board yes) (fields_autoplaced)
-    (property "Reference" "U40" (id 0) (at 162.56 74.4052 0))
+    (property "Reference" "U41" (id 0) (at 162.56 74.4052 0))
     (property "Value" "L7805" (id 1) (at 162.56 76.9421 0))
     (property "Footprint" "Package_TO_SOT_THT:TO-220-3_Horizontal_TabDown" (id 2) (at 163.195 83.82 0)
@@
     (pin "1")
   )
+  (symbol (lib_id "power:+BATT") (at 83.185 53.975 0) (unit 1)
+    (in_bom yes) (on_board yes) (fields_autoplaced)
+    (property "Reference" "#PWR077" (id 0) (at 83.185 57.785 0)
+      (effects (font (size 1.27 1.27)) hide)
+    )
+    (property "Value" "+BATT" (id 1) (at 83.185 50.3992 0))
+    (property "Footprint" "" (id 2) (at 83.185 53.975 0)
+      (effects (font (size 1.27 1.27)) hide)
+    )
+    (property "Datasheet" "" (id 3) (at 83.185 53.975 0)
+      (effects (font (size 1.27 1.27)) hide)
+    )
+    (pin "1")
+  )
   (symbol (lib_id "power:GND") (at 172.72 87.63 0) (unit 1)
     (in_bom yes) (on_board yes) (fields_autoplaced)
@@
   (symbol (lib_id "Diode:1N4148W") (at 90.17 55.88 180) (unit 1)
     (in_bom yes) (on_board yes) (fields_autoplaced)
-    (property "Reference" "D19" (id 0) (at 90.17 50.9102 0))
+    (property "Reference" "D20" (id 0) (at 90.17 50.9102 0))
     (property "Value" "1N4148W" (id 1) (at 90.17 53.4471 0))
     (property "Footprint" "Diode_SMD:D_SOD-123" (id 2) (at 90.17 51.435 0)

Commit message: logic ics, relays and relay driving electronics, voltage regulators placed
Parts:
- removed F1: Polyfuse, Fuse:Fuse_2010_5025Metric_Pad1.52x2.65mm_HandSolder, symbol Device:Polyfuse
- added F5: Fuse, Fuse:Fuseholder_Cylinder-5x20mm_Stelvio-Kontek_PTF78_Horizontal_Open, symbol Device:Fuse
- D20: value 1N4148W -> MURS120-E3; footprint Diode_SMD:D_SOD-123 -> Diode_SMD:D_SMB_Handsoldering
Connections:
- net at FL1.1: now also F5.2
- net at D20.1 (K): now also F5.1
Changed lines of the file:
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@@
     (pin "1")
+  )
+  (symbol (lib_id "Device:Fuse") (at 99.06 55.88 90) (unit 1)
+    (in_bom yes) (on_board yes) (fields_autoplaced)
+    (property "Reference" "F5" (id 0) (at 99.06 51.4182 90))
+    (property "Value" "Fuse" (id 1) (at 99.06 53.9551 90))
+    (property "Footprint" "Fuse:Fuseholder_Cylinder-5x20mm_Stelvio-Kontek_PTF78_Horizontal_Open" (id 2) (at 99.06 57.658 90)
+      (effects (font (size 1.27 1.27)) hide)
+    )
+    (property "Datasheet" "~" (id 3) (at 99.06 55.88 0)
+      (effects (font (size 1.27 1.27)) hide)
+    )
+    (pin "1")
+    (pin "2")
   )
   (symbol (lib_id "power:GND") (at 148.59 87.63 0) (unit 1)
@@
     (pin "1")
   )
-  (symbol (lib_id "Device:Polyfuse") (at 99.06 55.88 90) (unit 1)
-    (in_bom yes) (on_board yes) (fields_autoplaced)
-    (property "Reference" "F1" (id 0) (at 99.06 50.7832 90))
-    (property "Value" "Polyfuse" (id 1) (at 99.06 53.3201 90))
-    (property "Footprint" "Fuse:Fuse_2010_5025Metric_Pad1.52x2.65mm_HandSolder" (id 2) (at 104.14 54.61 0)
-      (effects (font (size 1.27 1.27)) (justify left) hide)
-    )
-    (property "Datasheet" "~" (id 3) (at 99.06 55.88 0)
-      (effects (font (size 1.27 1.27)) hide)
-    )
-    (pin "1")
-    (pin "2")
-  )
   (symbol (lib_id "power:GND") (at 182.88 63.5 0) (unit 1)
     (in_bom yes) (on_board yes) (fields_autoplaced)
@@
     (in_bom yes) (on_board yes) (fields_autoplaced)
     (property "Reference" "D20" (id 0) (at 90.17 50.9102 0))
-    (property "Value" "1N4148W" (id 1) (at 90.17 53.4471 0))
-    (property "Footprint" "Diode_SMD:D_SOD-123" (id 2) (at 90.17 51.435 0)
-      (effects (font (size 1.27 1.27)) hide)
-    )
+    (property "Value" "MURS120-E3" (id 1) (at 90.17 53.4471 0))
+    (property "Footprint" "Diode_SMD:D_SMB_Handsoldering" (id 2) (at 90.17 51.435 0)
+      (effects (font (size 1.27 1.27)) hide)
+    )

Commit message: +5v bus removed completely
Connections:
- net +5V: no longer names the net of F2.2
Changed lines of the file:
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@@
-    )
-  )
-  (global_label "+5V" (shape input) (at 208.28 80.01 0) (fields_autoplaced)
-    (effects (font (size 1.27 1.27)) (justify left))
-    (property "Intersheet References" "${INTERSHEET_REFS}" (id 0) (at 214.5636 79.9306 0)
-      (effects (font (size 1.27 1.27)) (justify left) hide)
     )
   )

Commit message: test
Connections:
- net +5V: now reaches F2.2
Changed lines of the file:
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@@
+    )
+  )
+  (global_label "+5V" (shape input) (at 208.28 80.01 0) (fields_autoplaced)
+    (effects (font (size 1.27 1.27)) (justify left))
+    (property "Intersheet References" "${INTERSHEET_REFS}" (id 0) (at 214.5636 79.9306 0)
+      (effects (font (size 1.27 1.27)) (justify left) hide)
     )
   )
