File: fm-rpt-control-power.kicad_sch (KiCad schematic)
At the start: 19 parts, among them J9 Jack-DC, U40 L7805, U41 L7805

Commit message: short fixed
Connections:
- net +5V_UNFUSED: now reaches C53.1, C55.1, C57.1, F2.1, U41.3 (OUT)
- net VDDA_UNFUSED: now reaches C52.1, C54.1, C56.1, L1.1, U40.3 (OUT)
Changed lines of the file:
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@@
     (stroke (width 0) (type default) (color 0 0 0 0))
+  )
+  (label "VDDA_UNFUSED" (at 174.625 55.88 0)
+    (effects (font (size 1.27 1.27)) (justify left bottom))
+  )
+  (label "+5V_UNFUSED" (at 175.26 80.01 0)
+    (effects (font (size 1.27 1.27)) (justify left bottom))
   )
   (global_label "VDDA" (shape input) (at 223.52 55.88 0) (fields_autoplaced)

Commit message: reannotated
Parts:
- renumbered C49 to C84, C50 to C85, C52 to C87, C54 to C88, C56 to C89, C58 to C91, C51 to C93, C53 to C95, C55 to C96, C57 to C97, D20 to D81, F5 to F82, F3 to F92, F2 to F98, FL1 to FL83, J9 to J80, L1 to L90, U40 to U86, U41 to U94
