File: fm-rpt-control.kicad_pcb (KiCad board)
At the start: 2 copper layers, 159.3 x 158.8 mm, 294 parts, among them IC1 74HC107D, IC2 74HC393M, IC3 74HC85D, IC4 74HC107D, IC5 LM567CH, IC6 74HC107D, J1 DUPLEX_RX, J2 SIMPLEX, J3 Conn_01x03_Male, J4 Conn_01x03_Male, J5 Conn_01x03_Male, J6 Conn_01x03_Male, J7 Conn_01x03_Male, J8 DUPLEX_TX, J9 Jack-DC, K1 RM12-3011-35-1005, K2 RM12__SPDT, Q1 BC856, Q2 BC856, Q3 BC856, Q4 BC846, Q5 BC858, Q6 BC858, Q7 BC848, SW1 SW_SPDT, SW2 SW_SPDT, SW3 SW_SPDT, SW4 SW_DPDT_x2, SW5 SW_SPDT, SW6 SW_DIP_x04, U1 SFH617A-1, U10 74LVC1G06GW, U11 74LVC1G06GW, U12 74AHC04, U13 74LVC1G06GW, U14 74HC74, U15 74HC08D, U16 74HC32D, U17 74HC32D, U18 74HC244D,652, U19 74HC02, U2 SFH617A-1, U20 74HC08D, U21 74HC08D, U22 74HC08D, U23 74HC32D, U24 74HC86, U25 74AHC04, U26 NE555D, U27 SFH617A-1, U28 SFH617A-1, U29 74HC244D,652, U3 SFH617A-1, U30 SFH617A-1, U31 HEF4093B, U32 LMV358, U33 LMV358, U34 LMV358, U35 LMV358, U36 LMV358, U37 LMV358, U38 74HC04, U39 L7805, U4 SFH617A-1, U40 L7805, U5 74HC244D,652, U6 SFH617A-1, U7 SFH617A-1, U8 74AHC1G08, U9 74LVC1G06GW, X1 REMOTE, X2 PC

Commit message: controlling to_pc_retransmission line
Parts:
- removed the IC4 at (-157.4, 108.5)
- removed the R29 at (-160.4, 125.5)
- removed the R34 at (-162.3, 129.9)
- removed the U9 at (-222.3, 101.2)
- added D5: LED, LED_SMD:LED_0805_2012Metric_Pad1.15x1.40mm_HandSolder, F.Cu at (-43.7, 185.0)
- added R10: 10k, Resistor_SMD:R_0805_2012Metric_Pad1.20x1.40mm_HandSolder, F.Cu at (-38.9, 185.0)
- added R21: 600, Resistor_SMD:R_0805_2012Metric_Pad1.20x1.40mm_HandSolder, F.Cu at (144.4, 8.00)
- added U31: 74AHC04, Package_SO:SOIC-14_3.9x8.7mm_P1.27mm, F.Cu at (-111.2, 51.6)
- C4, C5: value C_Polarized -> 120u
- R16: renamed from R15; value R -> 600
- SW1: value SW_SPDT -> DEBOUNCE
- SW2: value SW_SPDT -> SPX_ENABLE
- SW3: value SW_SPDT -> SPX_INHIBIT
- SW4: value SW_DPDT_x2 -> ROGER
- SW5: value SW_SPDT -> TX_TAIL
- moved U5 368.8 mm to (153.6, 41.3), turned to 90 degrees
- moved TR4 355.5 mm to (122.1, 47.0)
- moved TR6 326.2 mm to (99.6, 57.7)
- moved D10 316.5 mm to (123.7, 34.7)
- moved C4 298.3 mm to (114.8, 29.6), turned to -90 degrees
- moved C5 291.3 mm to (137.0, 33.2)
- moved R15 290.1 mm to (128.7, 34.3)
- moved R16 269.3 mm to (119.4, 34.4), turned to 180 degrees
- moved U6 242.6 mm to (108.7, 39.7), turned to -90 degrees
- moved TR1 237.6 mm to (26.6, 38.7)
- moved TR5 16.8 mm to (140.3, 47.0)
- moved U17 15.4 mm to (-146.7, 68.3)
- moved SW5 9.48 mm to (129.4, 169.5)
- moved SW1 8.39 mm to (120.3, 169.5)
- moved MAIN_OUT_VOL_SPX_1 4.99 mm to (40.3, 168.9)
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- renumbered D9 to D10, D10 to D11, D11 to D12, D12 to D13, D13 to D14, D14 to D15, D15 to D16, D16 to D17, D17 to D18, D18 to D19, D19 to D20, D5 to D6, D6 to D7, D7 to D8, D8 to D9, IC5 to IC4, IC6 to IC5, MASTER_AUD_DPX_1 to MAIN_OUT_VOL_DPX_1, MASTER_AUD_PC_1 to MAIN_OUT_VOL_PC_1, MASTER_AUD_SPX_1 to MAIN_OUT_VOL_SPX_1, R10 to R11, R11 to R12, R12 to R13, R13 to R14, R14 to R15, R16 to R17, R17 to R18, R18 to R19, R19 to R20, R20 to R22, R21 to R23, R22 to R24, R23 to R25, R24 to R26, R25 to R27, R26 to R28, R27 to R29, R28 to R30, R30 to R31, R31 to R32, R32 to R33, R33 to R34, U11 to U12, U12 to U13, U13 to U14, U14 to U15, U15 to U16, U16 to U17, U17 to U18, U18 to U19, U31 to U32, U32 to U33, U33 to U34, U34 to U35, U35 to U36, U36 to U37, U37 to U38, U38 to U39, U39 to U40, U40 to U41, U6 to U5, U7 to U6, U5 to U7, U19 to U8, U8 to U9
Connections:
- net Net-(D19-Pad2) renamed +BATT
- net Net-(IC2-Pad2) renamed /CNTR_CLR
- net Net-(U21-Pad3) renamed /SPX_PTT_CNTRL
- net Net-(U23-Pad3) renamed /DPX_PTT_CNTRL_WO_ROGER
- R22 pad 2: Net-(R20-Pad2) -> Net-(R22-Pad2)
- SW3 pad 3: unconnected-(SW3-Pad3) -> GND
- U10 pad 2: Net-(R20-Pad2) -> Net-(R22-Pad2)
- U10 pad 4: Net-(R29-Pad1) -> /~{RETRANSMIT_NEVER_DBCED}
- U21 pad 4: Net-(U19-Pad1) -> Net-(U21-Pad4)
- U5 pad 1: unconnected-(U6-Pad1) -> Net-(R21-Pad1)
- U5 pad 2: unconnected-(U6-Pad2) -> GND
- U6 pad 3: Net-(R20-Pad2) -> Net-(R22-Pad2)
- U8 pad 1: Net-(U19-Pad1) -> Net-(U8-Pad1)
- U8 pad 10: (no net) -> Net-(U21-Pad4)
- U8 pad 11: (no net) -> Net-(R22-Pad2)
- U8 pad 12: (no net) -> Net-(U31-Pad4)
- U8 pad 13: (no net) -> Net-(R21-Pad2)
- U8 pad 8: (no net) -> Net-(U8-Pad1)
- U8 pad 9: (no net) -> /SPX_CTCSS_DET_ISOL

Commit message: logic ics, relays and relay driving electronics, voltage regulators placed
Parts:
- added F4: Polyfuse, Fuse:Fuse_2010_5025Metric_Pad1.52x2.65mm_HandSolder, F.Cu at (112.3, 75.7)
- added F5: Fuse, Fuse:Fuseholder_Cylinder-5x20mm_Stelvio-Kontek_PTF78_Horizontal_Open, F.Cu at (166.9, 61.6)
- added R62: 0, Resistor_SMD:R_0805_2012Metric_Pad1.20x1.40mm_HandSolder, F.Cu at (198.2, 124.0)
- added R63: 0, Resistor_SMD:R_0805_2012Metric_Pad1.20x1.40mm_HandSolder, F.Cu at (202.9, 124.0)
- added R65: 10k, Resistor_SMD:R_0805_2012Metric_Pad1.20x1.40mm_HandSolder, F.Cu at (198.2, 121.1)
- added R66: 10k, Resistor_SMD:R_0805_2012Metric_Pad1.20x1.40mm_HandSolder, F.Cu at (202.9, 121.1)
- added U32: 74AHC1G32GW, Package_TO_SOT_SMD:SOT-353_SC-70-5_Handsoldering, F.Cu at (198.4, 110.0)
- D20: value 1N4148W -> MURS120-E3; footprint Diode_SMD:D_SOD-123 -> Diode_SMD:D_SMB_Handsoldering
- D7: moved to B.Cu
- DPX_HI1, DPX_LO1, DPX_VOL_1, PC_VOL_1, RV3, SPX_HI1, SPX_LO1, SPX_VOL_1: footprint Potentiometer_SMD:Potentiometer_Bourns_3314J_Vertical -> potentiometers:Potentiometer_SRpassives_1028F
- U9: value 74AHC1G08 -> 74AHC1G08GV
- moved ACC1 372.8 mm to (104.9, 72.8), turned to -90 degrees
- moved U22 366.7 mm to (131.8, 151.6), turned to -90 degrees
- moved RN1 362.0 mm to (101.4, 78.7), turned to 180 degrees
- moved U23 351.1 mm to (146.2, 151.6), turned to -90 degrees
- moved IC1 348.8 mm to (103.9, 126.4), turned to -90 degrees
- moved U10 347.5 mm to (110.8, 47.4), turned to -90 degrees
- moved U18 347.0 mm to (160.7, 138.9), turned to -90 degrees
- moved U25 344.4 mm to (160.7, 151.6), turned to -90 degrees
- moved C8 341.0 mm to (95.0, 38.8), turned to 90 degrees
- moved U15 339.4 mm to (117.3, 138.9), turned to -90 degrees
- moved IC5 339.4 mm to (65.4, 131.7)
- moved U29 330.0 mm to (74.7, 90.7), turned to -90 degrees
- moved J6 327.8 mm to (104.1, 30.2), turned to 90 degrees
- moved R56 325.3 mm to (157.0, 161.5)
- moved U7 325.1 mm to (139.8, 61.7), turned to 90 degrees
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- renumbered R96 to R100, R97 to R101, R98 to R102, R99 to R103, R100 to R104, R101 to R105, R102 to R106, R103 to R107, R104 to R108, R105 to R109, R106 to R110, R107 to R111, R108 to R112, R109 to R113, R110 to R114, R111 to R115, R112 to R116, R113 to R117, R114 to R118, R115 to R119, R116 to R120, R117 to R121, R118 to R122, R62 to R64, R63 to R67, R64 to R68, R65 to R69, R66 to R70, R67 to R71, R68 to R72, R69 to R73, R70 to R74, R71 to R75, R72 to R76, R73 to R77, R74 to R78, R75 to R79, R76 to R80, R77 to R81, R78 to R82, R79 to R83, R80 to R84, R81 to R85, R82 to R86, R83 to R87, R84 to R88, R85 to R89, R86 to R90, R87 to R91, R88 to R92, R89 to R93, R90 to R94, R91 to R95, R92 to R96, R93 to R97, R94 to R98, R95 to R99, U31 to U11, U32 to U31
Connections:
- net /RETRANSMIT_DBCED renamed RETRANSMIT_DBCED
- net /RETRANSMIT_NEVER_DBCED renamed RETRANSMIT_NEVER_DBCED
- net Net-(IC4-Pad8) renamed /AudioFilters/TONE_DET
- ACC1 pad 17: +5V -> /ACC_+V
- ACC1 pad 19: +5V -> /ACC_5V
- ACC1 pad 26: MASTER_AUD -> DPX_TX_ISOL
- ACC1 pad 28: MASTER_AUD -> SPX_TX_ISOL
- ACC1 pad 30: MASTER_AUD -> PC_TX_ISOL
- C19 pad 1: +5V -> VDDA
- C20 pad 1: +5V -> VDDA
- F1 pad 1: Net-(D20-Pad1) -> /ACC_+V
- F1 pad 2: Net-(F1-Pad2) -> +VDC
- FL1 pad 1: Net-(F1-Pad2) -> Net-(F5-Pad2)
- Q5 pad 2: +5V -> VDDA
- Q6 pad 2: +5V -> VDDA
- R103 pad 1: ROGER_AUDIO -> ROGER_AUDIO_SW
- R64 pad 1: +5V -> VDDA
- R73 pad 1: ROGER_AUDIO -> ROGER_AUDIO_SW
- SW4 pad 1: (no net) -> ROGER_AUDIO_SW
- SW4 pad 2: (no net) -> ROGER_AUDIO
- SW4 pad 3: (no net) -> unconnected-(SW4-Pad3)
- U31 pad 14: +5V -> VDDA
Routing:
- added copper zone on F.Cu, net GND

Commit message: before replacing some pinheaders with switches
Parts:
- added SW7: SW_SPDT, swtiches_spdt_dpdt:TL3XWO, F.Cu at (120.2, 169.5)
- added SW8: SKHHLRA010, Button_Switch_THT:SW_Tactile_SKHH_Angled, F.Cu at (167.1, 169.7)
- added SW9: SW_Push_DPDT, swtiches_spdt_dpdt:Ninigi_SS22F03-G6, F.Cu at (116.0, -8.25)
- SW1: footprint sterownik:TL3XWO -> swtiches_spdt_dpdt:Ninigi_MSS-2235S
- SW2, SW3, SW5: footprint sterownik:TL3XWO -> swtiches_spdt_dpdt:TL3XWO
- SW4: footprint sterownik:TL4XWO -> swtiches_spdt_dpdt:TL4XWO
- U35: value LMV358 -> 74AHC1G32GW; footprint Package_SO:SOIC-8_3.9x4.9mm_P1.27mm -> Package_TO_SOT_SMD:SOT-353_SC-70-5_Handsoldering
- moved U35 359.6 mm to (104.7, 88.0)
- moved U34 344.2 mm to (77.0, 128.5)
- moved U37 330.1 mm to (69.3, 156.7)
- moved C45 324.3 mm to (74.7, 153.2), turned to -90 degrees
- moved C33 323.1 mm to (72.6, 144.5), turned to 180 degrees
- moved C26 322.2 mm to (40.4, 115.8)
- moved U33 320.4 mm to (65.5, 142.5)
- moved R97 314.4 mm to (84.8, 125.5), turned to 180 degrees
- moved C40 313.5 mm to (47.8, 159.0)
- moved R113 311.4 mm to (83.6, 158.5), turned to 90 degrees
- moved R109 310.8 mm to (78.5, 155.7), turned to -90 degrees
- moved C30 310.7 mm to (72.9, 133.3), turned to 180 degrees
- moved R119 309.5 mm to (79.5, 145.0), turned to 180 degrees
- moved C34 307.3 mm to (80.8, 122.9), turned to 90 degrees
- moved C25 305.1 mm to (60.7, 120.1)
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Connections:
- net Net-(SW3-Pad2) renamed /SPX_INHIBIT_CNTRL
- net Net-(U14-Pad2) renamed /RETRNSMIT_ND_FROM_ACC
- ACC1 pad 15: GND -> +5V
- ACC1 pad 16: GND -> +5V
- C11 pad 2: GND -> +5V
- C12 pad 2: GND -> +5V
- C13 pad 2: GND -> +5V
- C14 pad 2: GND -> +5V
- C15 pad 2: GND -> +5V
- C16 pad 2: GND -> +5V
- C17 pad 2: GND -> +5V
- C18 pad 2: GND -> +5V
- C19 pad 1: VDDA -> +5V
- C19 pad 2: GND -> +5V
- C20 pad 1: VDDA -> +5V
- C20 pad 2: GND -> +5V
- C29 pad 1: GND -> +5V
- C30 pad 1: GND -> +5V
- C43 pad 1: GND -> +5V
- C44 pad 2: GND -> +5V
- C47 pad 2: GND -> +5V
- C49 pad 2: GND -> +5V
- C50 pad 2: GND -> +5V
- C51 pad 2: GND -> +5V
- C52 pad 2: GND -> +5V
- C53 pad 2: GND -> +5V
- C54 pad 2: GND -> +5V
- C55 pad 2: GND -> +5V
- C56 pad 2: GND -> +5V
- C57 pad 2: GND -> +5V
- C58 pad 2: GND -> +5V
- C6 pad 2: GND -> +5V
- C7 pad 2: GND -> +5V
- C8 pad 2: GND -> +5V
- C9 pad 2: GND -> +5V
- D11 pad 2: GND -> +5V
- D12 pad 2: GND -> +5V
- D13 pad 2: GND -> +5V
- D14 pad 2: GND -> +5V
- D8 pad 2: GND -> +5V
- DPX_HI1 pad 1: GND -> +5V
- DPX_LO1 pad 3: GND -> +5V
- DPX_VOL_1 pad 3: GND -> +5V
- FL1 pad 2: GND -> +5V
- FL1 pad 2_1: GND -> +5V
- FL1 pad 2_2: GND -> +5V
- IC1 pad 4: GND -> +5V
- IC1 pad 7: GND -> +5V
- IC2 pad 7: GND -> +5V
- IC3 pad 2: GND -> +5V
- IC3 pad 4: GND -> +5V
- IC3 pad 8: GND -> +5V
- IC4 pad 7: GND -> +5V
- IC5 pad 7: GND -> +5V
- J9 pad 2: GND -> +5V
- K1 pad 14: GND -> +5V
- K1 pad A1: GND -> +5V
- K2 pad A1: GND -> +5V
- MAIN_OUT_VOL_DPX_1 pad 3: GND -> +5V
- MAIN_OUT_VOL_PC_1 pad 3: GND -> +5V
- MAIN_OUT_VOL_SPX_1 pad 3: GND -> +5V
- PC_VOL_1 pad 3: GND -> +5V
- Q4 pad 2: GND -> +5V
- Q5 pad 2: VDDA -> +5V
- Q6 pad 2: VDDA -> +5V
- Q7 pad 2: GND -> +5V
- R10 pad 1: GND -> +5V
- R104 pad 2: GND -> +5V
- R110 pad 1: GND -> +5V
- R111 pad 1: GND -> +5V
- R121 pad 2: GND -> +5V
- R17 pad 2: GND -> +5V
- R18 pad 2: GND -> +5V
- R19 pad 2: GND -> +5V
- R22 pad 1: GND -> +5V
- R32 pad 2: GND -> +5V
- R33 pad 2: GND -> +5V
- R34 pad 1: GND -> +5V
- R35 pad 1: GND -> +5V
- R41 pad 2: GND -> +5V
- R52 pad 2: GND -> +5V
- R53 pad 2: GND -> +5V
- R54 pad 2: GND -> +5V
- R55 pad 2: GND -> +5V
- R56 pad 2: GND -> +5V
- R58 pad 1: GND -> +5V
- R59 pad 2: GND -> +5V
- R6 pad 1: GND -> +5V
- R64 pad 1: VDDA -> +5V
- R65 pad 1: GND -> +5V
- R66 pad 1: GND -> +5V
- R7 pad 1: GND -> +5V
- R74 pad 2: GND -> +5V
- R77 pad 2: GND -> +5V
- R79 pad 2: GND -> +5V
- R8 pad 1: GND -> +5V
- R81 pad 2: GND -> +5V
- R83 pad 2: GND -> +5V
- R85 pad 2: GND -> +5V
- R87 pad 2: GND -> +5V
- R9 pad 1: GND -> +5V
- R94 pad 1: GND -> +5V
- R95 pad 1: GND -> +5V
- RN1 pad 1: GND -> +5V
- RV3 pad 3: GND -> +5V
- SPX_HI1 pad 1: GND -> +5V
- SPX_LO1 pad 3: GND -> +5V
- SPX_VOL_1 pad 3: GND -> +5V
- SW3 pad 3: GND -> +5V
- SW6 pad 5: GND -> +5V
- SW6 pad 6: GND -> +5V
- SW6 pad 7: GND -> +5V
- SW6 pad 8: GND -> +5V
- TR1 pad P$3: GND -> +5V
- TR2 pad P$4: GND -> +5V
- TR3 pad P$4: GND -> +5V
- TR4 pad P$4: GND -> +5V
- TR5 pad P$4: GND -> +5V
- TR6 pad P$2: GND -> +5V
- U10 pad 3: GND -> +5V
- U11 pad 7: GND -> +5V
- U12 pad 3: GND -> +5V
- U13 pad 7: GND -> +5V
- U14 pad 3: GND -> +5V
- U15 pad 7: GND -> +5V
- U16 pad 7: GND -> +5V
- U17 pad 7: GND -> +5V
- U18 pad 7: GND -> +5V
- U19 pad 1: GND -> +5V
- U19 pad 10: GND -> +5V
- U19 pad 19: GND -> +5V
- U19 pad 9: /DPX_LOOP_INH_FROM_ACC -> Net-(U19-Pad9)
- U20 pad 7: GND -> +5V
- U21 pad 7: GND -> +5V
- U22 pad 7: GND -> +5V
- U23 pad 7: GND -> +5V
- U24 pad 7: GND -> +5V
- U25 pad 7: GND -> +5V
- U26 pad 1: GND -> +5V
- U27 pad 2: GND -> +5V
- U28 pad 2: GND -> +5V
- U29 pad 10: GND -> +5V
- U29 pad 13: GND -> +5V
- U29 pad 8: GND -> +5V
- U30 pad 2: GND -> +5V
- U31 pad 14: VDDA -> +5V
- U31 pad 7: GND -> +5V
- U32 pad 3: GND -> +5V
- U33 pad 1: Net-(C22-Pad1) -> Net-(C31-Pad2)
- U33 pad 2: Net-(R70-Pad2) -> Net-(C31-Pad2)
- U33 pad 3: Net-(R69-Pad2) -> Net-(C29-Pad2)
- U33 pad 4: unconnected-(U33-Pad4) -> +5V
- U34 pad 4: GND -> +5V
- U35 pad 1: Net-(C31-Pad2) -> /DPX_LOOP_INH_CNTRL
- U35 pad 2: Net-(C31-Pad2) -> Net-(U19-Pad9)
- U35 pad 3: Net-(C29-Pad2) -> +5V
- U35 pad 4: GND -> /DPX_LOOP_INH_FROM_ACC
- U35 pad 5: (no net) -> +5V
- U36 pad 1: Net-(C42-Pad1) -> Net-(C22-Pad1)
- U36 pad 2: Net-(R101-Pad2) -> Net-(R70-Pad2)
- U36 pad 3: Net-(R100-Pad2) -> Net-(R69-Pad2)
- U36 pad 4: (no net) -> +5V
- U36 pad 5: (no net) -> Net-(R100-Pad2)
- U36 pad 6: (no net) -> Net-(R101-Pad2)
- U36 pad 7: (no net) -> Net-(C42-Pad1)
- U36 pad 8: (no net) -> VDDA
- U37 pad 4: GND -> +5V
- U38 pad 4: unconnected-(U38-Pad4) -> +5V
- U38 pad 8: unconnected-(U38-Pad8) -> VDDA
- U39 pad 7: GND -> +5V
- U4 pad 2: GND -> +5V
- U40 pad 2: GND -> +5V
- U41 pad 2: GND -> +5V
- U5 pad 2: GND -> +5V
- U7 pad 1: GND -> +5V
- U7 pad 10: GND -> +5V
- U7 pad 19: GND -> +5V
- U8 pad 7: GND -> +5V
- U9 pad 3: GND -> +5V
- X1 pad 2: GND -> +5V
- X1 pad PE: GND -> +5V
- X1 pad PE@: GND -> +5V
Routing:
- added copper zone on F.Cu, net +5V
- removed copper zone on F.Cu, net GND
Other:
- board text added: "DUPLEX COR/CTCSS DEBOUNCE"
- board text added: "DUPLEX LOOP INH"
- board text added: "DUPLEX PTT"
- board text added: "ROGER BEEP"
- board text added: "SIMPLEX PORT INH ENABLE"
- board text added: "TX TAIL"

Commit message: short
Parts:
- removed J3, J4, J6, J7: Conn_01x03_Male, Connector_PinHeader_2.54mm:PinHeader_1x03_P2.54mm_Vertical
- added SW10: SW_Push_DPDT, swtiches_spdt_dpdt:Ninigi_SS22F03-G6, F.Cu at (94.1, 35.5)
- moved C15 282.5 mm to (168.1, 126.3), turned to -90 degrees
- moved SW9 53.7 mm to (79.8, 31.4), turned to 0 degrees
- moved R45 20.9 mm to (109.8, 50.0), turned to -90 degrees
- moved SW1 14.6 mm to (117.4, 113.3)
- moved C2 12.4 mm to (67.0, 31.8)
- moved C8 10.1 mm to (103.2, 44.7), turned to 0 degrees
- moved U6 4.12 mm to (108.0, 34.6)
- moved U30 3.99 mm to (101.8, 34.6)
- moved U10 3.63 mm to (110.8, 43.8)
- moved D14 3.06 mm to (87.6, 82.3)
- moved R37 3.06 mm to (100.3, 69.1)
- moved U19 3.06 mm to (96.5, 90.4)
- moved ACC1 3.06 mm to (107.9, 72.3)
- moved D13 3.06 mm to (99.3, 82.3)
- moved F1 3.06 mm to (115.3, 71.8)
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Connections:
- C11 pad 2: +5V -> unconnected-(C11-Pad2)
- C12 pad 2: +5V -> unconnected-(C12-Pad2)
- C13 pad 2: +5V -> unconnected-(C13-Pad2)
- C14 pad 2: +5V -> unconnected-(C14-Pad2)
- C15 pad 2: +5V -> unconnected-(C15-Pad2)
- C3 pad 1: Net-(C3-Pad1) -> Net-(SW9-Pad2)
- C9 pad 2: +5V -> unconnected-(C9-Pad2)
- IC4 pad 4: +5VA -> +5V
- R13 pad 1: Net-(J4-Pad2) -> Net-(R13-Pad1)
- SW9 pad 1: unconnected-(SW9-Pad1) -> /SPX_TX_AUD
- SW9 pad 2: unconnected-(SW9-Pad2) -> Net-(SW9-Pad2)
- SW9 pad 3: unconnected-(SW9-Pad3) -> /SPX_FLAT_TX_AUD
- SW9 pad 4: unconnected-(SW9-Pad4) -> /SPX_PTT
- SW9 pad 5: unconnected-(SW9-Pad5) -> Net-(R13-Pad1)
- SW9 pad 6: unconnected-(SW9-Pad6) -> /SPX_FLAT_PTT

Commit message: test
Connections:
- ACC1 pad 15: +5V -> GND
- ACC1 pad 16: +5V -> GND
- C11 pad 2: unconnected-(C11-Pad2) -> GND
- C12 pad 2: unconnected-(C12-Pad2) -> GND
- C13 pad 2: unconnected-(C13-Pad2) -> GND
- C14 pad 2: unconnected-(C14-Pad2) -> GND
- C15 pad 2: unconnected-(C15-Pad2) -> GND
- C16 pad 2: +5V -> GND
- C17 pad 2: +5V -> GND
- C18 pad 2: +5V -> GND
- C19 pad 1: +5V -> Net-(C19-Pad1)
- C19 pad 2: +5V -> GND
- C20 pad 1: +5V -> Net-(C19-Pad1)
- C20 pad 2: +5V -> GND
- C29 pad 1: +5V -> GND
- C30 pad 1: +5V -> GND
- C43 pad 1: +5V -> GND
- C44 pad 2: +5V -> GND
- C47 pad 2: +5V -> GND
- C49 pad 2: +5V -> GND
- C50 pad 2: +5V -> GND
- C51 pad 2: +5V -> GND
- C52 pad 2: +5V -> GND
- C53 pad 2: +5V -> GND
- C54 pad 2: +5V -> GND
- C55 pad 2: +5V -> GND
- C56 pad 2: +5V -> GND
- C57 pad 2: +5V -> GND
- C58 pad 2: +5V -> GND
- C6 pad 2: +5V -> GND
- C7 pad 2: +5V -> GND
- C8 pad 2: +5V -> GND
- C9 pad 2: unconnected-(C9-Pad2) -> GND
- D11 pad 2: +5V -> GND
- D12 pad 2: +5V -> GND
- D13 pad 2: +5V -> GND
- D14 pad 2: +5V -> GND
- D8 pad 2: +5V -> GND
- DPX_HI1 pad 1: +5V -> GND
- DPX_LO1 pad 3: +5V -> GND
- DPX_VOL_1 pad 3: +5V -> GND
- F4 pad 2: +5V -> unconnected-(F4-Pad2)
- FL1 pad 2: +5V -> GND
- FL1 pad 2_1: +5V -> GND
- FL1 pad 2_2: +5V -> GND
- IC1 pad 4: +5V -> GND
- IC1 pad 7: +5V -> GND
- IC2 pad 7: +5V -> GND
- IC3 pad 2: +5V -> GND
- IC3 pad 3: +5V -> unconnected-(IC3-Pad3)
- IC3 pad 4: +5V -> GND
- IC3 pad 8: +5V -> GND
- IC4 pad 4: +5V -> unconnected-(IC4-Pad4)
- IC4 pad 7: +5V -> GND
- IC5 pad 10: +5V -> unconnected-(IC5-Pad10)
- IC5 pad 11: +5V -> unconnected-(IC5-Pad11)
- IC5 pad 14: +5V -> unconnected-(IC5-Pad14)
- IC5 pad 7: +5V -> GND
- IC5 pad 8: +5V -> unconnected-(IC5-Pad8)
- J9 pad 2: +5V -> GND
- K1 pad 14: +5V -> GND
- K1 pad A1: +5V -> GND
- K2 pad A1: +5V -> GND
- MAIN_OUT_VOL_DPX_1 pad 3: +5V -> GND
- MAIN_OUT_VOL_PC_1 pad 3: +5V -> GND
- MAIN_OUT_VOL_SPX_1 pad 3: +5V -> GND
- PC_VOL_1 pad 3: +5V -> GND
- Q1 pad 2: +5V -> Net-(Q1-Pad2)
- Q4 pad 2: +5V -> GND
- Q5 pad 2: +5V -> unconnected-(Q5-Pad2)
- Q6 pad 2: +5V -> unconnected-(Q6-Pad2)
- Q7 pad 2: +5V -> GND
- R10 pad 1: +5V -> GND
- R104 pad 2: +5V -> GND
- R110 pad 1: +5V -> GND
- R111 pad 1: +5V -> GND
- R121 pad 2: +5V -> GND
- R17 pad 2: +5V -> GND
- R18 pad 2: +5V -> GND
- R19 pad 2: +5V -> GND
- R22 pad 1: +5V -> GND
- R26 pad 2: +5V -> Net-(Q1-Pad2)
- R30 pad 2: +5V -> unconnected-(R30-Pad2)
- R32 pad 2: +5V -> GND
- R33 pad 2: +5V -> GND
- R34 pad 1: +5V -> GND
- R35 pad 1: +5V -> GND
- R41 pad 2: +5V -> GND
- R52 pad 2: +5V -> GND
- R53 pad 2: +5V -> GND
- R54 pad 2: +5V -> GND
- R55 pad 2: +5V -> GND
- R56 pad 2: +5V -> GND
- R58 pad 1: +5V -> GND
- R59 pad 2: +5V -> GND
- R6 pad 1: +5V -> GND
- R64 pad 1: +5V -> unconnected-(R64-Pad1)
- R65 pad 1: +5V -> GND
- R66 pad 1: +5V -> GND
- R7 pad 1: +5V -> GND
- R74 pad 2: +5V -> GND
- R77 pad 2: +5V -> GND
- R79 pad 2: +5V -> GND
- R8 pad 1: +5V -> GND
- R81 pad 2: +5V -> GND
- R83 pad 2: +5V -> GND
- R85 pad 2: +5V -> GND
- R87 pad 2: +5V -> GND
- R9 pad 1: +5V -> GND
- R94 pad 1: +5V -> GND
- R95 pad 1: +5V -> GND
- RN1 pad 1: +5V -> GND
- RV3 pad 3: +5V -> GND
- SPX_HI1 pad 1: +5V -> GND
- SPX_LO1 pad 3: +5V -> GND
- SPX_VOL_1 pad 3: +5V -> GND
- SW2 pad 3: +5V -> unconnected-(SW2-Pad3)
- SW3 pad 1: +5V -> unconnected-(SW3-Pad1)
- SW3 pad 3: +5V -> GND
- SW6 pad 5: +5V -> GND
- SW6 pad 6: +5V -> GND
- SW6 pad 7: +5V -> GND
- SW6 pad 8: +5V -> GND
- SW7 pad 1: +5V -> GND
- SW7 pad 3: +5V -> unconnected-(SW7-Pad3)
- TR1 pad P$3: +5V -> GND
- TR2 pad P$4: +5V -> GND
- TR3 pad P$4: +5V -> GND
- TR4 pad P$4: +5V -> GND
- TR5 pad P$4: +5V -> GND
- TR6 pad P$2: +5V -> GND
- U1 pad 4: +5V -> unconnected-(U1-Pad4)
- U10 pad 3: +5V -> GND
- U10 pad 5: +5V -> GND
- U11 pad 7: +5V -> GND
- U12 pad 3: +5V -> GND
- U12 pad 5: +5V -> GND
- U13 pad 7: +5V -> GND
- U14 pad 3: +5V -> GND
- U14 pad 5: +5V -> GND
- U15 pad 7: +5V -> GND
- U16 pad 7: +5V -> GND
- U17 pad 7: +5V -> GND
- U18 pad 7: +5V -> GND
- U19 pad 1: +5V -> GND
- U19 pad 10: +5V -> GND
- U19 pad 19: +5V -> GND
- U19 pad 20: +5V -> unconnected-(U19-Pad20)
- U2 pad 4: +5V -> unconnected-(U2-Pad4)
- U20 pad 7: +5V -> GND
- U21 pad 7: +5V -> GND
- U22 pad 7: +5V -> GND
- U23 pad 7: +5V -> GND
- U24 pad 7: +5V -> GND
- U25 pad 7: +5V -> GND
- U26 pad 1: +5V -> GND
- U26 pad 4: +5V -> unconnected-(U26-Pad4)
- U27 pad 2: +5V -> GND
- U28 pad 2: +5V -> GND
- U29 pad 10: +5V -> GND
- U29 pad 13: +5V -> GND
- U29 pad 20: +5V -> unconnected-(U29-Pad20)
- U29 pad 8: +5V -> GND
- U3 pad 4: +5V -> unconnected-(U3-Pad4)
- U30 pad 2: +5V -> GND
- U31 pad 14: +5V -> Net-(C19-Pad1)
- U31 pad 7: +5V -> GND
- U32 pad 3: +5V -> GND
- U32 pad 5: +5V -> GND
- U33 pad 4: +5V -> GND
- U34 pad 4: +5V -> GND
- U35 pad 3: +5V -> GND
- U35 pad 5: +5V -> GND
- U36 pad 4: +5V -> GND
- U37 pad 4: +5V -> GND
- U38 pad 4: +5V -> GND
- U39 pad 14: +5V -> unconnected-(U39-Pad14)
- U39 pad 7: +5V -> GND
- U4 pad 2: +5V -> GND
- U40 pad 2: +5V -> GND
- U41 pad 2: +5V -> GND
- U5 pad 2: +5V -> GND
- U6 pad 4: +5V -> unconnected-(U6-Pad4)
- U7 pad 1: +5V -> GND
- U7 pad 10: +5V -> GND
- U7 pad 19: +5V -> GND
- U8 pad 7: +5V -> GND
- U9 pad 3: +5V -> GND
- U9 pad 5: +5V -> GND
- X1 pad 2: +5V -> GND
- X1 pad PE: +5V -> GND
- X1 pad PE@: +5V -> GND

Commit message: short fixed
Parts:
- SW7: value SW_SPDT -> SW_DPDT_x2; footprint swtiches_spdt_dpdt:TL3XWO -> swtiches_spdt_dpdt:TL4XWO
- U10: value 74LVC1G06GW -> 74LVC1G06
Connections:
- net Net-(C52-Pad1) renamed /Power/VDDA_UNFUSED
- net Net-(C53-Pad1) renamed /Power/+5V_UNFUSED
- net Net-(U19-Pad9) renamed /2Y3
- C19 pad 1: Net-(C19-Pad1) -> +5V
- C20 pad 1: Net-(C19-Pad1) -> +5V
- F4 pad 2: unconnected-(F4-Pad2) -> +5V
- IC3 pad 3: unconnected-(IC3-Pad3) -> +5V
- IC4 pad 4: unconnected-(IC4-Pad4) -> +5V
- IC5 pad 10: unconnected-(IC5-Pad10) -> +5V
- IC5 pad 11: unconnected-(IC5-Pad11) -> +5V
- IC5 pad 14: unconnected-(IC5-Pad14) -> +5V
- IC5 pad 8: unconnected-(IC5-Pad8) -> +5V
- Q5 pad 2: unconnected-(Q5-Pad2) -> +5V
- Q6 pad 2: unconnected-(Q6-Pad2) -> +5V
- R116 pad 2: +5VA -> +5V
- R30 pad 2: unconnected-(R30-Pad2) -> +5V
- R64 pad 1: unconnected-(R64-Pad1) -> +5V
- R71 pad 1: DUPLEX_MIX -> DUPLEX_MIX_SW
- SW2 pad 3: unconnected-(SW2-Pad3) -> +5V
- SW3 pad 1: unconnected-(SW3-Pad1) -> +5V
- SW7 pad 3: unconnected-(SW7-Pad3) -> +5V
- U10 pad 5: GND -> +5V
- U12 pad 5: GND -> +5V
- U14 pad 5: GND -> +5V
- U29 pad 1: unconnected-(U29-Pad1) -> GND
- U29 pad 19: unconnected-(U29-Pad19) -> GND
- U29 pad 20: unconnected-(U29-Pad20) -> +5V
- U31 pad 14: Net-(C19-Pad1) -> +5V
- U32 pad 5: GND -> +5V
- U35 pad 5: GND -> +5V
- U39 pad 14: unconnected-(U39-Pad14) -> +5V
- U9 pad 5: GND -> +5V
