File: fm-rpt-control.kicad_pcb (KiCad board)
At the start: 2 copper layers, 159.3 x 158.8 mm, 314 parts, among them IC1 74HC107D, IC2 74HC393M, IC3 74HC85D, IC4 LM567CH, IC5 74HC107D, J1 DUPLEX_RX, J2 SIMPLEX, J3 AudioJack3, J5 Conn_01x03_Male, J8 DUPLEX_TX, J9 Jack-DC, K1 RM12-3011-35-1005, K2 RM12__SPDT, Q1 BC856, Q2 BC856, Q3 BC856, Q4 BC846, Q5 BC858, Q6 BC858, Q7 BC848, SW1 DEBOUNCE, SW10 SW_Push_DPDT, SW2 SPX_ENABLE, SW3 SPX_INHIBIT, SW4 ROGER, SW5 TX_TAIL, SW6 SW_DIP_x04, SW7 SW_DPDT_x2, SW8 SKHHLRA010, SW9 SW_Push_DPDT, U1 SFH617A-1, U10 74LVC1G06, U11 74AHC04, U12 74LVC1G06GW, U13 74AHC04, U14 74LVC1G06GW, U15 74HC74, U16 74HC08D, U17 74HC32D, U18 74HC32D, U19 74HC244D,652, U2 SFH617A-1, U20 74HC08D, U21 74HC08D, U22 74HC08D, U23 74HC32D, U24 74HC86, U25 74AHC04, U26 NE555D, U27 SFH617A-1, U28 SFH617A-1, U29 74HC244D,652, U3 SFH617A-1, U30 SFH617A-1, U31 HEF4093B, U32 74AHC1G32GW, U33 LMV358, U34 LMV358, U35 74AHC1G32GW, U36 LMV358, U37 LMV358, U38 LMV358, U39 74HC04, U4 SFH617A-1, U40 L7805, U41 L7805, U5 SFH617A-1, U6 SFH617A-1, U7 74HC244D,652, U8 74HC02, U9 74AHC1G08GV, X1 REMOTE, X2 PC

Commit message: daily
Parts:
- moved C60 54.6 mm to (112.7, 64.9)
- moved R48 54.6 mm to (121.7, 65.8)
- moved R49 54.6 mm to (126.7, 59.1)
- moved U26 54.6 mm to (120.5, 62.1)
- moved C6 54.6 mm to (126.7, 63.0)
- moved C7 54.6 mm to (114.3, 61.2)
- moved R35 36.3 mm to (133.2, 158.2)
- moved R32 3.08 mm to (143.1, 119.2)
- moved R52 1.29 mm to (148.6, 160.0), turned to 90 degrees
- moved D2 1.10 mm to (170.4, 120.0)
- moved R7 1.10 mm to (170.4, 122.1)
- moved D1 1.08 mm to (170.4, 112.6)
- moved R6 1.08 mm to (170.4, 114.6)
- moved C12 0.95 mm to (167.0, 139.1)
- moved SW1 0.14 mm to (139.2, 112.0)
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Connections:
- IC3 pad 1: unconnected-(IC3-Pad1) -> /TAIL3
- IC3 pad 10: unconnected-(IC3-Pad10) -> /CNTR0
- IC3 pad 11: unconnected-(IC3-Pad11) -> /TAIL1
- IC3 pad 12: unconnected-(IC3-Pad12) -> /CNTR1
- IC3 pad 13: unconnected-(IC3-Pad13) -> /CNTR2
- IC3 pad 14: unconnected-(IC3-Pad14) -> /TAIL2
- IC3 pad 15: unconnected-(IC3-Pad15) -> /CNTR3
- IC3 pad 2: unconnected-(IC3-Pad2) -> GND
- IC3 pad 3: /DPX_TX_TAIL_CLR -> +5V
- IC3 pad 4: unconnected-(IC3-Pad4) -> GND
- IC3 pad 5: GND -> unconnected-(IC3-Pad5)
- IC3 pad 6: +5V -> /DPX_TX_TAIL_CLR
- IC3 pad 7: GND -> unconnected-(IC3-Pad7)
- IC3 pad 9: unconnected-(IC3-Pad9) -> /TAIL0
- U15 pad 1: unconnected-(U15-Pad1) -> +5V
Routing:
- net RETRANSMIT_DBCED: track 0.00 -> 146.0 mm, vias 0 -> 9
- net DUPLEX_MIX: track 0.00 -> 135.2 mm, vias 0 -> 5
- net ROGER_AUDIO_SW: track 0.00 -> 126.4 mm, vias 0 -> 1
- net DUPLEX_MIX_SW: track 0.00 -> 108.9 mm
- net /DPX_TX_TAIL: track 112.1 -> 210.0 mm, vias 7 -> 8
- net GND: track 21.6 -> 111.3 mm, vias 5 -> 31
- net /SPX_PTT_FROM_ACC: track 0.00 -> 89.0 mm, vias 0 -> 2
- net ROGER_PTT_CNTRL_OUT: track 0.00 -> 88.3 mm, vias 0 -> 3
- net +5V: track 381.7 -> 465.8 mm
- net /~{DPX_INHIBIT}: track 38.1 -> 113.3 mm, vias 1 -> 5
- net Net-(U13-Pad8): track 0.00 -> 73.9 mm, vias 0 -> 4
- net /SIMPLEX_PTT_ISOL: track 0.00 -> 72.8 mm, vias 0 -> 4
- net Net-(U13-Pad6): track 0.00 -> 67.1 mm, vias 0 -> 4
- net /DPX_LOOP_INH_CNTRL: track 0.00 -> 66.1 mm, vias 0 -> 1
- net /RETRANSMIT: track 0.00 -> 63.1 mm, vias 0 -> 5
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- added copper zone on B.Cu, net GND
- added copper zone on F.Cu, net GND
- removed copper zone on F.Cu, net +5V
Other:
- board text added: "ParaCNTRL Rev-A Mateusz Lubecki Bielsko-Biała 2023"
- board text removed: "ParaCNTRL Rev-A Mateusz Lubecki Bielsko-Biała"

Commit message: daily
Parts:
- moved C11 5.27 mm to (132.8, 144.0), turned to 180 degrees
- moved R92 1.27 mm to (71.2, 123.5)
- moved R13 1.10 mm to (56.0, 32.0), turned to 90 degrees
- moved R27 1.00 mm to (38.0, 74.7)
- moved R86 0.47 mm to (75.8, 122.2)
- moved R14 0.40 mm to (47.6, 48.4), turned to -90 degrees
- moved C44 0.40 mm to (47.5, 100.2)
- moved U28 0.40 mm to (51.9, 70.3)
- moved C57 0.38 mm to (147.7, 73.4), turned to 180 degrees
- moved R18 0.38 mm to (27.4, 62.2)
- moved C43 0.35 mm to (47.8, 105.7)
- moved C17 0.35 mm to (53.3, 92.0)
- moved R43 0.30 mm to (47.7, 75.5)
- moved R24 0.29 mm to (37.8, 61.9)
- moved U2 0.29 mm to (32.2, 58.6)
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Connections:
- ACC1 pad 25: DUPLEX_MASTER_AUD -> DPX_TX_ISOL
- ACC1 pad 26: DPX_TX_ISOL -> DUPLEX_MASTER_AUD
- ACC1 pad 27: SIMPLEX_MASTER_AUD -> SPX_TX_ISOL
- ACC1 pad 28: SPX_TX_ISOL -> SIMPLEX_MASTER_AUD
- ACC1 pad 29: PC_MASTER_AUD -> PC_TX_ISOL
- ACC1 pad 30: PC_TX_ISOL -> PC_MASTER_AUD
- MAIN_OUT_VOL_DPX_1 pad 2: DPX_TX_ISOL -> DUPLEX_MASTER_AUD
- MAIN_OUT_VOL_PC_1 pad 2: PC_TX_ISOL -> PC_MASTER_AUD
- MAIN_OUT_VOL_SPX_1 pad 2: SPX_TX_ISOL -> SIMPLEX_MASTER_AUD
- U1 pad 4: unconnected-(U1-Pad4) -> +5V
- U2 pad 4: unconnected-(U2-Pad4) -> +5V
- U3 pad 4: unconnected-(U3-Pad4) -> +5V
Routing:
- net +5V: track 465.8 -> 1026.7 mm, vias 22 -> 41
- net VDDA: track 0.00 -> 318.8 mm, vias 0 -> 12
- net GND: track 111.3 -> 418.6 mm, vias 31 -> 84
- net ROGER_AUDIO: track 0.00 -> 208.5 mm, vias 0 -> 4
- net SIMPLEX_MASTER_AUD: track 0.00 -> 199.4 mm, vias 0 -> 4
- net PC_MASTER_AUD: track 0.00 -> 172.8 mm, vias 0 -> 3
- net DUPLEX_MASTER_AUD: track 0.00 -> 154.1 mm, vias 0 -> 5
- net /RETRANSMIT: track 63.1 -> 196.9 mm, vias 5 -> 9
- net DPX_RX_ISOL_SW: track 0.00 -> 122.1 mm, vias 0 -> 6
- net ROGER_PTT_CNTRL_OUT: track 88.3 -> 188.2 mm, vias 3 -> 7
- net /DPX_TX_TAIL: track 210.0 -> 124.4 mm
- net SIMPLEX_MIX: track 0.00 -> 82.6 mm, vias 0 -> 3
- net Net-(C8-Pad1): track 0.00 -> 81.5 mm, vias 0 -> 5
- net SPX_ENABLE: track 47.1 -> 127.7 mm, vias 2 -> 4
- net PC_RX_ISOL: track 0.00 -> 77.5 mm, vias 0 -> 2
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