File: fm-rpt-control.kicad_sch (KiCad schematic)
At the start: 161 parts, among them IC1 74HC107D, IC2 74HC393M, IC3 74HC85D, J1 DUPLEX_RX, J2 SIMPLEX, J5 Conn_01x03_Male, J8 DUPLEX_TX, K1 RM12-3011-35-1005, K2 RM12__SPDT, Q1 BC856, Q2 BC856, Q3 BC856, Q4 BC846, SW1 DEBOUNCE, SW10 SW_Push_DPDT, SW2 SPX_ENABLE, SW3 SPX_INHIBIT, SW4 ROGER, SW5 TX_TAIL, SW6 SW_DIP_x04, SW7 SW_DPDT_x2, SW8 SKHHLRA010, SW9 SW_Push_DPDT, U1 SFH617A-1, U10 74LVC1G06, U11 74AHC04, U12 74LVC1G06GW, U13 74AHC04, U14 74LVC1G06GW, U15 74HC74, U16 74HC08D, U17 74HC32D, U18 74HC32D, U19 74HC244D,652, U2 SFH617A-1, U20 74HC08D, U21 74HC08D, U22 74HC08D, U23 74HC32D, U24 74HC86, U25 74AHC04, U27 SFH617A-1, U28 SFH617A-1, U29 74HC244D,652, U3 SFH617A-1, U30 SFH617A-1, U35 74AHC1G32GW, U4 SFH617A-1, U5 SFH617A-1, U6 SFH617A-1, U7 74HC244D,652, U8 74HC02, U9 74AHC1G08GV, X1 REMOTE, X2 PC

Commit message: daily
Connections:
- net +5V: now also IC3.3 (A=B_I), U15.1 (~{R}); no longer IC3.6 (A=B_O)
- net CNTR0: now also IC3.10 (A0)
- net CNTR1: now also IC3.12 (A1)
- net CNTR2: now also IC3.13 (A2)
- net CNTR3: now also IC3.15 (A3)
- net DPX_TX_TAIL_CLR: now also IC3.6 (A=B_O); no longer IC3.3 (A=B_I)
- net GND: now also IC3.2 (A<B_I), IC3.4 (A>B_I); no longer IC3.5 (A>B_O), IC3.7 (A<B_O)
- net TAIL0: now also IC3.9 (B0)
- net TAIL1: now also IC3.11 (B1)
- net TAIL2: now also IC3.14 (B2)
- net TAIL3: now also IC3.1 (B3)
Changed lines of the file:
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@@
     (stroke (width 0) (type default) (color 0 0 0 0))
   )
+  (wire (pts (xy 162.56 60.96) (xy 162.56 62.865))
+    (stroke (width 0) (type default) (color 0 0 0 0))
+  )
   (wire (pts (xy 80.01 189.23) (xy 82.55 189.23))
     (stroke (width 0) (type default) (color 0 0 0 0))
@@
     (stroke (width 0) (type default) (color 0 0 0 0))
   )
+  (wire (pts (xy 159.385 62.865) (xy 162.56 62.865))
+    (stroke (width 0) (type default) (color 0 0 0 0))
+  )
   (wire (pts (xy 30.48 115.57) (xy 33.02 115.57))
     (stroke (width 0) (type default) (color 0 0 0 0))
@@
     )
   )
+  (global_label "+5V" (shape input) (at 159.385 62.865 180) (fields_autoplaced)
+    (effects (font (size 1.27 1.27)) (justify right))
+    (property "Intersheet References" "${INTERSHEET_REFS}" (id 0) (at 153.1014 62.9444 0)
+      (effects (font (size 1.27 1.27)) (justify right) hide)
+    )
+  )
   (symbol (lib_id "Device:C_Polarized") (at 73.66 83.82 90) (unit 1)
     (in_bom yes) (on_board yes)
@@
     (pin "2")
   )
-  (symbol (lib_id "sterownik_eagle_import:7485D") (at 363.22 68.58 0) (mirror y) (unit 1)
+  (symbol (lib_id "sterownik_eagle_import:7485D") (at 363.22 68.58 0) (unit 1)
     (in_bom yes) (on_board yes) (fields_autoplaced)
     (property "Reference" "IC3" (id 0) (at 363.22 48.5974 0)
