File: fm-rpt-control.kicad_sch (KiCad schematic)
At the start: 100 parts, among them IC1 74HC107D, IC2 74HC393M, IC3 74HC85D, Q3 BC856, Q4 BC846, SW1 DEBOUNCE, SW2 SPX_ENABLE, SW3 SPX_INHIBIT, SW4 ROGER, SW5 TX_TAIL, SW6 SW_DIP_x04, SW7 SW_DPDT_x2, SW8 SKHHLRA010, U10 74LVC1G06, U11 74AHC04, U12 74LVC1G06GW, U13 74AHC04, U14 74LVC1G06GW, U15 74HC74, U16 74HC08D, U17 74HC32D, U18 74HC32D, U19 74HC244D,652, U20 74HC08D, U21 74HC08D, U22 74HC08D, U23 74HC32D, U24 74HC86, U25 74AHC04, U27 SFH617A-1, U28 SFH617A-1, U29 74HC244D,652, U35 74AHC1G32GW, U7 74HC244D,652, U8 74HC02, U9 74AHC1G08GV

Commit message: gerber files, some minor bugs in PCB solved
Other:
- moved on the sheet: U11C, U11D, U11E, U11F, U24E

Commit message: bugfix: not negating DPX_TX_TAIL_CLR before feeding 74hc107
Connections:
- net DPX_TX_TAIL_CLR: now also U11.5; no longer IC1.13 (~{RST})
- net ~{DPX_TX_TAIL_CLR}: now reaches U11.6
- net ~{DPX_TX_TAIL_CLR}: now also IC1.13 (~{RST})
Other:
- moved on the sheet: ACC1, C11, C12, C13, C14, C15, C59, C8, C9, D1, D13, D14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

Commit message: roger beep sligtly redesigned during assembly and debugging, bom with prices
Parts:
- R10, R123, R124, R125, R126, R52, R53, R54, R55, R56, R6, R7, R8, R9: value 10k -> 2k2
- R30, R34: value 51k -> 20k
- R35: value 10k -> 20k

Commit message: some minor changes in schematic only after protoype testing
Connections:
- net +5V: now also U19.20 (VCC)
- net ~{SPX_INHIBIT_FROM_RMT}: now also U8.2; no longer U13.5
- net at U13.6: no longer U8.2
Other:
- note added: "NOT was here"
- note added: "OR should be here"
- moved on the sheet: U13C
Changed lines of the file:
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@@
     (stroke (width 0) (type default) (color 0 0 0 0))
   )
-  (wire (pts (xy 124.46 120.65) (xy 151.13 120.65))
+  (wire (pts (xy 124.46 120.65) (xy 166.37 120.65))
     (stroke (width 0) (type default) (color 0 0 0 0))
   )
@@
     (stroke (width 0) (type default) (color 0 0 0 0))
   )
+  (wire (pts (xy 189.23 213.36) (xy 191.262 213.36))
+    (stroke (width 0) (type default) (color 0 0 0 0))
+  )
   (wire (pts (xy 137.16 90.17) (xy 137.16 100.33))
     (stroke (width 0) (type default) (color 0 0 0 0))
@@
     (stroke (width 0) (type default) (color 0 0 0 0))
   )
+  (text "NOT was here" (at 152.146 120.904 0)
+    (effects (font (size 1.27 1.27)) (justify left bottom))
+  )
+  (text "OR should be here" (at 171.196 195.072 0)
+    (effects (font (size 1.27 1.27)) (justify left bottom))
+  )
   (text "Switch DPDT: TST 2 N-RA KNITTER-SWITCH; \nSwtich SPDT: TST 1 D-RA KNITTER-SWITCH; 5FS1S102M6QE NINIGI\n"
     (at 103.505 17.145 0)
@@
     )
   )
+  (global_label "+5V" (shape input) (at 191.262 213.36 0) (fields_autoplaced)
+    (effects (font (size 1.27 1.27)) (justify left))
+    (property "Intersheet References" "${INTERSHEET_REFS}" (id 0) (at 197.5456 213.2806 0)
+      (effects (font (size 1.27 1.27)) (justify left) hide)
+    )
+  )
   (global_label "RETRANSMIT_DBCED" (shape input) (at 187.325 52.07 0) (fields_autoplaced)
     (effects (font (size 1.27 1.27)) (justify left))
@@
     (pin "2")
   )
-  (symbol (lib_id "74xx:74AHC04") (at 158.75 120.65 0) (unit 3)
+  (symbol (lib_id "74xx:74AHC04") (at 94.742 115.316 0) (unit 3)
     (in_bom yes) (on_board yes)
-    (property "Reference" "U13" (id 0) (at 161.29 118.11 0))
-    (property "Value" "74AHC04" (id 1) (at 158.75 115.6771 0))
-    (property "Footprint" "Package_SO:SOIC-14_3.9x8.7mm_P1.27mm" (id 2) (at 158.75 120.65 0)
+    (property "Reference" "U13" (id 0) (at 97.282 112.776 0))
+    (property "Value" "74AHC04" (id 1) (at 94.742 110.3431 0))
+    (property "Footprint" "Package_SO:SOIC-14_3.9x8.7mm_P1.27mm" (id 2) (at 94.742 115.316 0)
       (effects (font (size 1.27 1.27)) hide)
     )
-    (property "Datasheet" "https://assets.nexperia.com/documents/data-sheet/74AHC_AHCT04.pdf" (id 3) (at 158.75 120.65 0)
+    (property "Datasheet" "https://assets.nexperia.com/documents/data-sheet/74AHC_AHCT04.pdf" (id 3) (at 94.742 115.316 0)
       (effects (font (size 1.27 1.27)) hide)
     )

Commit message: pullup,pulldown resistors changed
Parts:
- R22, R23: value 22k -> 20k
- R25: value 2k2 -> 5k1
- R31: value 2k2 -> 51k
- R32, R33: value 51k -> 20k
- RN1: value 22k -> 10k
Other:
- moved on the sheet: U18D

Commit message: changes in pcb design rerouted except chanes around roger beep genrator. new hw rev
Parts:
- removed unit 5 of U20
- removed unit 4 of U20
- removed unit 3 of U20
- added U20: 74HC32D, Package_SO:SO-14_3.9x8.65mm_P1.27mm, symbol and_or_xor:74HC32D
- renumbered U20 to U22
Connections:
- net +5V: now also U20.14 (VCC)
- net GND: now also U20.7 (GND)
- net SPX_ENABLE: now also U20.13
- net SPX_ENABLE_CNTRL: now also U22.8; no longer U22.3
- net SPX_ENABLE_FROM_ACC: now also U20.9
- net SPX_MSTR_ENABLE: now also U22.10, U20.11; no longer U22.2
- net ~{SPX_INHIBIT}: now also U22.9; no longer U22.1
- net at R34.2, SW2.2 (B): now also U20.10
- new net: U20.12, U20.8
Other:
- moved on the sheet: U21E, U22E

Commit message: footprint of led indicators, rc delay network btween u9 and u12
Parts:
- added C1: 100n, Capacitor_SMD:C_0805_2012Metric_Pad1.18x1.45mm_HandSolder, symbol Device:C
- added R1: 630, Resistor_SMD:R_0603_1608Metric_Pad0.98x0.95mm_HandSolder, symbol Device:R
Connections:
- net GND: now also C1.2
- net at U12.2: now also C1.1, R1.1; no longer U9.4
- new net: R1.2, U9.4
Other:
- moved on the sheet: U12, U13C, U7, U9
