File: fm-rpt-control.kicad_sch (KiCad schematic)
At the start: 102 parts, among them IC1 74HC107D, IC2 74HC393M, IC3 74HC85D, Q3 BC856, Q4 BC846, SW1 DEBOUNCE, SW2 SPX_ENABLE, SW3 SPX_INHIBIT, SW4 ROGER, SW5 TX_TAIL, SW6 SW_DIP_x04, SW7 SW_DPDT_x2, SW8 SKHHLRA010, U10 74LVC1G06, U11 74AHC04, U12 74LVC1G06GW, U13 74AHC04, U14 74LVC1G06GW, U15 74HC74, U16 74HC08D, U17 74HC32D, U18 74HC32D, U19 74HC244D,652, U20 74HC32D, U21 74HC08D, U22 74HC08D, U23 74HC32D, U24 74HC86, U25 74AHC04, U27 SFH617A-1, U28 SFH617A-1, U29 74HC244D,652, U35 74AHC1G32GW, U7 74HC244D,652, U8 74HC02, U9 74AHC1G08GV

Commit message: reannotated
Parts:
- renumbered C8 to C2, C59 to C3, C9 to C4, C11 to C5, C12 to C6, C13 to C7, C14 to C8, C15 to C9, D13 to D1, D5 to D10, D16 to D11, D18 to D12, D23 to D13, D24 to D14, D14 to D2, D15 to D3, D21 to D4, D22 to D5, D1 to D6, D2 to D7, D3 to D8, D4 to D9, F4 to F2, IC1 to IC51, IC2 to IC52, IC3 to IC53, Q3 to Q1, Q4 to Q2, R22 to R1, R35 to R10, R36 to R11, R37 to R12, R38 to R13, R39 to R14, R40 to R15, R41 to R16, R42 to R17, R43 to R18, R44 to R19, R23 to R2, R45 to R20, R46 to R21, R47 to R22, R50 to R23, R123 to R24, R124 to R25, R6 to R26, R7 to R27, R8 to R28, R9 to R29, R1 to R3, R10 to R30, R125 to R31, R126 to R32, R54 to R33, R52 to R34, R53 to R35, R55 to R36, R56 to R37, R25 to R4, R30 to R5, R31 to R6, R32 to R7, R33 to R8, R34 to R9, SW7 to SW1, SW1 to SW2, SW2 to SW3, SW3 to SW4, SW4 to SW5, SW5 to SW6, SW8 to SW7, SW6 to SW8, U9 to U15, U10 to U16, U12 to U17, U14 to U18, U35 to U19, U19 to U20, U27 to U21, U28 to U22, U29 to U23, U25 to U50, U8 to U54, U11 to U55, U13 to U56, U15 to U57, U16 to U58, U17 to U59, U18 to U60, U20 to U61, U21 to U62, U22 to U63, U23 to U64, U24 to U65, U7 to U8

Commit message: simplex enable bugifx, now not inhibiting
Parts:
- removed unit 3 of U63
Connections:
- net SPX_MSTR_ENABLE is gone; now on net SPX_ENABLE_CNTRL: D9.2 (A), U61.11, U62.2
Changed lines of the file:
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@@
   (junction (at 207.01 228.6) (diameter 0) (color 0 0 0 0)
   )
-  (junction (at 209.55 186.69) (diameter 0) (color 0 0 0 0)
+  (junction (at 132.08 175.26) (diameter 0) (color 0 0 0 0)
   )
   (junction (at 335.28 29.845) (diameter 0) (color 0 0 0 0)
@@
     (stroke (width 0) (type default) (color 0 0 0 0))
   )
-  (wire (pts (xy 132.08 114.3) (xy 132.08 177.8))
+  (wire (pts (xy 132.08 114.3) (xy 132.08 175.26))
     (stroke (width 0) (type default) (color 0 0 0 0))
   )
@@
     (stroke (width 0) (type default) (color 0 0 0 0))
   )
+  (wire (pts (xy 132.08 175.26) (xy 209.55 175.26))
+    (stroke (width 0) (type default) (color 0 0 0 0))
+  )
   (wire (pts (xy 170.18 102.87) (xy 170.18 106.68))
     (stroke (width 0) (type default) (color 0 0 0 0))
@@
     (stroke (width 0) (type default) (color 0 0 0 0))
   )
-  (wire (pts (xy 121.92 175.26) (xy 245.11 175.26))
+  (wire (pts (xy 121.92 175.26) (xy 132.08 175.26))
     (stroke (width 0) (type default) (color 0 0 0 0))
   )
@@
     (stroke (width 0) (type default) (color 0 0 0 0))
   )
-  (wire (pts (xy 209.55 177.8) (xy 132.08 177.8))
-    (stroke (width 0) (type default) (color 0 0 0 0))
-  )
   (wire (pts (xy 195.58 71.12) (xy 201.93 71.12))
     (stroke (width 0) (type default) (color 0 0 0 0))
@@
     (stroke (width 0) (type default) (color 0 0 0 0))
   )
-  (wire (pts (xy 209.55 186.69) (xy 209.55 177.8))
-    (stroke (width 0) (type default) (color 0 0 0 0))
-  )
   (wire (pts (xy 377.825 206.375) (xy 381.635 206.375))
     (stroke (width 0) (type default) (color 0 0 0 0))
@@
     (stroke (width 0) (type default) (color 0 0 0 0))
   )
-  (wire (pts (xy 209.55 186.69) (xy 209.55 189.23))
+  (wire (pts (xy 209.55 175.26) (xy 209.55 189.23))
     (stroke (width 0) (type default) (color 0 0 0 0))
   )
@@
     (stroke (width 0) (type default) (color 0 0 0 0))
   )
-  (wire (pts (xy 209.55 186.69) (xy 228.6 186.69))
-    (stroke (width 0) (type default) (color 0 0 0 0))
-  )
   (wire (pts (xy 189.23 134.62) (xy 187.96 134.62))
     (stroke (width 0) (type default) (color 0 0 0 0))
@@
     (stroke (width 0) (type default) (color 0 0 0 0))
   )
-  (wire (pts (xy 245.11 175.26) (xy 245.11 184.15))
-    (stroke (width 0) (type default) (color 0 0 0 0))
-  )
   (wire (pts (xy 345.44 21.59) (xy 356.87 21.59))
     (stroke (width 0) (type default) (color 0 0 0 0))
@@
     (stroke (width 0) (type default) (color 0 0 0 0))
   )
-  (wire (pts (xy 217.17 181.61) (xy 228.6 181.61))
-    (stroke (width 0) (type default) (color 0 0 0 0))
-  )
   (wire (pts (xy 293.37 151.13) (xy 293.37 152.4))
     (stroke (width 0) (type default) (color 0 0 0 0))
@@
     (stroke (width 0) (type default) (color 0 0 0 0))
   )
-  (wire (pts (xy 245.11 184.15) (xy 243.84 184.15))
-    (stroke (width 0) (type default) (color 0 0 0 0))
-  )
   (wire (pts (xy 96.52 72.39) (xy 96.52 69.85))
     (stroke (width 0) (type default) (color 0 0 0 0))
@@
     (effects (font (size 1.27 1.27)) (justify left bottom))
   )
-  (label "SPX_MSTR_ENABLE" (at 157.48 114.3 0)
+  (label "SPX_ENABLE_CNTRL" (at 153.67 114.3 0)
     (effects (font (size 1.27 1.27)) (justify left bottom))
   )
@@
     (effects (font (size 1.27 1.27)) (justify left bottom))
   )
-  (label "SPX_MSTR_ENABLE" (at 153.67 177.8 0)
-    (effects (font (size 1.27 1.27)) (justify left bottom))
-  )
   (label "CLK" (at 119.38 53.34 0)
     (effects (font (size 1.27 1.27)) (justify left bottom))
@@
     (effects (font (size 1.27 1.27)) (justify left bottom))
   )
-  (label "SPX_MSTR_ENABLE" (at 345.44 199.39 0)
+  (label "SPX_ENABLE_CNTRL" (at 345.44 199.39 0)
     (effects (font (size 1.27 1.27)) (justify left bottom))
   )
@@
     (effects (font (size 1.27 1.27)) (justify left bottom))
   )
-  (label "SPX_MSTR_ENABLE" (at 210.82 186.69 0)
-    (effects (font (size 1.27 1.27)) (justify left bottom))
-  )
   (label "OACC_DPX_RETRN_ND" (at 242.57 209.55 0)
     (effects (font (size 1.27 1.27)) (justify left bottom))
@@
     (effects (font (size 1.27 1.27)) (justify left bottom))
   )
-  (label "~{SPX_INHIBIT}" (at 217.17 181.61 0)
-    (effects (font (size 1.27 1.27)) (justify left bottom))
-  )
   (label "~{DPX_PTT_DIR_FROM_RMT}" (at 86.36 168.91 0)
     (effects (font (size 1.27 1.27)) (justify left bottom))
@@
     (pin "1")
   )
-  (symbol (lib_id "and_or_xor:74HC08D") (at 236.22 184.15 0) (unit 3)
-    (in_bom yes) (on_board yes) (fields_autoplaced)
-    (property "Reference" "U63" (id 0) (at 236.22 176.6402 0))
-    (property "Value" "74HC08D" (id 1) (at 236.22 179.1771 0))
-    (property "Footprint" "Package_SO:SO-14_3.9x8.65mm_P1.27mm" (id 2) (at 236.22 184.15 0)
-      (effects (font (size 1.27 1.27)) hide)
-    )
-    (property "Datasheet" "https://assets.nexperia.com/documents/data-sheet/74HC_HCT08.pdf" (id 3) (at 236.22 184.15 0)
-      (effects (font (size 1.27 1.27)) hide)
-    )
-    (pin "10")
-    (pin "8")
-    (pin "9")
-  )
   (symbol (lib_id "Device:R") (at 265.43 256.54 0) (mirror y) (unit 1)
     (in_bom yes) (on_board yes)
@@
       (reference "U63") (unit 2) (value "74HC08D") (footprint "Package_SO:SO-14_3.9x8.65mm_P1.27mm")
     )
-    (path "/33cc48bc-5e0b-4602-822b-0931498e9cb5"
-      (reference "U63") (unit 3) (value "74HC08D") (footprint "Package_SO:SO-14_3.9x8.65mm_P1.27mm")
-    )
     (path "/d4e424cc-59bc-41d7-8b00-c5badfe2e2e5"

Commit message: simplex remote control tone detector redesigned, gerber files for hw-rev b
Connections:
- net SPX_ENABLE: now also D9.2 (A), U15.2, U23.15 (2A1), U61.11, U62.2; no longer U61.13
- net SPX_ENABLE_CNTRL: now also U61.13; no longer D9.2 (A), U15.2, U23.15 (2A1), U61.11, U62.2
Other:
- added sheet ToneDetect (fm-rpt-control-tonedetect.kicad_sch)
- moved on the sheet: U61D

Commit message: daily???
Parts:
- added unit 3 of U62
- ACC1: footprint Connector_PinHeader_2.54mm:PinHeader_2x15_P2.54mm_Vertical -> Connector_PinHeader_2.54mm:PinHeader_2x16_P2.54mm_Vertical; symbol Connector_Generic:Conn_02x15_Odd_Even -> Connector_Generic:Conn_02x16_Odd_Even
Connections:
- net SPX_ENABLE: now also U62.8; no longer U61.11
- net SPX_PTT_AFT_INHIBIT: now also U62.11; no longer U62.8
- net SPX_PTT_CNTRL: now also U62.12; no longer U62.9
- net ~{SPX_INHIBIT}: now also U62.13, U62.9; no longer U62.10
- new net: U61.11, U62.10
- new net DPX_RX_ISOL_SW: ACC1.31 (Pin_31)
- new net DPX_RX_ISOL_SW_LOOP: ACC1.32 (Pin_32)
Other:
- moved on the sheet: F1, F2, R11, R12, R13, R14, R15, R16, R17, R18, U21, U22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

Commit message: before fixing problems with potentiometers orientation
Parts:
- removed unit 4 of U59
- added unit 4 of U58
Connections:
- net ~{DPX_INHIBIT_FROM_RMT}: now also U58.12
- net ~{DPX_INHIBIT}: now also U58.11
- net at U56.4: now also U58.13
Changed lines of the file:
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@@
     (pin "3")
   )
+  (symbol (lib_id "and_or_xor:74HC08D") (at 170.18 87.63 0) (unit 4)
+    (in_bom yes) (on_board yes) (fields_autoplaced)
+    (property "Reference" "U58" (id 0) (at 170.18 80.1202 0))
+    (property "Value" "74HC08D" (id 1) (at 170.18 82.6571 0))
+    (property "Footprint" "Package_SO:SO-14_3.9x8.65mm_P1.27mm" (id 2) (at 170.18 87.63 0)
+      (effects (font (size 1.27 1.27)) hide)
+    )
+    (property "Datasheet" "https://assets.nexperia.com/documents/data-sheet/74HC_HCT08.pdf" (id 3) (at 170.18 87.63 0)
+      (effects (font (size 1.27 1.27)) hide)
+    )
+    (pin "11")
+    (pin "12")
+    (pin "13")
+  )
   (symbol (lib_id "Switch:SW_Push") (at 277.495 133.985 0) (unit 1)
     (in_bom yes) (on_board yes) (fields_autoplaced)
@@
     (pin "1")
   )
-  (symbol (lib_id "and_or_xor:74HC32D") (at 170.18 87.63 0) (unit 4)
-    (in_bom yes) (on_board yes) (fields_autoplaced)
-    (property "Reference" "U59" (id 0) (at 170.18 80.1202 0))
-    (property "Value" "74HC32D" (id 1) (at 170.18 82.6571 0))
-    (property "Footprint" "Package_SO:SO-14_3.9x8.65mm_P1.27mm" (id 2) (at 170.18 81.28 0)
-      (effects (font (size 1.27 1.27)) hide)
-    )
-    (property "Datasheet" "https://assets.nexperia.com/documents/data-sheet/74HC_HCT32.pdf" (id 3) (at 170.18 92.71 0)
-      (effects (font (size 1.27 1.27)) hide)
-    )
-    (pin "11")
-    (pin "12")
-    (pin "13")
-  )
   (symbol (lib_id "74xx:74AHC04") (at 167.64 165.1 0) (unit 5)
     (in_bom yes) (on_board yes)
@@
       (reference "#GND0101") (unit 1) (value "GND") (footprint "")
     )
+    (path "/c4cedb5a-0852-4d10-ad65-b93391ba7da5/428a0152-7118-4dc7-a429-d1474530d981"
+      (reference "#GND0102") (unit 1) (value "GND") (footprint "")
+    )
     (path "/e4c6fdbb-fdc7-4ad4-a516-240d84cdc120/393f0e56-c2d5-4ea4-8463-50265bc94d2d"
       (reference "#GND0203") (unit 1) (value "GND") (footprint "")
@@
     )
     (path "/c4cedb5a-0852-4d10-ad65-b93391ba7da5/b79ec85b-74d5-4cef-9912-36616da6e356"
-      (reference "IC?") (unit 3) (value "74HC107D") (footprint "Package_SO:SO-14_3.9x8.65mm_P1.27mm")
+      (reference "IC702") (unit 3) (value "74HC107D") (footprint "Package_SO:SO-14_3.9x8.65mm_P1.27mm")
     )
     (path "/78e4f606-ccca-418a-a2ce-b312716883d6/94a507f2-dd02-4248-92ef-4340458ab03a"
@@
       (reference "U58") (unit 2) (value "74HC08D") (footprint "Package_SO:SO-14_3.9x8.65mm_P1.27mm")
     )
+    (path "/7bc33526-a174-4440-8551-bf77b0128d4e"
+      (reference "U58") (unit 4) (value "74HC08D") (footprint "Package_SO:SO-14_3.9x8.65mm_P1.27mm")
+    )
     (path "/4d2614bd-c48e-4dce-ae5b-fcc800687924"
       (reference "U58") (unit 5) (value "74HC08D") (footprint "Package_SO:SO-14_3.9x8.65mm_P1.27mm")
@@
       (reference "U59") (unit 3) (value "74HC32D") (footprint "Package_SO:SO-14_3.9x8.65mm_P1.27mm")
     )
-    (path "/82165c80-a765-4460-84a2-154dcb632ff6"
-      (reference "U59") (unit 4) (value "74HC32D") (footprint "Package_SO:SO-14_3.9x8.65mm_P1.27mm")
-    )
     (path "/fa4c32a4-8dc8-40b7-b74c-b3f409f34c8b"
