File: fm-rpt-connectors.kicad_sch (KiCad schematic)
At the start: 0 parts

Commit message: moved to separate scheed, before reasigning designators
Parts:
- added C? (x4): C_Polarized, Capacitor_THT:C_Radial_D6.3mm_H7.0mm_P2.50mm, symbol Device:C_Polarized
- added C? (x2): 120u, Capacitor_THT:C_Radial_D6.3mm_H7.0mm_P2.50mm, symbol Device:C_Polarized
- added D? (x4): 1N4148W, Diode_SMD:D_SOD-123, symbol Diode:1N4148W
- added D? (x4): ESDA6V1-5SC6, Package_TO_SOT_SMD:SOT-23-6, symbol Power_Protection:ESDA6V1-5SC6
- added J?: DUPLEX_TX, Connector_Dsub:DSUB-9_Female_Horizontal_P2.77x2.84mm_EdgePinOffset4.94mm_Housed_MountingHolesOffset7.48mm, symbol Connector:DB9_Female
- added J?: Conn_01x03_Male, Connector_PinHeader_2.54mm:PinHeader_1x03_P2.54mm_Vertical, symbol Connector:Conn_01x03_Male
- added J?: DUPLEX_RX, Connector_Dsub:DSUB-9_Female_Horizontal_P2.77x2.84mm_EdgePinOffset4.94mm_Housed_MountingHolesOffset7.48mm, symbol Connector:DB9_Female
- added J?: SIMPLEX, Connector_Dsub:DSUB-9_Female_Horizontal_P2.77x2.84mm_EdgePinOffset4.94mm_Housed_MountingHolesOffset7.48mm, symbol Connector:DB9_Female
- added K?: RM12-3011-35-1005, relays:Relay_SPDT_Relpol_RM12, symbol relays:RM12__SPDT
- added K?: RM12__SPDT, relays:Relay_SPDT_Relpol_RM12, symbol relays:RM12__SPDT
- added Q? (x2): BC856, Package_TO_SOT_SMD:SOT-23, symbol Transistor_BJT:BC856
- added R? (x6): 10k, Resistor_SMD:R_0805_2012Metric_Pad1.20x1.40mm_HandSolder, symbol Device:R
- added R? (x4): 22k, Resistor_SMD:R_0805_2012Metric_Pad1.20x1.40mm_HandSolder, symbol Device:R
- added R? (x5): R, Resistor_SMD:R_0805_2012Metric_Pad1.20x1.40mm_HandSolder, symbol Device:R
- added R?: 2k2, Resistor_SMD:R_0805_2012Metric_Pad1.20x1.40mm_HandSolder, symbol Device:R
- added R? (x2): 600, Resistor_SMD:R_0805_2012Metric_Pad1.20x1.40mm_HandSolder, symbol Device:R
- added R?: 660, Resistor_SMD:R_0805_2012Metric_Pad1.20x1.40mm_HandSolder, symbol Device:R
- added R?: 330, Resistor_SMD:R_0805_2012Metric_Pad1.20x1.40mm_HandSolder, symbol Device:R
- added R? (x2): 51k, Resistor_SMD:R_0805_2012Metric_Pad1.20x1.40mm_HandSolder, symbol Device:R
- added SW? (x2): SW_Push_DPDT, swtiches_spdt_dpdt:Ninigi_SS22F03-G6, symbol Switch:SW_Push_DPDT
- added TR? (x6): CRIYCHLEY9000, paratnc_cp:NORMAL, symbol paratnc_cp_import:CRIYCHLEY9000
- added U? (x7): SFH617A-1, Package_DIP:SMDIP-4_W9.53mm, symbol Isolator:SFH617A-1
- added X?: REMOTE, sterownik:MAB8SH, symbol sterownik_eagle_import:MAB8SH
- added X?: PC, sterownik:MAB5SH, symbol sterownik_eagle_import:MAB5SH
Connections:
- new net: C?.1, SW?.5 (B)
- new net: C?.2, TR?.P$3
- new net: C?.2, TR?.P$1 (x4)
- new net: D?.1 (K), K?.A2, Q?.3 (C) (x2)
- new net: R?.1, U?.1 (x2)
- new net: R?.2, U?.4 (x2)
- new net: Q?.1 (B), R?.1, R?.2, R?.2
- new net: R?.2, U?.1 (x5)
- new net: Q?.1 (B), R?.1, R?.2
- new net: D?.1 (K), R?.1 (x2)
- new net: SW?.2 (B), U?.4
- new net: R?.1, SW?.5 (B)
- new net: C?.2, TR?.P$2
- new net: C?.1, SW?.2 (B)
- new net +5V: Q?.2 (E), Q?.2 (E), R?.2, R?.2, R?.2, R?.2, R?.2, R?.2, R?.2, U?.4, U?.4, U?.4, U?.4
- new net DPX_CARRIER_DET: D?.5 (IO4), J?.6, R?.1
- new net DPX_CARRIER_DET_ISOL: J?.3 (Pin_3), R?.1, U?.3
- new net DPX_CTCSS_DET: D?.6 (IO5), J?.1, R?.1
- new net DPX_CTCSS_DET_ISOL: J?.1 (Pin_1), R?.1, U?.3
- new net DPX_FLAT_PTT: D?.4 (IO3), J?.9, SW?.3 (C)
- new net DPX_FLAT_TX_AUD: D?.6 (IO5), J?.2, SW?.6 (C)
- new net DPX_PTT: D?.5 (IO4), J?.4, SW?.1 (A)
- new net DPX_RX_AUD: C?.1, D?.4 (IO3), J?.3
- new net DPX_RX_ISOL: K?.12, TR?.P$4
- new net DPX_RX_ISOL_SW: K?.11
- new net DPX_TX_AUD: D?.3 (IO2), J?.5, SW?.4 (A)
- new net DPX_TX_ISOL: TR?.P$1
- new net DUPLEX_PTT_ISOL_MASTER: R?.1
- new net GND: D?.2 (A), D?.2 (A), D?.2 (GND), K?.14, K?.A1, K?.A1, R?.2, R?.2, R?.2, TR?.P$2, TR?.P$3, TR?.P$4, TR?.P$4, TR?.P$4, TR?.P$4, U?.2, U?.2, U?.2, X?.2, X?.PE, X?.PE@ (PE)
- new net GND1: TR?.P$2, TR?.P$2, U?.2, U?.3, X?.2, X?.PE, X?.PE@ (PE)
- new net GND2: J?.7, TR?.P$1
- new net GND3: D?.2 (GND), J?.7, TR?.P$4, U?.3
- new net GNDS: D?.2 (GND), D?.2 (GND), J?.7, TR?.P$2, TR?.P$2, U?.2, U?.2, U?.2, U?.3
- new net PC_FROM_AUD: C?.1, X?.1
- new net PC_FROM_PTT: D?.2 (A), X?.3
- new net PC_FROM_PTT_ISOL: U?.3
- new net PC_RX_ISOL: TR?.P$3
- new net PC_TO_AUD: C?.1, X?.4
- new net PC_TO_RETR_ACTIVE: R?.1, X?.5
- new net PC_TO_RETR_ACTIVE_ISOL: R?.2
- new net PC_TX_ISOL: TR?.P$3
- new net RETRANSMIT: J?.2 (Pin_2)
- new net RMT_ACC_PIN4: X?.4
- new net RMT_ACC_PIN5: X?.5
- new net SIMPLEX_PTT_ISOL: R?.2
- new net SPX_CTCSS_DET: D?.2 (A), D?.6 (IO5), J?.1
- new net SPX_CTCSS_DET_ISOL: R?.1, U?.3
- new net SPX_ENABLE_CNTRL: R?.1
- new net SPX_FLAT_PTT: D?.3 (IO2), J?.9, SW?.6 (C)
- new net SPX_FLAT_TX_AUD: D?.4 (IO3), J?.2, SW?.3 (C)
- new net SPX_PIN6: J?.6
- new net SPX_PIN8: J?.8
- new net SPX_PTT: D?.1 (IO1), J?.4, SW?.4 (A)
- new net SPX_RX_AUD: C?.1, D?.5 (IO4), J?.3
- new net SPX_RX_ISOL: K?.12, TR?.P$3
- new net SPX_RX_ISOL_SW: K?.11
- new net SPX_TX_AUD: J?.5, SW?.1 (A)
- new net SPX_TX_ISOL: TR?.P$3
- new net ~{DPX_INHIBIT}: R?.1
- new net ~{DPX_MUTE}: R?.1
- new net ~{RMT_DIR_DUPLEX_PTT}: D?.3 (IO2), R?.1, X?.8
- new net ~{RMT_DIR_SIMPLEX_PTT}: D?.4 (IO3), R?.1, X?.3
- new net ~{RMT_DPX_INHIBIT}: D?.6 (IO5), R?.1, X?.7
- new net ~{RMT_DPX_LOOP_INHIBIT}: D?.1 (IO1), R?.1, X?.6
- new net ~{RMT_SPX_INHIBIT}: D?.5 (IO4), R?.1, X?.1
- no-connect marks 0 -> 7

Commit message: connector annotated
pcb updated after manually annotating back connector sheet

all scheets reanotated in new way

all scheets reanotated in new way ...
Parts:
- gave numbers to parts that had none: 61
