File: fm-rpt-connectors.kicad_sch (KiCad schematic)
At the start: 61 parts, among them J601 DUPLEX_RX, J602 SIMPLEX, J603 Conn_01x03_Male, J604 DUPLEX_TX, K601 RM12-3011-35-1005, K602 RM12__SPDT, Q601 BC856, Q602 BC856, SW601 SW_Push_DPDT, SW602 SW_Push_DPDT, U601 SFH617A-1, U602 SFH617A-1, U603 SFH617A-1, U604 SFH617A-1, U605 SFH617A-1, U606 SFH617A-1, U607 SFH617A-1, X601 PC, X602 REMOTE

Commit message: gerber files, some minor bugs in PCB solved
Parts:
- added R623, R624: 0, Resistor_SMD:R_0805_2012Metric_Pad1.20x1.40mm_HandSolder, symbol Device:R
- added R625: 660, Resistor_SMD:R_0805_2012Metric_Pad1.20x1.40mm_HandSolder, symbol Device:R
- R601, R602, R603: value R -> 680
Connections:
- net GND2: now also U601.2, R623.1
- net GND3: now also R624.1
- net GNDS: no longer U601.2, U602.2
- net at U607.4: now also R625.1; no longer SW602.2 (B)
- new net: R623.2, R624.2, U602.2
- new net: R625.2, SW602.2 (B)
Other:
- note added: "R623/R624/R625 is used to configure what kind of interface duplex radios have. Normally place only R623, DO NOT place R624 and use 0R as R625. This is when two radios are working as a part of full duplex port. In such config RX radio must have separate CTCSS / Carrier detect output and single ended line audio out (non bridged audio power amp like in Motorola GP300) If controller should work as tw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"
- company: (none) -> ML Elektronika Mateusz Lubecki
- title: (none) -> ParaCNTRL - FM repeater controller made of 74xx and analog
- moved on the sheet: D601, R602

Commit message: bugfix: not negating DPX_TX_TAIL_CLR before feeding 74hc107
Other:
- note added: "R623/R624/R625 are used to configure what kind of interface duplex radios have. Normally place only R623, DO NOT place R624 and use 0R as R625. This is when two radios are working as a part of full duplex port. In such config RX radio must have separate CTCSS / Carrier detect, active high output and single ended, line level audio out (not a bridged audio power amp like in Motorola GP300) If contr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"
- note removed: "R623/R624/R625 is used to configure what kind of interface duplex radios have. Normally place only R623, DO NOT place R624 and use 0R as R625. This is when two radios are working as a part of full duplex port. In such config RX radio must have separate CTCSS / Carrier detect output and single ended line audio out (non bridged audio power amp like in Motorola GP300) If controller should work as tw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"
Changed lines of the file:
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@@
     (stroke (width 0) (type default) (color 0 0 0 0))
   )
-  (text "R623/R624/R625 is used to configure what \nkind of interface duplex radios have.\n\nNormally place only R623, DO NOT place R624\nand use 0R as R625. This is when two radios\nare working as a part of full duplex port. \nIn such config RX radio must have separate\nCTCSS / Carrier detect output and single\nended line audio out (non bridged audio\npower amp like in Motorola GP300)\n\nIf controller should work as two direction\nsimplex-simplex repeater, with handheld \nradio on a 'duplex' port side, DO NOT place\nR623, place R624 and use about 1k as R625. \nThen connect RX audio output between pin7 \nand pin3 of J601 "
-    (at 128.27 168.275 0)
+  (text "R623/R624/R625 are used to configure what \nkind of interface duplex radios have.\n\nNormally place only R623, DO NOT place R624\nand use 0R as R625. This is when two radios\nare working as a part of full duplex port. \nIn such config RX radio must have separate\nCTCSS / Carrier detect, active high output\nand single ended, line level audio out \n(not a bridged audio power amp \nlike in Motorola GP300)\n\nIf controller should work as two direction\nsimplex-simplex repeater, with handheld \nradio on a 'duplex' port side, DO NOT place\nR623, place R624 and use about 1k as R625. \nThen connect RX audio output between pin7 \nand pin3 of J601. a SPK+ (positive DC offset\nin relation to radio ground) must be on\npin7 and SPK- (negative DC offset in relation\nto ground or no offset at all) must be on\npin7. Otherwise input blocking capacitor might\nexplode!"
+    (at 128.905 177.8 0)
     (effects (font (size 1.27 1.27)) (justify left bottom))
   )

Commit message: roger beep sligtly redesigned during assembly and debugging, bom with prices
Parts:
- R617, R618, R619, R620, R621: value 10k -> 20k
Changed lines of the file:
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@@
     (in_bom yes) (on_board yes)
     (property "Reference" "R620" (id 0) (at 206.375 72.39 90))
-    (property "Value" "10k" (id 1) (at 206.375 74.9269 90))
+    (property "Value" "20k" (id 1) (at 206.375 74.9269 90))
     (property "Footprint" "Resistor_SMD:R_0805_2012Metric_Pad1.20x1.40mm_HandSolder" (id 2) (at 206.375 75.057 90)
       (effects (font (size 1.27 1.27)) hide)
@@
     (in_bom yes) (on_board yes) (fields_autoplaced)
     (property "Reference" "R621" (id 0) (at 206.375 79.7392 90))
-    (property "Value" "10k" (id 1) (at 206.375 82.2761 90))
+    (property "Value" "20k" (id 1) (at 206.375 82.2761 90))
     (property "Footprint" "Resistor_SMD:R_0805_2012Metric_Pad1.20x1.40mm_HandSolder" (id 2) (at 206.375 82.677 90)
       (effects (font (size 1.27 1.27)) hide)
@@
     (in_bom yes) (on_board yes) (fields_autoplaced)
     (property "Reference" "R618" (id 0) (at 203.835 122.9192 90))
-    (property "Value" "10k" (id 1) (at 203.835 125.4561 90))
+    (property "Value" "20k" (id 1) (at 203.835 125.4561 90))
     (property "Footprint" "Resistor_SMD:R_0805_2012Metric_Pad1.20x1.40mm_HandSolder" (id 2) (at 203.835 125.857 90)
       (effects (font (size 1.27 1.27)) hide)
@@
     (in_bom yes) (on_board yes) (fields_autoplaced)
     (property "Reference" "R617" (id 0) (at 203.835 115.2992 90))
-    (property "Value" "10k" (id 1) (at 203.835 117.8361 90))
+    (property "Value" "20k" (id 1) (at 203.835 117.8361 90))
     (property "Footprint" "Resistor_SMD:R_0805_2012Metric_Pad1.20x1.40mm_HandSolder" (id 2) (at 203.835 118.237 90)
       (effects (font (size 1.27 1.27)) hide)
@@
     (in_bom yes) (on_board yes) (fields_autoplaced)
     (property "Reference" "R619" (id 0) (at 203.835 130.5392 90))
-    (property "Value" "10k" (id 1) (at 203.835 133.0761 90))
+    (property "Value" "20k" (id 1) (at 203.835 133.0761 90))
     (property "Footprint" "Resistor_SMD:R_0805_2012Metric_Pad1.20x1.40mm_HandSolder" (id 2) (at 203.835 133.477 90)
       (effects (font (size 1.27 1.27)) hide)

Commit message: pullup,pulldown resistors changed
Parts:
- R607, R608: value 51k -> 20k
- R610: value 10k -> 20k
- R612, R616: value 22k -> 51k
- R613, R615: value 22k -> 20k
- R614: value 2k2 -> 51k
Changed lines of the file:
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@@
     (in_bom yes) (on_board yes) (fields_autoplaced)
     (property "Reference" "R610" (id 0) (at 102.235 121.6492 90))
-    (property "Value" "10k" (id 1) (at 102.235 124.1861 90))
+    (property "Value" "20k" (id 1) (at 102.235 124.1861 90))
     (property "Footprint" "Resistor_SMD:R_0805_2012Metric_Pad1.20x1.40mm_HandSolder" (id 2) (at 102.235 128.143 90)
       (effects (font (size 1.27 1.27)) hide)
@@
       (effects (font (size 1.27 1.27)) (justify right))
     )
-    (property "Value" "22k" (id 1) (at 140.843 27.7372 0)
+    (property "Value" "20k" (id 1) (at 140.843 27.7372 0)
       (effects (font (size 1.27 1.27)) (justify right))
     )
@@
       (effects (font (size 1.27 1.27)) (justify right))
     )
-    (property "Value" "22k" (id 1) (at 137.033 116.6372 0)
+    (property "Value" "20k" (id 1) (at 137.033 116.6372 0)
       (effects (font (size 1.27 1.27)) (justify right))
     )
@@
       (effects (font (size 1.27 1.27)) (justify right))
     )
-    (property "Value" "22k" (id 1) (at 140.843 35.3572 0)
+    (property "Value" "51k" (id 1) (at 140.843 35.3572 0)
       (effects (font (size 1.27 1.27)) (justify right))
     )
@@
       (effects (font (size 1.27 1.27)) (justify right))
     )
-    (property "Value" "2k2" (id 1) (at 137.033 124.2572 0)
+    (property "Value" "51k" (id 1) (at 137.033 124.2572 0)
       (effects (font (size 1.27 1.27)) (justify right))
     )
@@
       (effects (font (size 1.27 1.27)) (justify right))
     )
-    (property "Value" "22k" (id 1) (at 133.223 35.3572 0)
+    (property "Value" "51k" (id 1) (at 133.223 35.3572 0)
       (effects (font (size 1.27 1.27)) (justify right))
     )
@@
     (in_bom yes) (on_board yes) (fields_autoplaced)
     (property "Reference" "R608" (id 0) (at 98.425 61.9592 90))
-    (property "Value" "51k" (id 1) (at 98.425 64.4961 90))
+    (property "Value" "20k" (id 1) (at 98.425 64.4961 90))
     (property "Footprint" "Resistor_SMD:R_0805_2012Metric_Pad1.20x1.40mm_HandSolder" (id 2) (at 98.425 68.453 90)
       (effects (font (size 1.27 1.27)) hide)
@@
     (in_bom yes) (on_board yes) (fields_autoplaced)
     (property "Reference" "R607" (id 0) (at 98.425 49.2592 90))
-    (property "Value" "51k" (id 1) (at 98.425 51.7961 90))
+    (property "Value" "20k" (id 1) (at 98.425 51.7961 90))
     (property "Footprint" "Resistor_SMD:R_0805_2012Metric_Pad1.20x1.40mm_HandSolder" (id 2) (at 98.425 55.753 90)
       (effects (font (size 1.27 1.27)) hide)

Commit message: simplex remote control tone detector redesigned, gerber files for hw-rev b
Connections:
- net SPX_ENABLE_CNTRL renamed SPX_ENABLE
Changed lines of the file:
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@@
   (title_block
     (title "ParaCNTRL - FM repeater controller made of 74xx and analog")
-    (date "2023-02-23")
+    (date "2023-05-07")
     (rev "B")
     (company "ML Elektronika Mateusz Lubecki")
@@
     )
   )
-  (global_label "SPX_ENABLE_CNTRL" (shape input) (at 137.795 128.27 0) (fields_autoplaced)
+  (global_label "SPX_ENABLE" (shape input) (at 137.795 128.27 0) (fields_autoplaced)
     (effects (font (size 1.27 1.27)) (justify left))
-    (property "Intersheet References" "${INTERSHEET_REFS}" (id 0) (at 158.7138 128.3494 0)
+    (property "Intersheet References" "${INTERSHEET_REFS}" (id 0) (at 151.88 128.1906 0)
       (effects (font (size 1.27 1.27)) (justify left) hide)
     )

Commit message: some changes after testing hw revision b
Parts:
- R603: value 680 -> 620
- R611: value 330 -> 390
- R622: value 660 -> 390
Changed lines of the file:
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@@
   (title_block
     (title "ParaCNTRL - FM repeater controller made of 74xx and analog")
-    (date "2023-05-07")
-    (rev "B")
+    (date "2023-06-17")
+    (rev "C")
     (company "ML Elektronika Mateusz Lubecki")
     (comment 1 "Connectors and ground separation circuits")
@@
     (in_bom yes) (on_board yes) (fields_autoplaced)
     (property "Reference" "R622" (id 0) (at 208.28 39.7342 90))
-    (property "Value" "660" (id 1) (at 208.28 42.2711 90))
+    (property "Value" "390" (id 1) (at 208.28 42.2711 90))
     (property "Footprint" "Resistor_SMD:R_0805_2012Metric_Pad1.20x1.40mm_HandSolder" (id 2) (at 208.28 46.228 90)
       (effects (font (size 1.27 1.27)) hide)
@@
     (in_bom yes) (on_board yes) (fields_autoplaced)
     (property "Reference" "R611" (id 0) (at 106.045 86.0892 90))
-    (property "Value" "330" (id 1) (at 106.045 88.6261 90))
+    (property "Value" "390" (id 1) (at 106.045 88.6261 90))
     (property "Footprint" "Resistor_SMD:R_0805_2012Metric_Pad1.20x1.40mm_HandSolder" (id 2) (at 106.045 92.583 90)
       (effects (font (size 1.27 1.27)) hide)
@@
     (in_bom yes) (on_board yes) (fields_autoplaced)
     (property "Reference" "R603" (id 0) (at 73.025 116.5692 90))
-    (property "Value" "680" (id 1) (at 73.025 119.1061 90))
+    (property "Value" "620" (id 1) (at 73.025 119.1061 90))
     (property "Footprint" "Resistor_SMD:R_0805_2012Metric_Pad1.20x1.40mm_HandSolder" (id 2) (at 73.025 123.063 90)
       (effects (font (size 1.27 1.27)) hide)
