File: fm-rpt-control-555.kicad_sch (KiCad schematic)
At the start: 6 parts, among them U26 NE555D

Commit message: connector annotated
pcb updated after manually annotating back connector sheet

all scheets reanotated in new way

all scheets reanotated in new way ...
Parts:
- renumbered C6 to C501, C7 to C502, C60 to C503, R48 to R501, R49 to R502, U26 to U501
Changed lines of the file:
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@@
   (symbol (lib_id "paratnc_cp_import:GND") (at 141.605 112.395 0) (unit 1)
     (in_bom yes) (on_board yes) (fields_autoplaced)
-    (property "Reference" "#GND0109" (id 0) (at 141.605 112.395 0)
+    (property "Reference" "#GND0503" (id 0) (at 141.605 112.395 0)
       (effects (font (size 1.27 1.27)) hide)
     )
@@
   (symbol (lib_id "paratnc_cp_import:GND") (at 111.76 111.76 0) (unit 1)
     (in_bom yes) (on_board yes) (fields_autoplaced)
-    (property "Reference" "#GND0107" (id 0) (at 111.76 111.76 0)
+    (property "Reference" "#GND0501" (id 0) (at 111.76 111.76 0)
       (effects (font (size 1.27 1.27)) hide)
     )
@@
   (symbol (lib_id "Device:R") (at 167.005 99.695 180) (unit 1)
     (in_bom yes) (on_board yes) (fields_autoplaced)
-    (property "Reference" "R49" (id 0) (at 168.783 98.8603 0)
+    (property "Reference" "R502" (id 0) (at 168.783 98.8603 0)
       (effects (font (size 1.27 1.27)) (justify right))
     )
@@
   (symbol (lib_id "Device:R") (at 167.005 90.805 180) (unit 1)
     (in_bom yes) (on_board yes)
-    (property "Reference" "R48" (id 0) (at 168.783 89.9703 0)
+    (property "Reference" "R501" (id 0) (at 168.783 89.9703 0)
       (effects (font (size 1.27 1.27)) (justify right))
     )
@@
   (symbol (lib_id "Timer:NE555D") (at 141.605 98.425 0) (unit 1)
     (in_bom yes) (on_board yes) (fields_autoplaced)
-    (property "Reference" "U26" (id 0) (at 143.6244 87.1052 0)
+    (property "Reference" "U501" (id 0) (at 143.6244 87.1052 0)
       (effects (font (size 1.27 1.27)) (justify left))
     )
@@
   (symbol (lib_id "Device:C") (at 111.76 102.87 0) (unit 1)
     (in_bom yes) (on_board yes) (fields_autoplaced)
-    (property "Reference" "C6" (id 0) (at 114.681 102.0353 0)
+    (property "Reference" "C501" (id 0) (at 114.681 102.0353 0)
       (effects (font (size 1.27 1.27)) (justify left))
     )
@@
   (symbol (lib_id "Device:C") (at 126.365 107.315 0) (unit 1)
     (in_bom yes) (on_board yes) (fields_autoplaced)
-    (property "Reference" "C7" (id 0) (at 129.286 106.4803 0)
+    (property "Reference" "C502" (id 0) (at 129.286 106.4803 0)
       (effects (font (size 1.27 1.27)) (justify left))
     )
@@
   (symbol (lib_id "paratnc_cp_import:GND") (at 126.365 113.665 0) (unit 1)
     (in_bom yes) (on_board yes) (fields_autoplaced)
-    (property "Reference" "#GND0111" (id 0) (at 126.365 113.665 0)
+    (property "Reference" "#GND0502" (id 0) (at 126.365 113.665 0)
       (effects (font (size 1.27 1.27)) hide)
     )
@@
   (symbol (lib_id "Device:C_Polarized") (at 163.195 107.315 0) (unit 1)
     (in_bom yes) (on_board yes) (fields_autoplaced)
-    (property "Reference" "C60" (id 0) (at 166.116 105.5913 0)
+    (property "Reference" "C503" (id 0) (at 166.116 105.5913 0)
       (effects (font (size 1.27 1.27)) (justify left))
     )
