File: fm-rpt-control-tonedetect.kicad_sch (KiCad schematic)
At the start: 16 parts, among them IC701 LM567CH, IC702 74HC107D, U701 LMV358

Commit message: changing rogereep duration depends on simplex enable or not
Connections:
- net ~{SPX_ENABLE_CNTRL}: now reaches IC702.6 (~{Q})
Changed lines of the file:
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@@
+    (stroke (width 0) (type default) (color 0 0 0 0))
+  )
+  (wire (pts (xy 220.726 76.454) (xy 223.012 76.454))
     (stroke (width 0) (type default) (color 0 0 0 0))
   )
@@
     (effects (font (size 1.27 1.27)) (justify left bottom))
   )
+  (global_label "~{SPX_ENABLE_CNTRL}" (shape input) (at 223.012 76.454 0) (fields_autoplaced)
+    (effects (font (size 1.27 1.27)) (justify left))
+    (property "Intersheet References" "${INTERSHEET_REFS}" (id 0) (at 243.9308 76.3746 0)
+      (effects (font (size 1.27 1.27)) (justify left) hide)
+    )
+  )
   (global_label "+5V" (shape input) (at 194.056 63.754 180) (fields_autoplaced)

Commit message: some changes after testing hw revision b
Parts:
- added IC?: 74HC107D, Package_SO:SO-14_3.9x8.65mm_P1.27mm, symbol jk_flipflop:74HC107D
- C703: value 2u2 -> 4u7
- R702: value 33k -> 10k
- R704: value 33k -> 51k
- R705: value 20k -> 5k1
Changed lines of the file:
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@@
   (title_block
     (title "ParaCNTRL - FM repeater controller made of 74xx and analog")
-    (date "2023-05-07")
-    (rev "B")
+    (date "2023-06-17")
+    (rev "C")
     (company "ML Elektronika Mateusz Lubecki")
     (comment 1 "Simplex enable remote control")
@@
     (in_bom yes) (on_board yes)
     (property "Reference" "R702" (id 0) (at 93.98 90.17 90))
-    (property "Value" "33k" (id 1) (at 93.98 92.202 90))
+    (property "Value" "10k" (id 1) (at 93.98 92.202 90))
     (property "Footprint" "Resistor_SMD:R_0805_2012Metric_Pad1.20x1.40mm_HandSolder" (id 2) (at 93.98 89.662 90)
       (effects (font (size 1.27 1.27)) hide)
@@
     (in_bom yes) (on_board yes)
     (property "Reference" "C703" (id 0) (at 128.524 83.82 90))
-    (property "Value" "2u2" (id 1) (at 128.524 76.9421 90))
+    (property "Value" "4u7" (id 1) (at 128.524 76.9421 90))
     (property "Footprint" "Capacitor_SMD:C_0805_2012Metric_Pad1.18x1.45mm_HandSolder" (id 2) (at 132.334 79.2988 0)
       (effects (font (size 1.27 1.27)) hide)
@@
     (pin "7")
   )
+  (symbol (lib_id "jk_flipflop:74HC107D") (at 211.328 97.282 0) (unit 3)
+    (in_bom yes) (on_board yes) (fields_autoplaced)
+    (property "Reference" "IC?" (id 0) (at 211.328 85.7794 0)
+      (effects (font (size 1.778 1.5113)))
+    )
+    (property "Value" "74HC107D" (id 1) (at 203.708 107.442 0)
+      (effects (font (size 1.778 1.5113)) (justify left bottom) hide)
+    )
+    (property "Footprint" "Package_SO:SO-14_3.9x8.65mm_P1.27mm" (id 2) (at 211.328 97.282 0)
+      (effects (font (size 1.27 1.27)) hide)
+    )
+    (property "Datasheet" "https://assets.nexperia.com/documents/data-sheet/74HC_HCT107.pdf" (id 3) (at 211.328 97.282 0)
+      (effects (font (size 1.27 1.27)) hide)
+    )
+    (pin "14")
+    (pin "7")
+  )
   (symbol (lib_id "Device:R") (at 170.942 82.804 180) (unit 1)
     (in_bom yes) (on_board yes) (fields_autoplaced)
@@
     (in_bom yes) (on_board yes)
     (property "Reference" "R704" (id 0) (at 110.49 90.424 90))
-    (property "Value" "33k" (id 1) (at 110.49 88.646 90))
+    (property "Value" "51k" (id 1) (at 110.49 88.646 90))
     (property "Footprint" "Resistor_SMD:R_0805_2012Metric_Pad1.20x1.40mm_HandSolder" (id 2) (at 110.49 94.234 90)
       (effects (font (size 1.27 1.27)) hide)
@@
       (effects (font (size 1.27 1.27)) (justify right))
     )
-    (property "Value" "20k" (id 1) (at 170.18 66.7262 0)
-      (effects (font (size 1.27 1.27)) (justify right))
-    )
+    (property "Value" "5k1" (id 1) (at 170.18 66.7262 0)
+      (effects (font (size 1.27 1.27)) (justify right))
+    )

Commit message: before fixing problems with potentiometers orientation
Parts:
- gave numbers to parts that had none: 1
Connections:
- net +5V: now also IC702.14 (VCC)
- net GND: now also IC702.7 (GND)
- net DPX_RX_ISOL_SW renamed DPX_RX_ISOL_SW_LOOP
Other:
- moved on the sheet: IC702C
Changed lines of the file:
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@@
+    (stroke (width 0) (type default) (color 0 0 0 0))
+  )
+  (wire (pts (xy 238.506 133.35) (xy 238.506 134.112))
     (stroke (width 0) (type default) (color 0 0 0 0))
   )
@@
   )
   (wire (pts (xy 249.428 113.03) (xy 249.428 116.332))
+    (stroke (width 0) (type default) (color 0 0 0 0))
+  )
+  (wire (pts (xy 238.506 109.728) (xy 238.506 111.76))
     (stroke (width 0) (type default) (color 0 0 0 0))
   )
@@
     (effects (font (size 1.27 1.27)) (justify left))
     (property "Intersheet References" "${INTERSHEET_REFS}" (id 0) (at 243.9308 76.3746 0)
+      (effects (font (size 1.27 1.27)) (justify left) hide)
+    )
+  )
+  (global_label "+5V" (shape input) (at 238.506 109.728 90) (fields_autoplaced)
+    (effects (font (size 1.27 1.27)) (justify left))
+    (property "Intersheet References" "${INTERSHEET_REFS}" (id 0) (at 238.4266 103.4444 90)
       (effects (font (size 1.27 1.27)) (justify left) hide)
     )
@@
     )
   )
-  (global_label "DPX_RX_ISOL_SW" (shape input) (at 75.438 82.55 180) (fields_autoplaced)
+  (global_label "DPX_RX_ISOL_SW_LOOP" (shape input) (at 75.438 82.55 180) (fields_autoplaced)
     (effects (font (size 1.27 1.27)) (justify right))
-    (property "Intersheet References" "${INTERSHEET_REFS}" (id 0) (at 57.0592 82.4706 0)
+    (property "Intersheet References" "${INTERSHEET_REFS}" (id 0) (at 51.1325 82.4706 0)
       (effects (font (size 1.27 1.27)) (justify right) hide)
     )
@@
     (pin "1")
     (pin "2")
+  )
+  (symbol (lib_id "paratnc_cp_import:GND") (at 238.506 136.652 0) (unit 1)
+    (in_bom yes) (on_board yes) (fields_autoplaced)
+    (property "Reference" "#GND0102" (id 0) (at 238.506 136.652 0)
+      (effects (font (size 1.27 1.27)) hide)
+    )
+    (property "Value" "GND" (id 1) (at 238.506 138.7608 0)
+      (effects (font (size 1.4986 1.4986)))
+    )
+    (property "Footprint" "" (id 2) (at 238.506 136.652 0)
+      (effects (font (size 1.27 1.27)) hide)
+    )
+    (property "Datasheet" "" (id 3) (at 238.506 136.652 0)
+      (effects (font (size 1.27 1.27)) hide)
+    )
+    (pin "1")
   )
   (symbol (lib_id "paratnc_cp_import:GND") (at 249.428 134.874 0) (unit 1)
@@
     (pin "7")
   )
-  (symbol (lib_id "jk_flipflop:74HC107D") (at 211.328 97.282 0) (unit 3)
-    (in_bom yes) (on_board yes) (fields_autoplaced)
-    (property "Reference" "IC?" (id 0) (at 211.328 85.7794 0)
+  (symbol (lib_id "jk_flipflop:74HC107D") (at 238.506 123.19 0) (unit 3)
+    (in_bom yes) (on_board yes) (fields_autoplaced)
+    (property "Reference" "IC702" (id 0) (at 238.506 111.6874 0)
       (effects (font (size 1.778 1.5113)))
     )
-    (property "Value" "74HC107D" (id 1) (at 203.708 107.442 0)
+    (property "Value" "74HC107D" (id 1) (at 230.886 133.35 0)
       (effects (font (size 1.778 1.5113)) (justify left bottom) hide)
     )
-    (property "Footprint" "Package_SO:SO-14_3.9x8.65mm_P1.27mm" (id 2) (at 211.328 97.282 0)
-      (effects (font (size 1.27 1.27)) hide)
-    )
-    (property "Datasheet" "https://assets.nexperia.com/documents/data-sheet/74HC_HCT107.pdf" (id 3) (at 211.328 97.282 0)
-      (effects (font (size 1.27 1.27)) hide)
-    )
+    (property "Footprint" "Package_SO:SO-14_3.9x8.65mm_P1.27mm" (id 2) (at 238.506 123.19 0)
+      (effects (font (size 1.27 1.27)) hide)
+    )
+    (property "Datasheet" "https://assets.nexperia.com/documents/data-sheet/74HC_HCT107.pdf" (id 3) (at 238.506 123.19 0)
+      (effects (font (size 1.27 1.27)) hide)
+    )
